File: design-files/CoPicoVision.kicad_sch (KiCad schematic)
At the start: 0 parts

Commit message: Reset and clock.
Parts:
- added C101, C103, C104: 0.1µF, symbol Device:C_Small
- added C102: 100µF, symbol Device:C_Polarized_Small
- added D101: 1N4148, Diode_THT:D_DO-35_SOD27_P7.62mm_Horizontal, symbol Diode:1N4148
- added RN101: 3K3, Resistor_THT:R_Array_SIP9, symbol Device:R_Network08_Split
- added SW101: SW_Push, symbol Switch:SW_Push
- added U101: Z80CPU, symbol CPU:Z80CPU
- added U102: DS1813, Package_TO_SOT_THT:TO-92_Inline, symbol jrt-ICs:DS1813
- added U103: 74LS05, symbol 74xx:74LS05
- added X101: 3.579545MHZ, Oscillator:Oscillator_DIP-8, symbol Oscillator:CXO_DIP8
Connections:
- new net: C102.1, D101.2 (A), RN101.2 (R1.2), U102.2 (Vcc)
- new net: SW101.2, U102.3 (GND)
- new net A0: U101.30 (A0)
- new net A1: U101.31 (A1)
- new net A10: U101.40 (A10)
- new net A11: U101.1 (A11)
- new net A12: U101.2 (A12)
- new net A13: U101.3 (A13)
- new net A14: U101.4 (A14)
- new net A15: U101.5 (A15)
- new net A2: U101.32 (A2)
- new net A3: U101.33 (A3)
- new net A4: U101.34 (A4)
- new net A5: U101.35 (A5)
- new net A6: U101.36 (A6)
- new net A7: U101.37 (A7)
- new net A8: U101.38 (A8)
- new net A9: U101.39 (A9)
- new net CPUCLK: X101.5 (OUT)
- new net D0: U101.14 (D0)
- new net D1: U101.15 (D1)
- new net D2: U101.12 (D2)
- new net D3: U101.8 (D3)
- new net D4: U101.7 (D4)
- new net D5: U101.9 (D5)
- new net D6: U101.10 (D6)
- new net D7: U101.13 (D7)
- new net GND: C101.2, C102.2, C103.2, C104.2, U101.29 (GND), U103.7 (GND), X101.4 (GND)
- new net VCC: C101.1, C103.1, C104.1, D101.1 (K), RN101.1 (R1), RN101.1 (R1), RN101.1 (R1), RN101.1 (R1), U101.11 (VCC), U101.25 (~{BUSRQ}), U103.14 (VCC), X101.8 (Vcc)
- new net ~{CPUCLK}: U101.6 (~{CLK})
- new net ~{INT}: RN101.4 (R3.2), U101.16 (~{INT})
- new net ~{IORQ}: U101.20 (~{IORQ})
- new net ~{M1}: U101.27 (~{M1})
- new net ~{MREQ}: U101.19 (~{MREQ})
- new net ~{NMI}: RN101.5 (R4.2), U101.17 (~{NMI})
- new net ~{RD}: U101.21 (~{RD})
- new net ~{RESET}: SW101.1, U101.26 (~{RESET}), U102.1 (~{RST})
- new net ~{RFSH}: U101.28 (~{RFSH})
- new net ~{WAIT}: RN101.3 (R2.2), U101.24 (~{WAIT})
- new net ~{WR}: U101.22 (~{WR})
- no-connect marks 0 -> 3

Commit message: Use a 74ACT05 rather than a 74LS05.
Parts:
- U103: value 74LS05 -> 74ACT05
Changed lines of the file:
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@@
       (effects (font (size 1.27 1.27)) (justify left))
     )
-    (property "Value" "74LS05" (at 247.65 147.193 0)
+    (property "Value" "74ACT05" (at 247.65 147.193 0)
       (effects (font (size 1.27 1.27)) (justify left))
     )
@@
       (effects (font (size 1.27 1.27)) hide)
     )
-    (property "Datasheet" "http://www.ti.com/lit/gpn/sn74LS05" (at 241.046 145.288 0)
+    (property "Datasheet" "https://www.ti.com/lit/ds/symlink/cd74act05.pdf" (at 241.046 145.288 0)
       (effects (font (size 1.27 1.27)) hide)
     )

Commit message: Added video circuit.
Parts:
- added unit 6 of RN101
- added unit 7 of RN101
- added unit 8 of RN101
- added unit 5 of RN101
- added unit 4 of U103
- added unit 3 of U103
- added unit 5 of U103
- added unit 6 of U103
- U101: footprint (none) -> Package_DIP:DIP-40_W15.24mm_Socket
Connections:
- net GND: now also U103.11, U103.13, U103.5, U103.9
- no-connect marks 3 -> 15
Other:
- added sheet Video (CoPicoVision_video.kicad_sch)

Commit message: Get footprints on everything.
Parts:
- C101, C103, C104: footprint (none) -> Capacitor_THT:C_Disc_D3.8mm_W2.6mm_P2.50mm
- C102: footprint (none) -> Capacitor_THT:CP_Radial_D6.3mm_P2.50mm
- SW101: footprint (none) -> Button_Switch_THT:SW_PUSH_6mm
- U103: footprint (none) -> Package_DIP:DIP-14_W7.62mm_Socket
Changed lines of the file:
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@@
       (effects (font (size 1.27 1.27)) (justify left))
     )
-    (property "Footprint" "" (at 266.446 129.159 0)
+    (property "Footprint" "Package_DIP:DIP-14_W7.62mm_Socket" (at 266.446 129.159 0)
       (effects (font (size 1.27 1.27)) hide)
     )
@@
       (effects (font (size 1.27 1.27)) (justify left))
     )
-    (property "Footprint" "" (at 266.446 120.015 0)
+    (property "Footprint" "Package_DIP:DIP-14_W7.62mm_Socket" (at 266.446 120.015 0)
       (effects (font (size 1.27 1.27)) hide)
     )
@@
       (effects (font (size 1.27 1.27)) (justify left))
     )
-    (property "Footprint" "" (at 30.988 176.276 0)
+    (property "Footprint" "Capacitor_THT:C_Disc_D3.8mm_W2.6mm_P2.50mm" (at 30.988 176.276 0)
       (effects (font (size 1.27 1.27)) hide)
     )
@@
       (effects (font (size 1.27 1.27)) (justify left))
     )
-    (property "Footprint" "" (at 266.446 138.684 0)
+    (property "Footprint" "Package_DIP:DIP-14_W7.62mm_Socket" (at 266.446 138.684 0)
       (effects (font (size 1.27 1.27)) hide)
     )
@@
       (effects (font (size 1.27 1.27)) (justify left))
     )
-    (property "Footprint" "" (at 241.046 145.288 0)
+    (property "Footprint" "Package_DIP:DIP-14_W7.62mm_Socket" (at 241.046 145.288 0)
       (effects (font (size 1.27 1.27)) hide)
     )
@@
       (effects (font (size 1.27 1.27)))
     )
-    (property "Footprint" "" (at 188.468 151.257 0)
+    (property "Footprint" "Button_Switch_THT:SW_PUSH_6mm" (at 188.468 151.257 0)
       (effects (font (size 1.27 1.27)) hide)
     )
@@
       (effects (font (size 1.27 1.27)) (justify left))
     )
-    (property "Footprint" "" (at 42.037 176.276 0)
+    (property "Footprint" "Capacitor_THT:C_Disc_D3.8mm_W2.6mm_P2.50mm" (at 42.037 176.276 0)
       (effects (font (size 1.27 1.27)) hide)
     )
@@
       (effects (font (size 1.27 1.27)) (justify left))
     )
-    (property "Footprint" "" (at 53.213 176.276 0)
+    (property "Footprint" "Capacitor_THT:C_Disc_D3.8mm_W2.6mm_P2.50mm" (at 53.213 176.276 0)
       (effects (font (size 1.27 1.27)) hide)
     )
@@
       (effects (font (size 1.27 1.27)) (justify left))
     )
-    (property "Footprint" "" (at 162.687 142.24 0)
+    (property "Footprint" "Capacitor_THT:CP_Radial_D6.3mm_P2.50mm" (at 162.687 142.24 0)
       (effects (font (size 1.27 1.27)) hide)
     )
@@
       (effects (font (size 1.27 1.27)) (justify left))
     )
-    (property "Footprint" "" (at 266.446 148.082 0)
-      (effects (font (size 1.27 1.27)) hide)
-    )
+    (property "Footprint" "Package_DIP:DIP-14_W7.62mm_Socket" (at 266.446 148.082 0)
+      (effects (font (size 1.27 1.27)) hide)
+    )

Commit message: First pass at rough PCB layout.
Connections:
- net ~{CPUCLK} is gone; now on net CPUCLK: U101.6 (~{CLK})
Changed lines of the file:
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@@
     )
   )
-  (global_label "~{CPUCLK}" (shape input) (at 29.845 88.392 180) (fields_autoplaced)
+  (global_label "CPUCLK" (shape input) (at 29.845 88.392 180) (fields_autoplaced)
     (effects (font (size 1.27 1.27)) (justify right))
     (property "Intersheetrefs" "${INTERSHEET_REFS}" (at 19.5006 88.392 0)

Commit message: Add controller ports just to get them onto the board.
Other:
- added sheet Controller Interface (CoPicoVision_controllers.kicad_sch)
Changed lines of the file:
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@@
+    )
+  )
+  (sheet (at 93.218 17.018) (size 26.543 16.383) (fields_autoplaced)
+    (stroke (width 0.1524) (type solid))
+    (fill (color 0 0 0 0.0000))
+    (property "Sheetname" "Controller Interface" (at 93.218 16.3064 0)
+      (effects (font (size 1.27 1.27)) (justify left bottom))
+    )
+    (property "Sheetfile" "CoPicoVision_controllers.kicad_sch" (at 93.218 33.9856 0)
+      (effects (font (size 1.27 1.27)) (justify left top))
+    )
+    (instances
+      (project "CoPicoVision"
+        (path "/d4d4c0fa-7a39-4b72-9fdb-c481b1e41ed4" (page "4"))
+      )
     )
   )

Commit message: Lay out some additional bits.
Other:
- added sheet Audio (CoPicoVision_audio.kicad_sch)
Changed lines of the file:
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@@
+    )
+  )
+  (sheet (at 134.62 16.891) (size 29.21 17.018) (fields_autoplaced)
+    (stroke (width 0.1524) (type solid))
+    (fill (color 0 0 0 0.0000))
+    (property "Sheetname" "Audio" (at 134.62 16.1794 0)
+      (effects (font (size 1.27 1.27)) (justify left bottom))
+    )
+    (property "Sheetfile" "CoPicoVision_audio.kicad_sch" (at 134.62 34.4936 0)
+      (effects (font (size 1.27 1.27)) (justify left top))
+    )
+    (instances
+      (project "CoPicoVision"
+        (path "/d4d4c0fa-7a39-4b72-9fdb-c481b1e41ed4" (page "5"))
+      )
     )
   )

Commit message: Add power supply.  PCB checkpoint.
Parts:
- added C105: 100µF, Capacitor_THT:CP_Radial_D6.3mm_P2.50mm, symbol Device:C_Polarized_Small
- added C106, C107: 10µF, Capacitor_SMD:C_0805_2012Metric_Pad1.18x1.45mm_HandSolder, symbol Device:C_Small
- added D102: ESDA25L, Package_TO_SOT_SMD:SOT-23, symbol Power_Protection:SP0502BAHT
- added H101, H102, H103, H104: MountingHole, MountingHole:MountingHole_3.5mm, symbol Mechanical:MountingHole
- added J101: USB_C_Receptacle_PowerOnly_6P, Connector_USB:USB_C_Receptacle_GCT_USB4085, symbol Connector:USB_C_Receptacle_PowerOnly_6P
- added Q101: MMFTP3334K-AQ, Package_TO_SOT_SMD:SOT-23, symbol Device:Q_PMOS_GSD
- added R101, R102: 5K1, Resistor_SMD:R_0805_2012Metric_Pad1.20x1.40mm_HandSolder, symbol Device:R_Small
- added R103: 10K, Resistor_SMD:R_0805_2012Metric_Pad1.20x1.40mm_HandSolder, symbol Device:R_Small
- added SW102: SW_Push, Button_Switch_THT:SW_PUSH_6mm, symbol Switch:SW_Push
- added U104: ICL7660A, Package_SO:SOIC-8_3.9x4.9mm_P1.27mm, symbol Regulator_SwitchedCapacitor:ICL7660
- added U105: MAX16054, Package_TO_SOT_SMD:SOT-23-6, symbol jrt-ICs:MAX16054
Connections:
- net GND: now also C105.2, C107.2, D102.3 (A), J101.A12 (GND), J101.B12 (GND), J101.S1 (SHIELD), R101.2, R102.2, SW102.1, U104.3 (GND), U105.2 (GND), U105.3 (CLEAR)
- net VCC: now also Q101.3 (D), U104.8 (V+)
- new net: C106.1, U104.2 (CAP+)
- new net: C106.2, U104.4 (CAP-)
- new net: C105.1, J101.A9 (VBUS), J101.B9 (VBUS), Q101.2 (S), R103.1, U105.6 (Vcc)
- new net: Q101.1 (G), R103.2, U105.4 (~{OUT})
- new net: D102.1 (K), J101.B5 (CC2), R101.1
- new net: D102.2 (K), J101.A5 (CC1), R102.1
- new net: SW102.2, U105.1 (IN)
- new net -5V: C107.1, U104.5 (VOUT)
- no-connect marks 15 -> 18
Other:
- moved on the sheet: C101, C102, C103, C104, D101, RN101A, RN101B, RN101C, RN101D, RN101E, RN101F, RN101G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
