File: design-files/CoPicoVision.kicad_sch (KiCad schematic)
At the start: 33 parts, among them J101 USB_C_Receptacle_PowerOnly_6P, J102 Conn_02x15_Odd_Even, Q101 MMFTP3334K-AQ, SW101 SW_Push, SW102 SW_Push, U101 Z80CPU, U102 DS1813, U103 74ACT05, U104 ICL7660A, U105 MAX16054, X101 3.579545MHZ

Commit message: More routing.
Connections:
- net VBUS: now reaches C105.1, J101.A9 (VBUS), J101.B9 (VBUS), Q101.2 (S), R103.1, U105.6 (Vcc)
Changed lines of the file:
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@@
   (no_connect (at 201.676 161.925))
   (no_connect (at 179.197 154.559))
-  (no_connect (at 272.669 138.557))
+  (no_connect (at 272.796 138.557))
   (no_connect (at 29.845 113.792))
   (no_connect (at 98.552 170.434))
@@
     (stroke (width 0) (type default))
   )
+  (label "VBUS" (at 114.173 50.165 90) (fields_autoplaced)
+    (effects (font (size 1.27 1.27)) (justify left bottom))
+  )
   (global_label "A14" (shape input) (at 205.232 122.936 0) (fields_autoplaced)

Commit message: Checkpoint on controller circuit.
Parts:
- removed unit 5 of RN101
- removed unit 3 of U103
Connections:
- no-connect marks 18 -> 15
Changed lines of the file:
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@@
   (junction (at 31.369 188.468) (diameter 0) (color 0 0 0 0)
-  )
-  (junction (at 257.556 138.557) (diameter 0) (color 0 0 0 0)
   )
   (junction (at 20.32 183.388) (diameter 0) (color 0 0 0 0)
@@
   (no_connect (at 272.796 157.48))
   (no_connect (at 201.676 161.925))
-  (no_connect (at 179.197 154.559))
   (no_connect (at 272.796 138.557))
   (no_connect (at 29.845 113.792))
   (no_connect (at 98.552 170.434))
   (no_connect (at 201.676 154.305))
-  (no_connect (at 272.796 129.413))
-  (no_connect (at 179.197 162.179))
   (no_connect (at 29.845 141.732))
   (no_connect (at 149.479 94.615))
@@
   )
   (wire (pts (xy 100.965 70.358) (xy 100.965 65.405))
-    (stroke (width 0) (type default))
-  )
-  (wire (pts (xy 257.556 129.413) (xy 257.556 138.557))
     (stroke (width 0) (type default))
   )
@@
         (path "/d4d4c0fa-7a39-4b72-9fdb-c481b1e41ed4"
           (reference "Q101") (unit 1)
-        )
-      )
-    )
-  )
-  (symbol (lib_id "74xx:74LS05") (at 265.176 129.413 0) (unit 3)
-    (in_bom yes) (on_board yes) (dnp no)
-    (property "Reference" "U103" (at 265.684 126.365 0)
-      (effects (font (size 1.27 1.27)) (justify left))
-    )
-    (property "Value" "74ACT05" (at 271.78 131.318 0)
-      (effects (font (size 1.27 1.27)) (justify left))
-    )
-    (property "Footprint" "Package_DIP:DIP-14_W7.62mm_Socket" (at 265.176 129.413 0)
-      (effects (font (size 1.27 1.27)) hide)
-    )
-    (property "Datasheet" "https://www.ti.com/lit/ds/symlink/cd74act05.pdf" (at 265.176 129.413 0)
-      (effects (font (size 1.27 1.27)) hide)
-    )
-    (pin "1")
-    (pin "2")
-    (pin "3")
-    (pin "4")
-    (pin "5")
-    (pin "6")
-    (pin "8")
-    (pin "9")
-    (pin "10")
-    (pin "11")
-    (pin "12")
-    (pin "13")
-    (pin "14")
-    (pin "7")
-    (instances
-      (project "CoPicoVision"
-        (path "/d4d4c0fa-7a39-4b72-9fdb-c481b1e41ed4"
-          (reference "U103") (unit 3)
         )
       )
@@
         )
       )
-    )
-  )
-  (symbol (lib_id "Device:R_Network08_Split") (at 179.197 158.369 0) (unit 5)
-    (in_bom yes) (on_board yes) (dnp no) (fields_autoplaced)
-    (property "Reference" "RN101" (at 181.229 157.734 0)
-      (effects (font (size 1.27 1.27)) (justify left))
-    )
-    (property "Value" "3K3" (at 181.229 160.274 0)
-      (effects (font (size 1.27 1.27)) (justify left))
-    )
-    (property "Footprint" "Resistor_THT:R_Array_SIP9" (at 177.165 158.369 90)
-      (effects (font (size 1.27 1.27)) hide)
-    )
-    (property "Datasheet" "http://www.vishay.com/docs/31509/csc.pdf" (at 179.197 158.369 0)
-      (effects (font (size 1.27 1.27)) hide)
-    )
-    (pin "1")
-    (pin "2")
-    (pin "3")
-    (pin "4")
-    (pin "5")
-    (pin "6")
-    (pin "7")
-    (pin "8")
-    (pin "9")
-    (instances
-      (project "CoPicoVision"
-        (path "/d4d4c0fa-7a39-4b72-9fdb-c481b1e41ed4"
-          (reference "RN101") (unit 5)
-        )
-      )

Commit message: Final controller checkpoint.  Managed to sqeeeze it all onto the board.
Parts:
- removed unit 4 of U103
Changed lines of the file:
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@@
-    )
-  )
-  (symbol (lib_id "74xx:74LS05") (at 265.176 138.557 0) (unit 4)
-    (in_bom yes) (on_board yes) (dnp no)
-    (property "Reference" "U103" (at 265.684 135.509 0)
-      (effects (font (size 1.27 1.27)) (justify left))
-    )
-    (property "Value" "74ACT05" (at 271.78 140.462 0)
-      (effects (font (size 1.27 1.27)) (justify left))
-    )
-    (property "Footprint" "Package_DIP:DIP-14_W7.62mm_Socket" (at 265.176 138.557 0)
-      (effects (font (size 1.27 1.27)) hide)
-    )
-    (property "Datasheet" "https://www.ti.com/lit/ds/symlink/cd74act05.pdf" (at 265.176 138.557 0)
-      (effects (font (size 1.27 1.27)) hide)
-    )
-    (pin "1")
-    (pin "2")
-    (pin "3")
-    (pin "4")
-    (pin "5")
-    (pin "6")
-    (pin "8")
-    (pin "9")
-    (pin "10")
-    (pin "11")
-    (pin "12")
-    (pin "13")
-    (pin "14")
-    (pin "7")
-    (instances
-      (project "CoPicoVision"
-        (path "/d4d4c0fa-7a39-4b72-9fdb-c481b1e41ed4"
-          (reference "U103") (unit 4)
-        )
-      )
     )
   )
