File: design-files/CoPicoVision.kicad_sch (KiCad schematic)
At the start: 36 parts, among them J101 USB_C_Receptacle_PowerOnly_6P, J102 Conn_02x15_Odd_Even, Q101 MMFTP3334K-AQ, SW101 SW_Push, SW102 SW_Push, U101 Z80CPU, U102 DS1813, U103 74ACT05, U104 ICL7660A, U105 MAX16054, X101 3.579545MHZ

Commit message: Controller section is mostly SMT now.
Parts:
- C101, C103, C104: footprint Capacitor_THT:C_Disc_D3.8mm_W2.6mm_P2.50mm -> Capacitor_SMD:C_0805_2012Metric_Pad1.18x1.45mm_HandSolder
- U103: footprint Package_DIP:DIP-14_W7.62mm_Socket -> Package_SO:SOIC-14_3.9x8.7mm_P1.27mm
Changed lines of the file:
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@@
       (effects (font (size 1.27 1.27)) (justify left))
     )
-    (property "Footprint" "Capacitor_THT:C_Disc_D3.8mm_W2.6mm_P2.50mm" (at 20.32 185.928 0)
+    (property "Footprint" "Capacitor_SMD:C_0805_2012Metric_Pad1.18x1.45mm_HandSolder" (at 20.32 185.928 0)
       (effects (font (size 1.27 1.27)) hide)
     )
@@
       (effects (font (size 1.27 1.27)) (justify left))
     )
-    (property "Footprint" "Package_DIP:DIP-14_W7.62mm_Socket" (at 265.176 148.082 0)
+    (property "Footprint" "Package_SO:SOIC-14_3.9x8.7mm_P1.27mm" (at 265.176 148.082 0)
       (effects (font (size 1.27 1.27)) hide)
     )
@@
       (effects (font (size 1.27 1.27)) (justify left))
     )
-    (property "Footprint" "Package_DIP:DIP-14_W7.62mm_Socket" (at 137.541 174.752 0)
+    (property "Footprint" "Package_SO:SOIC-14_3.9x8.7mm_P1.27mm" (at 137.541 174.752 0)
       (effects (font (size 1.27 1.27)) hide)
     )
@@
       (effects (font (size 1.27 1.27)) (justify left))
     )
-    (property "Footprint" "Capacitor_THT:C_Disc_D3.8mm_W2.6mm_P2.50mm" (at 31.369 185.928 0)
+    (property "Footprint" "Capacitor_SMD:C_0805_2012Metric_Pad1.18x1.45mm_HandSolder" (at 31.369 185.928 0)
       (effects (font (size 1.27 1.27)) hide)
     )
@@
       (effects (font (size 1.27 1.27)) (justify left))
     )
-    (property "Footprint" "Capacitor_THT:C_Disc_D3.8mm_W2.6mm_P2.50mm" (at 42.545 185.928 0)
+    (property "Footprint" "Capacitor_SMD:C_0805_2012Metric_Pad1.18x1.45mm_HandSolder" (at 42.545 185.928 0)
       (effects (font (size 1.27 1.27)) hide)
     )
@@
       (effects (font (size 1.27 1.27)) (justify left))
     )
-    (property "Footprint" "Package_DIP:DIP-14_W7.62mm_Socket" (at 265.176 157.48 0)
-      (effects (font (size 1.27 1.27)) hide)
-    )
+    (property "Footprint" "Package_SO:SOIC-14_3.9x8.7mm_P1.27mm" (at 265.176 157.48 0)
+      (effects (font (size 1.27 1.27)) hide)
+    )

Commit message: A couple more SMT resistors on the main sheet.
Parts:
- R412: footprint Resistor_THT:R_Axial_DIN0207_L6.3mm_D2.5mm_P7.62mm_Horizontal -> Resistor_SMD:R_0805_2012Metric_Pad1.20x1.40mm_HandSolder
Changed lines of the file:
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@@
       (effects (font (size 1.27 1.27)) (justify right))
     )
-    (property "Footprint" "Resistor_THT:R_Axial_DIN0207_L6.3mm_D2.5mm_P7.62mm_Horizontal" (at 59.69 160.401 0)
+    (property "Footprint" "Resistor_SMD:R_0805_2012Metric_Pad1.20x1.40mm_HandSolder" (at 59.69 160.401 0)
       (effects (font (size 1.27 1.27)) hide)
     )
@@
       (effects (font (size 1.27 1.27)) (justify right))
     )
-    (property "Footprint" "Resistor_THT:R_Axial_DIN0207_L6.3mm_D2.5mm_P7.62mm_Horizontal" (at 234.315 58.166 0)
+    (property "Footprint" "Resistor_SMD:R_0805_2012Metric_Pad1.20x1.40mm_HandSolder" (at 234.315 58.166 0)
       (effects (font (size 1.27 1.27)) hide)
     )

Commit message: Put the AY-3-8910 on the board, clarify part numbers for the 74xx chips to ensure the correct SOIC footprints.
Parts:
- U103: value 74ACT05 -> MC74ACT05DR2G
Other:
- moved on the sheet: U103E, U103F
Changed lines of the file:
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@@
   (junction (at 180.975 135.636) (diameter 0) (color 0 0 0 0)
   )
-  (junction (at 257.556 157.48) (diameter 0) (color 0 0 0 0)
+  (junction (at 251.714 157.734) (diameter 0) (color 0 0 0 0)
   )
   (junction (at 129.667 80.518) (diameter 0) (color 0 0 0 0)
@@
   )
   (no_connect (at 183.896 58.42))
-  (no_connect (at 272.796 148.082))
+  (no_connect (at 266.954 148.336))
   (no_connect (at 183.896 63.5))
-  (no_connect (at 272.796 157.48))
+  (no_connect (at 266.954 157.734))
   (no_connect (at 29.845 113.792))
   (no_connect (at 98.552 170.434))
@@
     (stroke (width 0) (type default))
   )
-  (wire (pts (xy 257.556 148.082) (xy 257.556 157.48))
+  (wire (pts (xy 251.714 148.336) (xy 251.714 157.734))
     (stroke (width 0) (type default))
   )
@@
     )
   )
-  (symbol (lib_id "74xx:74LS05") (at 265.176 148.082 0) (unit 5)
+  (symbol (lib_id "74xx:74LS05") (at 259.334 148.336 0) (unit 5)
     (in_bom yes) (on_board yes) (dnp no)
-    (property "Reference" "U103" (at 266.446 144.907 0)
-      (effects (font (size 1.27 1.27)) (justify left))
-    )
-    (property "Value" "74ACT05" (at 271.78 149.987 0)
-      (effects (font (size 1.27 1.27)) (justify left))
-    )
-    (property "Footprint" "Package_SO:SOIC-14_3.9x8.7mm_P1.27mm" (at 265.176 148.082 0)
-      (effects (font (size 1.27 1.27)) hide)
-    )
-    (property "Datasheet" "https://www.ti.com/lit/ds/symlink/cd74act05.pdf" (at 265.176 148.082 0)
-      (effects (font (size 1.27 1.27)) hide)
-    )
-    (property "Mouser" "595-CD74ACT05EE4" (at 265.176 148.082 0)
+    (property "Reference" "U103" (at 260.604 145.161 0)
+      (effects (font (size 1.27 1.27)) (justify left))
+    )
+    (property "Value" "MC74ACT05DR2G" (at 261.874 150.495 0)
+      (effects (font (size 1.27 1.27)) (justify left))
+    )
+    (property "Footprint" "Package_SO:SOIC-14_3.9x8.7mm_P1.27mm" (at 259.334 148.336 0)
+      (effects (font (size 1.27 1.27)) hide)
+    )
+    (property "Datasheet" "https://www.ti.com/lit/ds/symlink/cd74act05.pdf" (at 259.334 148.336 0)
+      (effects (font (size 1.27 1.27)) hide)
+    )
+    (property "Mouser" "595-CD74ACT05EE4" (at 259.334 148.336 0)
       (effects (font (size 1.27 1.27)) hide)
     )
@@
       (effects (font (size 1.27 1.27)) (justify left))
     )
-    (property "Value" "74ACT05" (at 144.145 176.657 0)
+    (property "Value" "MC74ACT05DR2G" (at 144.145 176.657 0)
       (effects (font (size 1.27 1.27)) (justify left))
     )
@@
     )
   )
-  (symbol (lib_id "power:GND") (at 257.556 157.48 0) (unit 1)
-    (in_bom yes) (on_board yes) (dnp no) (fields_autoplaced)
-    (property "Reference" "#PWR0113" (at 257.556 163.83 0)
-      (effects (font (size 1.27 1.27)) hide)
-    )
-    (property "Value" "GND" (at 257.556 163.068 0)
-      (effects (font (size 1.27 1.27)))
-    )
-    (property "Footprint" "" (at 257.556 157.48 0)
-      (effects (font (size 1.27 1.27)) hide)
-    )
-    (property "Datasheet" "" (at 257.556 157.48 0)
+  (symbol (lib_id "power:GND") (at 251.714 157.734 0) (unit 1)
+    (in_bom yes) (on_board yes) (dnp no) (fields_autoplaced)
+    (property "Reference" "#PWR0113" (at 251.714 164.084 0)
+      (effects (font (size 1.27 1.27)) hide)
+    )
+    (property "Value" "GND" (at 251.714 163.322 0)
+      (effects (font (size 1.27 1.27)))
+    )
+    (property "Footprint" "" (at 251.714 157.734 0)
+      (effects (font (size 1.27 1.27)) hide)
+    )
+    (property "Datasheet" "" (at 251.714 157.734 0)
       (effects (font (size 1.27 1.27)) hide)
     )
@@
     )
   )
-  (symbol (lib_id "74xx:74LS05") (at 265.176 157.48 0) (unit 6)
+  (symbol (lib_id "74xx:74LS05") (at 259.334 157.734 0) (unit 6)
     (in_bom yes) (on_board yes) (dnp no)
-    (property "Reference" "U103" (at 266.065 154.432 0)
-      (effects (font (size 1.27 1.27)) (justify left))
-    )
-    (property "Value" "74ACT05" (at 271.78 159.385 0)
-      (effects (font (size 1.27 1.27)) (justify left))
-    )
-    (property "Footprint" "Package_SO:SOIC-14_3.9x8.7mm_P1.27mm" (at 265.176 157.48 0)
-      (effects (font (size 1.27 1.27)) hide)
-    )
-    (property "Datasheet" "https://www.ti.com/lit/ds/symlink/cd74act05.pdf" (at 265.176 157.48 0)
-      (effects (font (size 1.27 1.27)) hide)
-    )
-    (property "Mouser" "595-CD74ACT05EE4" (at 265.176 157.48 0)
-      (effects (font (size 1.27 1.27)) hide)
-    )
+    (property "Reference" "U103" (at 260.223 154.686 0)
+      (effects (font (size 1.27 1.27)) (justify left))
+    )
+    (property "Value" "MC74ACT05DR2G" (at 260.858 160.401 0)
+      (effects (font (size 1.27 1.27)) (justify left))
+    )
+    (property "Footprint" "Package_SO:SOIC-14_3.9x8.7mm_P1.27mm" (at 259.334 157.734 0)
+      (effects (font (size 1.27 1.27)) hide)
+    )
+    (property "Datasheet" "https://www.ti.com/lit/ds/symlink/cd74act05.pdf" (at 259.334 157.734 0)
+      (effects (font (size 1.27 1.27)) hide)
+    )
+    (property "Mouser" "595-CD74ACT05EE4" (at 259.334 157.734 0)
+      (effects (font (size 1.27 1.27)) hide)
+    )

Commit message: Fix a dumb mistake in the power supply (put the reservoir cap on VCC, not VBUS), and fix a bunch of unconnected items.
Connections:
- net VBUS: no longer C105.1
- net VCC: now also C105.1
Other:
- moved on the sheet: C105
Changed lines of the file:
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@@
   (junction (at 20.32 188.468) (diameter 0) (color 0 0 0 0)
   )
+  (junction (at 172.847 60.325) (diameter 0) (color 0 0 0 0)
+  )
   (junction (at 131.699 107.315) (diameter 0) (color 0 0 0 0)
   )
@@
   (junction (at 103.505 80.518) (diameter 0) (color 0 0 0 0)
   )
-  (junction (at 137.795 50.165) (diameter 0) (color 0 0 0 0)
-  )
   (junction (at 77.724 138.303) (diameter 0) (color 0 0 0 0)
   )
@@
   )
   (junction (at 251.714 157.734) (diameter 0) (color 0 0 0 0)
-  )
-  (junction (at 129.667 80.518) (diameter 0) (color 0 0 0 0)
   )
   (junction (at 214.376 50.8) (diameter 0) (color 0 0 0 0)
@@
     (stroke (width 0) (type default))
   )
-  (wire (pts (xy 137.795 55.245) (xy 137.795 80.518))
-    (stroke (width 0) (type default))
-  )
   (wire (pts (xy 149.479 98.425) (xy 152.019 98.425))
     (stroke (width 0) (type default))
@@
     (stroke (width 0) (type default))
   )
-  (wire (pts (xy 137.795 50.165) (xy 100.965 50.165))
-    (stroke (width 0) (type default))
-  )
   (wire (pts (xy 121.539 107.315) (xy 131.699 107.315))
     (stroke (width 0) (type default))
@@
     (stroke (width 0) (type default))
   )
-  (wire (pts (xy 137.795 50.165) (xy 140.589 50.165))
+  (wire (pts (xy 100.965 50.165) (xy 140.589 50.165))
     (stroke (width 0) (type default))
   )
@@
     (stroke (width 0) (type default))
   )
+  (wire (pts (xy 172.847 60.325) (xy 179.578 60.325))
+    (stroke (width 0) (type default))
+  )
   (wire (pts (xy 129.667 62.865) (xy 129.667 73.279))
     (stroke (width 0) (type default))
@@
     (stroke (width 0) (type default))
   )
-  (wire (pts (xy 137.795 80.518) (xy 129.667 80.518))
-    (stroke (width 0) (type default))
-  )
   (wire (pts (xy 59.69 156.718) (xy 59.69 157.861))
     (stroke (width 0) (type default))
@@
     (stroke (width 0) (type default))
   )
-  (wire (pts (xy 159.639 60.325) (xy 179.578 60.325))
+  (wire (pts (xy 159.639 60.325) (xy 172.847 60.325))
     (stroke (width 0) (type default))
   )
@@
     )
   )
+  (symbol (lib_id "power:GND") (at 172.847 65.405 0) (unit 1)
+    (in_bom yes) (on_board yes) (dnp no) (fields_autoplaced)
+    (property "Reference" "#PWR0124" (at 172.847 71.755 0)
+      (effects (font (size 1.27 1.27)) hide)
+    )
+    (property "Value" "GND" (at 172.847 69.977 0)
+      (effects (font (size 1.27 1.27)))
+    )
+    (property "Footprint" "" (at 172.847 65.405 0)
+      (effects (font (size 1.27 1.27)) hide)
+    )
+    (property "Datasheet" "" (at 172.847 65.405 0)
+      (effects (font (size 1.27 1.27)) hide)
+    )
+    (pin "1")
+    (instances
+      (project "CoPicoVision"
+        (path "/d4d4c0fa-7a39-4b72-9fdb-c481b1e41ed4"
+          (reference "#PWR0124") (unit 1)
+        )
+      )
+    )
+  )
   (symbol (lib_id "Regulator_SwitchedCapacitor:ICL7660") (at 194.056 58.42 0) (unit 1)
     (in_bom yes) (on_board yes) (dnp no) (fields_autoplaced)
@@
     )
   )
-  (symbol (lib_id "Device:C_Polarized_Small") (at 137.795 52.705 0) (unit 1)
-    (in_bom yes) (on_board yes) (dnp no) (fields_autoplaced)
-    (property "Reference" "C105" (at 141.097 51.5239 0)
-      (effects (font (size 1.27 1.27)) (justify left))
-    )
-    (property "Value" "100µF" (at 141.097 54.0639 0)
-      (effects (font (size 1.27 1.27)) (justify left))
-    )
-    (property "Footprint" "Capacitor_THT:CP_Radial_D6.3mm_P2.50mm" (at 137.795 52.705 0)
-      (effects (font (size 1.27 1.27)) hide)
-    )
-    (property "Datasheet" "~" (at 137.795 52.705 0)
-      (effects (font (size 1.27 1.27)) hide)
-    )
-    (property "Mouser" "710-860040373002" (at 137.795 52.705 0)
-      (effects (font (size 1.27 1.27)) hide)
-    )
+  (symbol (lib_id "Device:C_Polarized_Small") (at 172.847 62.865 0) (unit 1)
+    (in_bom yes) (on_board yes) (dnp no)
+    (property "Reference" "C105" (at 174.879 61.722 0)
+      (effects (font (size 1.27 1.27)) (justify left))
+    )
+    (property "Value" "100µF" (at 174.879 64.262 0)
+      (effects (font (size 1.27 1.27)) (justify left))
+    )
+    (property "Footprint" "Capacitor_THT:CP_Radial_D6.3mm_P2.50mm" (at 172.847 62.865 0)
+      (effects (font (size 1.27 1.27)) hide)
+    )
+    (property "Datasheet" "~" (at 172.847 62.865 0)
+      (effects (font (size 1.27 1.27)) hide)
+    )
+    (property "Mouser" "710-860040373002" (at 172.847 62.865 0)
+      (effects (font (size 1.27 1.27)) hide)
+    )

Commit message: Update Mouser part numbers / data sheet links.
Parts:
- U103: value MC74ACT05DR2G -> MC74ACT05D; Mouser 595-CD74ACT05EE4 -> 863-MC74ACT05DR2G
Changed lines of the file:
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@@
       (effects (font (size 1.27 1.27)) (justify left))
     )
-    (property "Value" "MC74ACT05DR2G" (at 261.874 150.495 0)
+    (property "Value" "MC74ACT05D" (at 261.874 150.495 0)
       (effects (font (size 1.27 1.27)) (justify left))
     )
@@
       (effects (font (size 1.27 1.27)) hide)
     )
-    (property "Datasheet" "https://www.ti.com/lit/ds/symlink/cd74act05.pdf" (at 259.334 148.336 0)
-      (effects (font (size 1.27 1.27)) hide)
-    )
-    (property "Mouser" "595-CD74ACT05EE4" (at 259.334 148.336 0)
+    (property "Datasheet" "https://www.mouser.com/datasheet/2/308/1/MC74AC05_D-2315319.pdf" (at 259.334 148.336 0)
+      (effects (font (size 1.27 1.27)) hide)
+    )
+    (property "Mouser" "863-MC74ACT05DR2G" (at 259.334 148.336 0)
       (effects (font (size 1.27 1.27)) hide)
     )
@@
   (symbol (lib_id "74xx:74LS05") (at 137.541 174.752 0) (unit 7)
     (in_bom yes) (on_board yes) (dnp no) (fields_autoplaced)
-    (property "Reference" "U103" (at 144.145 174.117 0)
-      (effects (font (size 1.27 1.27)) (justify left))
-    )
-    (property "Value" "MC74ACT05DR2G" (at 144.145 176.657 0)
+    (property "Reference" "U103" (at 143.51 174.117 0)
+      (effects (font (size 1.27 1.27)) (justify left))
+    )
+    (property "Value" "MC74ACT05D" (at 143.51 176.657 0)
       (effects (font (size 1.27 1.27)) (justify left))
     )
@@
       (effects (font (size 1.27 1.27)) hide)
     )
-    (property "Datasheet" "https://www.ti.com/lit/ds/symlink/cd74act05.pdf" (at 137.541 174.752 0)
-      (effects (font (size 1.27 1.27)) hide)
-    )
-    (property "Mouser" "595-CD74ACT05EE4" (at 137.541 174.752 0)
+    (property "Datasheet" "https://www.mouser.com/datasheet/2/308/1/MC74AC05_D-2315319.pdf" (at 137.541 174.752 0)
+      (effects (font (size 1.27 1.27)) hide)
+    )
+    (property "Mouser" "863-MC74ACT05DR2G" (at 137.541 174.752 0)
       (effects (font (size 1.27 1.27)) hide)
     )
@@
       (effects (font (size 1.27 1.27)) (justify left))
     )
-    (property "Value" "MC74ACT05DR2G" (at 260.858 160.401 0)
+    (property "Value" "MC74ACT05D" (at 260.858 160.401 0)
       (effects (font (size 1.27 1.27)) (justify left))
     )
@@
       (effects (font (size 1.27 1.27)) hide)
     )
-    (property "Datasheet" "https://www.ti.com/lit/ds/symlink/cd74act05.pdf" (at 259.334 157.734 0)
-      (effects (font (size 1.27 1.27)) hide)
-    )
-    (property "Mouser" "595-CD74ACT05EE4" (at 259.334 157.734 0)
-      (effects (font (size 1.27 1.27)) hide)
-    )
+    (property "Datasheet" "https://www.mouser.com/datasheet/2/308/1/MC74AC05_D-2315319.pdf" (at 259.334 157.734 0)
+      (effects (font (size 1.27 1.27)) hide)
+    )
+    (property "Mouser" "863-MC74ACT05DR2G" (at 259.334 157.734 0)
+      (effects (font (size 1.27 1.27)) hide)
+    )

Commit message: Add / correct a bunch of Mouser part numbers for the BoM.
Parts:
- C101, C103, C104: Mouser 81-RCER71E104K0A2H3B -> 581-KAM21BR71H104JT
- C106, C107: Mouser (none) -> 80-C0805C106J8RAUTLR
- R101, R102: Mouser (none) -> 71-CRCW0805-5.1K-E3
- R103: Mouser (none) -> 71-CRCW0805-10K-E3
- R412: Mouser (none) -> 71-CRCW0805-3.3K-E3
- R412: Mouser (none) -> 71-CRCW0805-330-E3
Changed lines of the file:
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@@
+      (effects (font (size 1.27 1.27)) hide)
+    )
+    (property "Mouser" "80-C0805C106J8RAUTLR" (at 205.486 60.452 0)
       (effects (font (size 1.27 1.27)) hide)
     )
@@
     )
     (property "Datasheet" "~" (at 59.69 160.401 0)
+      (effects (font (size 1.27 1.27)) hide)
+    )
+    (property "Mouser" "71-CRCW0805-3.3K-E3" (at 59.69 160.401 0)
       (effects (font (size 1.27 1.27)) hide)
     )
@@
       (effects (font (size 1.27 1.27)) hide)
     )
+    (property "Mouser" "71-CRCW0805-10K-E3" (at 148.717 52.705 0)
+      (effects (font (size 1.27 1.27)) hide)
+    )
     (pin "1")
     (pin "2")
@@
     )
     (property "Datasheet" "~" (at 234.315 58.166 0)
+      (effects (font (size 1.27 1.27)) hide)
+    )
+    (property "Mouser" "71-CRCW0805-330-E3" (at 234.315 58.166 0)
       (effects (font (size 1.27 1.27)) hide)
     )
@@
       (effects (font (size 1.27 1.27)) hide)
     )
+    (property "Mouser" "71-CRCW0805-5.1K-E3" (at 121.031 75.819 0)
+      (effects (font (size 1.27 1.27)) hide)
+    )
     (pin "1")
     (pin "2")
@@
       (effects (font (size 1.27 1.27)) hide)
     )
-    (property "Mouser" "81-RCER71E104K0A2H3B" (at 20.32 185.928 0)
+    (property "Mouser" "581-KAM21BR71H104JT" (at 20.32 185.928 0)
       (effects (font (size 1.27 1.27)) hide)
     )
@@
     )
     (property "Datasheet" "~" (at 129.667 75.819 0)
+      (effects (font (size 1.27 1.27)) hide)
+    )
+    (property "Mouser" "71-CRCW0805-5.1K-E3" (at 129.667 75.819 0)
       (effects (font (size 1.27 1.27)) hide)
     )
@@
       (effects (font (size 1.27 1.27)) hide)
     )
+    (property "Mouser" "80-C0805C106J8RAUTLR" (at 214.376 53.34 0)
+      (effects (font (size 1.27 1.27)) hide)
+    )
     (pin "1")
     (pin "2")
@@
       (effects (font (size 1.27 1.27)) hide)
     )
-    (property "Mouser" "81-RCER71E104K0A2H3B" (at 31.369 185.928 0)
+    (property "Mouser" "581-KAM21BR71H104JT" (at 31.369 185.928 0)
       (effects (font (size 1.27 1.27)) hide)
     )
@@
       (effects (font (size 1.27 1.27)) hide)
     )
-    (property "Mouser" "81-RCER71E104K0A2H3B" (at 42.545 185.928 0)
-      (effects (font (size 1.27 1.27)) hide)
-    )
+    (property "Mouser" "581-KAM21BR71H104JT" (at 42.545 185.928 0)
+      (effects (font (size 1.27 1.27)) hide)
+    )
