File: design-files/CoPicoVision.kicad_pcb (KiCad board)
At the start: 2 copper layers, 33 parts, among them J301 DE15_Receptacle_HighDensity_M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, SW101 SW_Push, U101 Z80CPU, U102 DS1813, U103 74ACT05, U201 GAL22V10, U202 GAL22V10, U203 AT28C64, U204 AS6C6264, U301 Pico, U302 74LVC245, U303 74LVC245, X101 3.579545MHZ

Commit message: Add controller ports just to get them onto the board.
Parts:
- added J401: DE9_Plug_MountingHoles, Connector_Dsub:DSUB-9_Male_Horizontal_P2.77x2.84mm_EdgePinOffset7.70mm_Housed_MountingHolesOffset9.12mm, F.Cu at (91.7, 130.8)
- added J402: DE9_Plug_MountingHoles, Connector_Dsub:DSUB-9_Male_Horizontal_P2.77x2.84mm_EdgePinOffset7.70mm_Housed_MountingHolesOffset9.12mm, F.Cu at (145.3, 130.8)
- moved D101 42.7 mm to (120.7, 80.0), turned to -90 degrees
- moved C102 33.2 mm to (126.0, 84.2)
- moved U102 33.2 mm to (132.6, 84.3)
- moved D301 15.0 mm to (183.4, 42.4)
- moved J301 15.0 mm to (135.4, 50.4)
- moved RN306 15.0 mm to (151.6, 72.4)
- moved U302 15.0 mm to (183.4, 50.3)
- moved RN301 15.0 mm to (125.5, 54.9)
- moved RN302 15.0 mm to (125.5, 58.4)
- moved RN303 15.0 mm to (125.5, 62.0)
- moved RN304 15.0 mm to (125.5, 65.5)
- moved C301 15.0 mm to (191.0, 47.0)
- moved C302 15.0 mm to (201.9, 47.0)
- moved RN305 15.0 mm to (148.1, 72.4)
- moved RN307 15.0 mm to (155.2, 72.4)
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Other:
- board outline added: 165.9 x 110 mm

Commit message: Lay out some additional bits.
Parts:
- added C501: 0.1µF, Capacitor_THT:C_Disc_D3.8mm_W2.6mm_P2.50mm, F.Cu at (113.6, 41.4)
- added C502: 10µF, Capacitor_THT:CP_Radial_D6.3mm_P2.50mm, F.Cu at (118.6, 46.0)
- added C503: 470µF, Capacitor_THT:CP_Radial_D6.3mm_P2.50mm, F.Cu at (97.8, 56.6)
- added J501: AudioJack3, Connector_Audio:Jack_3.5mm_CUI_SJ1-3523N_Horizontal, F.Cu at (97.7, 42.4)
- added Q501: KSD1616A, Package_TO_SOT_THT:TO-92L_Inline_Wide, F.Cu at (95.2, 63.2)
- added R501: 100R, Resistor_THT:R_Axial_DIN0204_L3.6mm_D1.6mm_P5.08mm_Horizontal, F.Cu at (91.7, 59.9)
- added U501: SN76489AN, Package_DIP:DIP-16_W7.62mm_Socket, F.Cu at (105.9, 44.7)
- moved U102 12.5 mm to (140.7, 74.8)
- moved D101 12.5 mm to (128.8, 70.5)
- moved C102 12.5 mm to (134.1, 74.7)

Commit message: Add power supply.  PCB checkpoint.
Parts:
- added C105: 100µF, Capacitor_THT:CP_Radial_D6.3mm_P2.50mm, F.Cu at (65.4, 43.2)
- added C106: 10µF, Capacitor_SMD:C_0805_2012Metric_Pad1.18x1.45mm_HandSolder, F.Cu at (61.5, 51.8)
- added C107: 10µF, Capacitor_SMD:C_0805_2012Metric_Pad1.18x1.45mm_HandSolder, F.Cu at (71.1, 51.8)
- added D102: ESDA25L, Package_TO_SOT_SMD:SOT-23, F.Cu at (57.7, 48.4)
- added H101: MountingHole, MountingHole:MountingHole_3.5mm, F.Cu at (47.5, 44.2)
- added H102: MountingHole, MountingHole:MountingHole_3.5mm, F.Cu at (47.5, 141.5)
- added H103: MountingHole, MountingHole:MountingHole_3.5mm, F.Cu at (200.7, 44.2)
- added H104: MountingHole, MountingHole:MountingHole_3.5mm, F.Cu at (200.7, 141.5)
- added J101: USB_C_Receptacle_PowerOnly_6P, Connector_USB:USB_C_Receptacle_GCT_USB4085, F.Cu at (60.4, 43.9)
- added Q101: MMFTP3334K-AQ, Package_TO_SOT_SMD:SOT-23, F.Cu at (72.1, 42.7)
- added R101: 5K1, Resistor_SMD:R_0805_2012Metric_Pad1.20x1.40mm_HandSolder, F.Cu at (54.9, 48.5)
- added R102: 5K1, Resistor_SMD:R_0805_2012Metric_Pad1.20x1.40mm_HandSolder, F.Cu at (57.7, 51.6)
- added R103: 10K, Resistor_SMD:R_0805_2012Metric_Pad1.20x1.40mm_HandSolder, F.Cu at (72.1, 39.6)
- added SW102: SW_Push, Button_Switch_THT:SW_PUSH_6mm, F.Cu at (56.9, 139.2)
- added U104: ICL7660A, Package_SO:SOIC-8_3.9x4.9mm_P1.27mm, F.Cu at (66.3, 51.1)
- added U105: MAX16054, Package_TO_SOT_SMD:SOT-23-6, F.Cu at (72.1, 48.0)
- moved C302 6.10 mm to (201.9, 53.1)
- moved U303 6.10 mm to (194.3, 56.4)
- moved SW101 0.35 mm to (184.7, 139.2)

Commit message: Another PCB checkpoint.
Parts:
- moved C202 64.4 mm to (45.5, 96.2), turned to 90 degrees
- moved C102 61.1 mm to (193.8, 87.8)
- moved D101 61.1 mm to (188.5, 83.6)
- moved U102 61.1 mm to (200.4, 87.9)
- moved U202 56.5 mm to (48.8, 103.9), turned to 90 degrees
- moved C203 13.7 mm to (45.5, 77.7)
- moved U203 13.7 mm to (48.8, 93.0)
- moved U204 13.7 mm to (48.8, 74.4)
- moved C204 13.7 mm to (45.5, 59.2)
- moved RN101 13.7 mm to (48.8, 55.9)
- moved C103 12.5 mm to (101.8, 96.3)
- moved X101 12.5 mm to (101.9, 108.5)
- moved C503 11.8 mm to (87.6, 50.5)
- moved C104 11.0 mm to (105.2, 71.1)
- moved U103 11.0 mm to (97.5, 74.4)
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Other:
- board text added: "Controller 1"
- board text added: "Controller 2"
- board text added: "IODEC"
- board text added: "MEMDEC"
- board text added: "Power"
- board text added: "Reset"

Commit message: Another PCB checkpoint.
Parts:
- moved X101 16.9 mm to (86.6, 101.1)
- moved U103 16.8 mm to (86.6, 61.7)
- moved C103 16.7 mm to (86.6, 89.4), turned to 90 degrees
- moved C201 15.9 mm to (110.0, 68.9), turned to -90 degrees
- moved U201 13.6 mm to (99.1, 68.8)
- moved C104 12.1 mm to (97.5, 61.7), turned to -90 degrees
- moved J401 9.22 mm to (82.4, 130.8)
- moved J402 8.85 mm to (154.2, 130.8)
Changed lines of the file:
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@@
   )
   (footprint "Package_DIP:DIP-14_W7.62mm_Socket" (layer "F.Cu")
-    (at 97.536 74.422)
+    (at 86.614 61.717)
     (descr "14-lead though-hole mounted DIP package, row spacing 7.62 mm (300 mils), Socket")
     (tags "THT DIP DIL PDIP 2.54mm 7.62mm 300mil Socket")
@@
   )
   (footprint "Capacitor_THT:C_Disc_D3.8mm_W2.6mm_P2.50mm" (layer "F.Cu")
-    (at 94.274 71.12)
+    (at 109.982 68.854 -90)
     (descr "C, Disc series, Radial, pin pitch=2.50mm, , diameter*width=3.8*2.6mm^2, Capacitor, http://www.vishay.com/docs/45233/krseries.pdf")
     (tags "C Disc series Radial pin pitch 2.50mm  diameter 3.8mm width 2.6mm Capacitor")
@@
     (property "ki_keywords" "capacitor cap")
     (attr through_hole)
-    (fp_text reference "C201" (at 1.25 -2.55) (layer "F.SilkS")
+    (fp_text reference "C201" (at 1.25 -2.55 90) (layer "F.SilkS")
         (effects (font (size 1 1) (thickness 0.15)))
     )
-    (fp_text value "0.1µF" (at 1.25 2.55) (layer "F.Fab")
+    (fp_text value "0.1µF" (at 1.25 2.55 90) (layer "F.Fab")
         (effects (font (size 1 1) (thickness 0.15)))
     )
-    (fp_text user "${REFERENCE}" (at 1.25 0) (layer "F.Fab")
+    (fp_text user "${REFERENCE}" (at 1.25 0 90) (layer "F.Fab")
         (effects (font (size 0.76 0.76) (thickness 0.114)))
     )
@@
     (fp_line (start 3.15 1.3) (end 3.15 -1.3)
       (stroke (width 0.1) (type solid)) (layer "F.Fab"))
-    (pad "1" thru_hole circle (at 0 0) (size 1.6 1.6) (drill 0.8) (layers "*.Cu" "*.Mask")
+    (pad "1" thru_hole circle (at 0 0 270) (size 1.6 1.6) (drill 0.8) (layers "*.Cu" "*.Mask")
       (net 1 "VCC") (pintype "passive"))
-    (pad "2" thru_hole circle (at 2.5 0) (size 1.6 1.6) (drill 0.8) (layers "*.Cu" "*.Mask")
+    (pad "2" thru_hole circle (at 2.5 0 270) (size 1.6 1.6) (drill 0.8) (layers "*.Cu" "*.Mask")
       (net 2 "GND") (pintype "passive"))
     (model "${KICAD6_3DMODEL_DIR}/Capacitor_THT.3dshapes/C_Disc_D3.8mm_W2.6mm_P2.50mm.wrl"
@@
   )
   (footprint "Package_DIP:DIP-24_W7.62mm_Socket" (layer "F.Cu")
-    (at 86.614 74.422)
+    (at 99.06 68.834)
     (descr "24-lead though-hole mounted DIP package, row spacing 7.62 mm (300 mils), Socket")
     (tags "THT DIP DIL PDIP 2.54mm 7.62mm 300mil Socket")
@@
   )
   (footprint "Connector_Dsub:DSUB-9_Male_Horizontal_P2.77x2.84mm_EdgePinOffset7.70mm_Housed_MountingHolesOffset9.12mm" (layer "F.Cu")
-    (at 91.651 130.764)
+    (at 82.435 130.764)
     (descr "9-pin D-Sub connector, horizontal/angled (90 deg), THT-mount, male, pitch 2.77x2.84mm, pin-PCB-offset 7.699999999999999mm, distance of mounting holes 25mm, distance of mounting holes to PCB edge 9.12mm, see https://disti-assets.s3.amazonaws.com/tonar/files/datasheets/16730.pdf")
     (tags "9-pin D-Sub connector horizontal angled 90deg THT male pitch 2.77x2.84mm pin-PCB-offset 7.699999999999999mm mounting-holes-distance 25mm mounting-hole-offset 25mm")
@@
   )
   (footprint "Connector_Dsub:DSUB-9_Male_Horizontal_P2.77x2.84mm_EdgePinOffset7.70mm_Housed_MountingHolesOffset9.12mm" (layer "F.Cu")
-    (at 145.326 130.764)
+    (at 154.172 130.764)
     (descr "9-pin D-Sub connector, horizontal/angled (90 deg), THT-mount, male, pitch 2.77x2.84mm, pin-PCB-offset 7.699999999999999mm, distance of mounting holes 25mm, distance of mounting holes to PCB edge 9.12mm, see https://disti-assets.s3.amazonaws.com/tonar/files/datasheets/16730.pdf")
     (tags "9-pin D-Sub connector horizontal angled 90deg THT male pitch 2.77x2.84mm pin-PCB-offset 7.699999999999999mm mounting-holes-distance 25mm mounting-hole-offset 25mm")
@@
   )
   (footprint "Capacitor_THT:C_Disc_D3.8mm_W2.6mm_P2.50mm" (layer "F.Cu")
-    (at 101.834 96.266 180)
+    (at 86.614 89.388 90)
     (descr "C, Disc series, Radial, pin pitch=2.50mm, , diameter*width=3.8*2.6mm^2, Capacitor, http://www.vishay.com/docs/45233/krseries.pdf")
     (tags "C Disc series Radial pin pitch 2.50mm  diameter 3.8mm width 2.6mm Capacitor")
@@
     (property "ki_keywords" "capacitor cap")
     (attr through_hole)
-    (fp_text reference "C103" (at 1.25 -2.55) (layer "F.SilkS")
+    (fp_text reference "C103" (at 4.298 0 180) (layer "F.SilkS")
         (effects (font (size 1 1) (thickness 0.15)))
     )
-    (fp_text value "0.1µF" (at 1.25 2.55) (layer "F.Fab")
+    (fp_text value "0.1µF" (at 1.25 2.55 90) (layer "F.Fab")
         (effects (font (size 1 1) (thickness 0.15)))
     )
-    (fp_text user "${REFERENCE}" (at 1.25 0) (layer "F.Fab")
+    (fp_text user "${REFERENCE}" (at 1.25 0 90) (layer "F.Fab")
         (effects (font (size 0.76 0.76) (thickness 0.114)))
     )
@@
     (fp_line (start 3.15 1.3) (end 3.15 -1.3)
       (stroke (width 0.1) (type solid)) (layer "F.Fab"))
-    (pad "1" thru_hole circle (at 0 0 180) (size 1.6 1.6) (drill 0.8) (layers "*.Cu" "*.Mask")
+    (pad "1" thru_hole circle (at 0 0 90) (size 1.6 1.6) (drill 0.8) (layers "*.Cu" "*.Mask")
       (net 1 "VCC") (pintype "passive"))
-    (pad "2" thru_hole circle (at 2.5 0 180) (size 1.6 1.6) (drill 0.8) (layers "*.Cu" "*.Mask")
+    (pad "2" thru_hole circle (at 2.5 0 90) (size 1.6 1.6) (drill 0.8) (layers "*.Cu" "*.Mask")
       (net 2 "GND") (pintype "passive"))
     (model "${KICAD6_3DMODEL_DIR}/Capacitor_THT.3dshapes/C_Disc_D3.8mm_W2.6mm_P2.50mm.wrl"
@@
   )
   (footprint "Capacitor_THT:C_Disc_D3.8mm_W2.6mm_P2.50mm" (layer "F.Cu")
-    (at 105.176 71.12)
+    (at 97.536 61.737 -90)
     (descr "C, Disc series, Radial, pin pitch=2.50mm, , diameter*width=3.8*2.6mm^2, Capacitor, http://www.vishay.com/docs/45233/krseries.pdf")
     (tags "C Disc series Radial pin pitch 2.50mm  diameter 3.8mm width 2.6mm Capacitor")
@@
     (property "ki_keywords" "capacitor cap")
     (attr through_hole)
-    (fp_text reference "C104" (at 1.25 -2.55) (layer "F.SilkS")
+    (fp_text reference "C104" (at 1.25 -2.55 90) (layer "F.SilkS")
         (effects (font (size 1 1) (thickness 0.15)))
     )
-    (fp_text value "0.1µF" (at 1.25 2.55) (layer "F.Fab")
+    (fp_text value "0.1µF" (at 1.25 2.55 90) (layer "F.Fab")
         (effects (font (size 1 1) (thickness 0.15)))
     )
-    (fp_text user "${REFERENCE}" (at 1.25 0) (layer "F.Fab")
+    (fp_text user "${REFERENCE}" (at 1.25 0 90) (layer "F.Fab")
         (effects (font (size 0.76 0.76) (thickness 0.114)))
     )
@@
     (fp_line (start 3.15 1.3) (end 3.15 -1.3)
       (stroke (width 0.1) (type solid)) (layer "F.Fab"))
-    (pad "1" thru_hole circle (at 0 0) (size 1.6 1.6) (drill 0.8) (layers "*.Cu" "*.Mask")
+    (pad "1" thru_hole circle (at 0 0 270) (size 1.6 1.6) (drill 0.8) (layers "*.Cu" "*.Mask")
       (net 1 "VCC") (pintype "passive"))
-    (pad "2" thru_hole circle (at 2.5 0) (size 1.6 1.6) (drill 0.8) (layers "*.Cu" "*.Mask")
+    (pad "2" thru_hole circle (at 2.5 0 270) (size 1.6 1.6) (drill 0.8) (layers "*.Cu" "*.Mask")
       (net 2 "GND") (pintype "passive"))
     (model "${KICAD6_3DMODEL_DIR}/Capacitor_THT.3dshapes/C_Disc_D3.8mm_W2.6mm_P2.50mm.wrl"
@@
   )
   (footprint "Oscillator:Oscillator_DIP-8" (layer "F.Cu")
-    (at 101.854 108.458)
+    (at 86.614 101.092)
     (descr "Oscillator, DIP8,http://cdn-reichelt.de/documents/datenblatt/B400/OSZI.pdf")
     (tags "oscillator")
@@
   (gr_rect (start 41.148 37.846) (end 207.01 147.828)
     (stroke (width 0.1) (type default)) (fill none) (layer "Edge.Cuts"))
-  (gr_text "Controller 2" (at 167.64 145.288) (layer "F.SilkS")
+  (gr_text "Controller 2" (at 169.926 145.288) (layer "F.SilkS")
     (effects (font (size 1 1) (thickness 0.15) italic) (justify left bottom))
   )
@@
     (effects (font (size 1 1) (thickness 0.15) italic) (justify left bottom))
   )
-  (gr_text "Controller 1" (at 71.628 144.78) (layer "F.SilkS")
+  (gr_text "Controller 1" (at 68.834 144.78) (layer "F.SilkS")
     (effects (font (size 1 1) (thickness 0.15) italic) (justify left bottom))
   )
@@
     (effects (font (size 1 1) (thickness 0.15) italic) (justify left bottom))
   )
-  (gr_text "IODEC" (at 88.392 105.41) (layer "F.SilkS")
+  (gr_text "IODEC" (at 100.584 99.822) (layer "F.SilkS")
     (effects (font (size 1 1) (thickness 0.15) italic) (justify left bottom))
   )

Commit message: Getting closer with PCB layout.
Parts:
- moved RN302 34.4 mm to (157.2, 45.2), turned to -90 degrees
- moved RN303 32.1 mm to (157.2, 66.5), turned to -90 degrees
- moved RN301 28.3 mm to (153.7, 57.7), turned to 180 degrees
- moved RN304 28.2 mm to (153.7, 64.3), turned to 180 degrees
- moved RN305 18.9 mm to (153.7, 54.4), turned to 180 degrees
- moved RN306 11.6 mm to (153.7, 61.0), turned to 180 degrees
- moved RN307 5.06 mm to (153.7, 67.6), turned to 180 degrees
- moved C301 4.67 mm to (194.3, 50.3), turned to -90 degrees
- moved J401 1.17 mm to (82.4, 131.9)
- moved J101 1.15 mm to (61.5, 43.9)
- moved R101 1.15 mm to (56.0, 48.5)
- moved C105 1.15 mm to (66.5, 43.2)
- moved C106 1.15 mm to (62.6, 51.8)
- moved C107 1.15 mm to (72.3, 51.8)
- moved D102 1.15 mm to (58.8, 48.4)
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Connections:
- SW101 pad 2: Net-(U102-GND) -> GND
- U102 pad 3: Net-(U102-GND) -> GND
- U301 pad 13: Net-(U301-AGND) -> GND
- U301 pad 18: Net-(U301-AGND) -> GND
- U301 pad 23: Net-(U301-AGND) -> GND
- U301 pad 28: Net-(U301-AGND) -> GND
- U301 pad 3: Net-(U301-AGND) -> GND
- U301 pad 33: Net-(U301-AGND) -> GND
- U301 pad 38: Net-(U301-AGND) -> GND
- U301 pad 42: Net-(U301-AGND) -> GND
- U301 pad 8: Net-(U301-AGND) -> GND
