File: design-files/CoPicoVision.kicad_pcb (KiCad board)
At the start: 2 copper layers, 165.9 x 110 mm, 58 parts, among them J101 USB_C_Receptacle_PowerOnly_6P, J301 DE15_Receptacle_HighDensity_M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, J401 DE9_Plug_MountingHoles, J402 DE9_Plug_MountingHoles, J501 AudioJack3, Q101 MMFTP3334K-AQ, Q501 KSD1616A, SW101 SW_Push, SW102 SW_Push, U101 Z80CPU, U102 DS1813, U103 74ACT05, U104 ICL7660A, U105 MAX16054, U201 GAL22V10, U202 GAL22V10, U203 AT28C64, U204 AS6C6264, U301 Pico, U302 74LVC245, U303 74LVC245, U501 SN76489AN, X101 3.579545MHZ

Commit message: Add mounting holes around the cartridge area to reinforce it when carts are being inserted.
Parts:
- added H105: MountingHole, MountingHole:MountingHole_3.5mm, F.Cu at (118.9, 93.2)
- added H106: MountingHole, MountingHole:MountingHole_3.5mm, F.Cu at (118.9, 123.4)
- added H107: MountingHole, MountingHole:MountingHole_3.5mm, F.Cu at (200.4, 93.2)
- added H108: MountingHole, MountingHole:MountingHole_3.5mm, F.Cu at (200.4, 123.4)
- moved C102 9.51 mm to (187.2, 80.9), turned to 90 degrees
- moved U102 6.75 mm to (193.8, 86.5)
- moved D101 5.68 mm to (183.4, 86.1), turned to 0 degrees
Changed lines of the file:
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@@
   )
   (footprint "Diode_THT:D_DO-35_SOD27_P7.62mm_Horizontal" (layer "F.Cu")
-    (at 188.468 83.566 -90)
+    (at 183.388 86.106)
     (descr "Diode, DO-35_SOD27 series, Axial, Horizontal, pin pitch=7.62mm, , length*diameter=4*2mm^2, , http://www.diodes.com/_files/packages/DO-35.pdf")
     (tags "Diode DO-35_SOD27 series Axial Horizontal pin pitch 7.62mm  length 4mm diameter 2mm")
@@
     (property "ki_keywords" "diode")
     (attr through_hole)
-    (fp_text reference "D101" (at 3.81 -2.12 90) (layer "F.SilkS")
+    (fp_text reference "D101" (at 3.81 -2.12) (layer "F.SilkS")
         (effects (font (size 1 1) (thickness 0.15)))
     )
-    (fp_text value "1N4148" (at 3.81 2.12 90) (layer "F.SilkS")
+    (fp_text value "1N4148" (at 3.81 2.12) (layer "F.SilkS")
         (effects (font (size 1 1) (thickness 0.15)))
     )
-    (fp_text user "K" (at 0 -1.8 90) (layer "F.SilkS")
+    (fp_text user "K" (at 0 -1.8) (layer "F.SilkS")
         (effects (font (size 1 1) (thickness 0.15)))
     )
-    (fp_text user "K" (at 0 -1.8 90) (layer "F.Fab")
+    (fp_text user "K" (at 0 -1.8) (layer "F.Fab")
         (effects (font (size 1 1) (thickness 0.15)))
     )
-    (fp_text user "${REFERENCE}" (at 4.11 -14.986 90) (layer "F.Fab")
+    (fp_text user "${REFERENCE}" (at 4.11 0) (layer "F.Fab")
         (effects (font (size 0.8 0.8) (thickness 0.12)))
     )
@@
     (fp_line (start 7.62 0) (end 5.81 0)
       (stroke (width 0.1) (type solid)) (layer "F.Fab"))
-    (pad "1" thru_hole rect (at 0 0 270) (size 1.6 1.6) (drill 0.8) (layers "*.Cu" "*.Mask")
+    (pad "1" thru_hole rect (at 0 0) (size 1.6 1.6) (drill 0.8) (layers "*.Cu" "*.Mask")
       (net 1 "VCC") (pinfunction "K") (pintype "passive"))
-    (pad "2" thru_hole oval (at 7.62 0 270) (size 1.6 1.6) (drill 0.8) (layers "*.Cu" "*.Mask")
+    (pad "2" thru_hole oval (at 7.62 0) (size 1.6 1.6) (drill 0.8) (layers "*.Cu" "*.Mask")
       (net 3 "Net-(D101-A)") (pinfunction "A") (pintype "passive"))
     (model "${KICAD6_3DMODEL_DIR}/Diode_THT.3dshapes/D_DO-35_SOD27_P7.62mm_Horizontal.wrl"
@@
     )
   )
+  (footprint "MountingHole:MountingHole_3.5mm" (layer "F.Cu")
+    (at 200.406 123.444)
+    (descr "Mounting Hole 3.5mm, no annular")
+    (tags "mounting hole 3.5mm no annular")
+    (property "Sheetfile" "CoPicoVision.kicad_sch")
+    (property "Sheetname" "")
+    (property "ki_description" "Mounting Hole without connection")
+    (property "ki_keywords" "mounting hole")
+    (attr exclude_from_pos_files)
+    (fp_text reference "H108" (at 0 -4.5) (layer "F.SilkS") hide
+        (effects (font (size 1 1) (thickness 0.15)))
+    )
+    (fp_text value "MountingHole" (at 0 4.5) (layer "F.Fab")
+        (effects (font (size 1 1) (thickness 0.15)))
+    )
+    (fp_text user "${REFERENCE}" (at 0 0) (layer "F.Fab")
+        (effects (font (size 1 1) (thickness 0.15)))
+    )
+    (fp_circle (center 0 0) (end 3.5 0)
+      (stroke (width 0.15) (type solid)) (fill none) (layer "Cmts.User"))
+    (fp_circle (center 0 0) (end 3.75 0)
+      (stroke (width 0.05) (type solid)) (fill none) (layer "F.CrtYd"))
+    (pad "" np_thru_hole circle (at 0 0) (size 3.5 3.5) (drill 3.5) (layers "*.Cu" "*.Mask"))
+  )
   (footprint "Resistor_THT:R_Array_SIP8" (layer "F.Cu")
     (at 153.67 57.658 180)
@@
   )
   (footprint "Package_TO_SOT_THT:TO-92_Inline" (layer "F.Cu")
-    (at 200.406 87.884)
+    (at 193.802 86.466)
     (descr "TO-92 leads in-line, narrow, oval pads, drill 0.75mm (see NXP sot054_po.pdf)")
     (tags "to-92 sc-43 sc-43a sot54 PA33 transistor")
@@
     )
   )
+  (footprint "MountingHole:MountingHole_3.5mm" (layer "F.Cu")
+    (at 118.872 123.444)
+    (descr "Mounting Hole 3.5mm, no annular")
+    (tags "mounting hole 3.5mm no annular")
+    (property "Sheetfile" "CoPicoVision.kicad_sch")
+    (property "Sheetname" "")
+    (property "ki_description" "Mounting Hole without connection")
+    (property "ki_keywords" "mounting hole")
+    (attr exclude_from_pos_files)
+    (fp_text reference "H106" (at 0 -4.5) (layer "F.SilkS") hide
+        (effects (font (size 1 1) (thickness 0.15)))
+    )
+    (fp_text value "MountingHole" (at 0 4.5) (layer "F.Fab")
+        (effects (font (size 1 1) (thickness 0.15)))
+    )
+    (fp_text user "${REFERENCE}" (at 0 0) (layer "F.Fab")
+        (effects (font (size 1 1) (thickness 0.15)))
+    )
+    (fp_circle (center 0 0) (end 3.5 0)
+      (stroke (width 0.15) (type solid)) (fill none) (layer "Cmts.User"))
+    (fp_circle (center 0 0) (end 3.75 0)
+      (stroke (width 0.05) (type solid)) (fill none) (layer "F.CrtYd"))
+    (pad "" np_thru_hole circle (at 0 0) (size 3.5 3.5) (drill 3.5) (layers "*.Cu" "*.Mask"))
+  )
+  (footprint "MountingHole:MountingHole_3.5mm" (layer "F.Cu")
+    (at 200.406 93.218)
+    (descr "Mounting Hole 3.5mm, no annular")
+    (tags "mounting hole 3.5mm no annular")
+    (property "Sheetfile" "CoPicoVision.kicad_sch")
+    (property "Sheetname" "")
+    (property "ki_description" "Mounting Hole without connection")
+    (property "ki_keywords" "mounting hole")
+    (attr exclude_from_pos_files)
+    (fp_text reference "H107" (at 0 -4.5) (layer "F.SilkS") hide
+        (effects (font (size 1 1) (thickness 0.15)))
+    )
+    (fp_text value "MountingHole" (at 0 4.5) (layer "F.Fab")
+        (effects (font (size 1 1) (thickness 0.15)))
+    )
+    (fp_text user "${REFERENCE}" (at 0 0) (layer "F.Fab")
+        (effects (font (size 1 1) (thickness 0.15)))
+    )
+    (fp_circle (center 0 0) (end 3.5 0)
+      (stroke (width 0.15) (type solid)) (fill none) (layer "Cmts.User"))
+    (fp_circle (center 0 0) (end 3.75 0)
+      (stroke (width 0.05) (type solid)) (fill none) (layer "F.CrtYd"))
+    (pad "" np_thru_hole circle (at 0 0) (size 3.5 3.5) (drill 3.5) (layers "*.Cu" "*.Mask"))
+  )
   (footprint "Connector_Dsub:DSUB-9_Male_Horizontal_P2.77x2.84mm_EdgePinOffset7.70mm_Housed_MountingHolesOffset9.12mm" (layer "F.Cu")
     (at 154.172 131.861669)
@@
   )
   (footprint "Capacitor_THT:CP_Radial_D6.3mm_P2.50mm" (layer "F.Cu")
-    (at 193.802 87.778)
+    (at 187.198 80.938379 90)
     (descr "CP, Radial series, Radial, pin pitch=2.50mm, , diameter=6.3mm, Electrolytic Capacitor")
     (tags "CP Radial series Radial pin pitch 2.50mm  diameter 6.3mm Electrolytic Capacitor")
@@
     (property "ki_keywords" "cap capacitor")
     (attr through_hole)
-    (fp_text reference "C102" (at 1.25 -4.4) (layer "F.SilkS")
+    (fp_text reference "C102" (at 1.25 -4.4 90) (layer "F.SilkS")
         (effects (font (size 1 1) (thickness 0.15)))
     )
-    (fp_text value "100µF" (at 1.25 4.4) (layer "F.Fab")
+    (fp_text value "100µF" (at 1.25 4.4 90) (layer "F.Fab")
         (effects (font (size 1 1) (thickness 0.15)))
     )
-    (fp_text user "${REFERENCE}" (at 1.25 0) (layer "F.Fab")
+    (fp_text user "${REFERENCE}" (at 1.25 0 90) (layer "F.Fab")
         (effects (font (size 1 1) (thickness 0.15)))
     )
@@
     (fp_circle (center 1.25 0) (end 4.4 0)
       (stroke (width 0.1) (type solid)) (fill none) (layer "F.Fab"))
-    (pad "1" thru_hole rect (at 0 0) (size 1.6 1.6) (drill 0.8) (layers "*.Cu" "*.Mask")
+    (pad "1" thru_hole rect (at 0 0 90) (size 1.6 1.6) (drill 0.8) (layers "*.Cu" "*.Mask")
       (net 3 "Net-(D101-A)") (pintype "passive"))
-    (pad "2" thru_hole circle (at 2.5 0) (size 1.6 1.6) (drill 0.8) (layers "*.Cu" "*.Mask")
+    (pad "2" thru_hole circle (at 2.5 0 90) (size 1.6 1.6) (drill 0.8) (layers "*.Cu" "*.Mask")
       (net 2 "GND") (pintype "passive"))
     (model "${KICAD6_3DMODEL_DIR}/Capacitor_THT.3dshapes/CP_Radial_D6.3mm_P2.50mm.wrl"
@@
     )
   )
+  (footprint "MountingHole:MountingHole_3.5mm" (layer "F.Cu")
+    (at 118.872 93.218)
+    (descr "Mounting Hole 3.5mm, no annular")
+    (tags "mounting hole 3.5mm no annular")
+    (property "Sheetfile" "CoPicoVision.kicad_sch")
+    (property "Sheetname" "")
+    (property "ki_description" "Mounting Hole without connection")
+    (property "ki_keywords" "mounting hole")
+    (attr exclude_from_pos_files)
+    (fp_text reference "H105" (at 0 -4.5) (layer "F.SilkS") hide
+        (effects (font (size 1 1) (thickness 0.15)))
+    )
+    (fp_text value "MountingHole" (at 0 4.5) (layer "F.Fab")
+        (effects (font (size 1 1) (thickness 0.15)))
+    )
+    (fp_text user "${REFERENCE}" (at 0 0) (layer "F.Fab")
+        (effects (font (size 1 1) (thickness 0.15)))
+    )
+    (fp_circle (center 0 0) (end 3.5 0)
+      (stroke (width 0.15) (type solid)) (fill none) (layer "Cmts.User"))
+    (fp_circle (center 0 0) (end 3.75 0)
+      (stroke (width 0.05) (type solid)) (fill none) (layer "F.CrtYd"))
+    (pad "" np_thru_hole circle (at 0 0) (size 3.5 3.5) (drill 3.5) (layers "*.Cu" "*.Mask"))
+  )
   (footprint "Package_DIP:DIP-20_W7.62mm_Socket" (layer "F.Cu")
     (at 194.31 56.388)
@@
     (effects (font (size 1 1) (thickness 0.15) italic) (justify left bottom))
   )
+  (dimension (type aligned) (layer "F.Fab")
+    (pts (xy 41.148 147.828) (xy 207.01 147.828))
+    (height 5.08)
+    (gr_text "165.8620 mm" (at 124.079 151.758) (layer "F.Fab")
+      (effects (font (size 1 1) (thickness 0.15)))
+    )
+    (format (prefix "") (suffix "") (units 3) (units_format 1) (precision 4))
+    (style (thickness 0.1) (arrow_length 1.27) (text_position_mode 0) (extension_height 0.58642) (extension_offset 0.5) keep_text_aligned)
+  )
+  (dimension (type aligned) (layer "F.Fab")
+    (pts (xy 41.148 37.846) (xy 41.148 147.828))
+    (height 5.08)
+    (gr_text "109.9820 mm" (at 34.918 92.837 90) (layer "F.Fab")
+      (effects (font (size 1 1) (thickness 0.15)))
+    )
+    (format (prefix "") (suffix "") (units 3) (units_format 1) (precision 4))
+    (style (thickness 0.1) (arrow_length 1.27) (text_position_mode 0) (extension_height 0.58642) (extension_offset 0.5) keep_text_aligned)
+  )
   (zone (net 0) (net_name "") (layers "F&B.Cu" "Dwgs.User") (hatch edge 0.5)

Commit message: PCB checkpoint -- some trace routing done.
Parts:
- moved RN101 71.2 mm to (102.9, 102.1), turned to -90 degrees
Routing:
- net CPUCLK: track 0.00 -> 150.0 mm, vias 0 -> 4
- net ~{RESET}: track 0.00 -> 108.5 mm, vias 0 -> 2
- net ~{WAIT}: track 0.00 -> 91.4 mm, vias 0 -> 1
- net ~{NMI}: track 0.00 -> 67.9 mm, vias 0 -> 1
- net D6: track 0.00 -> 64.9 mm, vias 0 -> 1
- net ~{MREQ}: track 0.00 -> 63.4 mm, vias 0 -> 1
- net D5: track 0.00 -> 62.9 mm, vias 0 -> 1
- net D7: track 0.00 -> 58.0 mm
- net A8: track 0.00 -> 52.9 mm, vias 0 -> 1
- net Net-(U202-IO2): track 0.00 -> 50.6 mm, vias 0 -> 2
- net /Video/CD6_L: track 0.00 -> 46.1 mm, vias 0 -> 2
- net Net-(Q101-S): track 0.00 -> 45.0 mm
- net ~{RAMSEL}: track 0.00 -> 44.3 mm, vias 0 -> 3
- net /Video/CD7_L: track 0.00 -> 42.0 mm, vias 0 -> 2
- net ~{M1}: track 0.00 -> 36.9 mm, vias 0 -> 1
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- added copper zone on In1.Cu, net GND
- added copper zone on In2.Cu, net VCC
Other:
- copper layers 2 -> 4
