File: design-files/CoPicoVision.kicad_pcb (KiCad board)
At the start: 4 copper layers, 165.9 x 110 mm, 101 parts, among them J101 USB_C_Receptacle_PowerOnly_6P, J102 Conn_02x15_Odd_Even, J301 DE15_Receptacle_HighDensity_M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, J401 Controller 1, J402 Controller 2, J501 AudioJack3, Q101 MMFTP3334K-AQ, Q401 2N3904, Q402 2N3904, Q501 KSD1616A, SW101 SW_Push, SW102 SW_Push, U101 Z80CPU, U102 DS1813, U103 74ACT05, U104 ICL7660A, U105 MAX16054, U201 GAL22V10, U202 GAL22V10, U203 AT28C64, U204 AS6C6264, U301 Pico, U302 74LVC245, U303 74LVC245, U401 74LS541, U402 74LS541, U403 74HCT00, U501 SN76489AN, X101 3.579545MHZ

Commit message: Another routing checkpoint.
Routing:
- net /Controller Interface/C2_D7: track 46.8 -> 67.7 mm, vias 2 -> 3
Changed lines of the file:
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@@
   (segment (start 175.135 115.461) (end 174.01 116.586) (width 0.25) (layer "F.Cu") (net 183))
   (segment (start 161.554 121.158) (end 179.07 121.158) (width 0.25) (layer "F.Cu") (net 183))
+  (segment (start 142.494 118.364) (end 158.76 118.364) (width 0.25) (layer "F.Cu") (net 183))
   (segment (start 178.816 116.586) (end 177.691 115.461) (width 0.25) (layer "F.Cu") (net 183))
   (segment (start 190.5 127.508) (end 189.23 126.238) (width 0.25) (layer "F.Cu") (net 183))
+  (segment (start 158.76 118.364) (end 160.274 119.878) (width 0.25) (layer "F.Cu") (net 183))
   (segment (start 189.23 126.238) (end 179.07 126.238) (width 0.25) (layer "F.Cu") (net 183))
   (via (at 179.07 126.238) (size 0.8) (drill 0.4) (layers "F.Cu" "B.Cu") (net 183))
   (via (at 179.07 121.158) (size 0.8) (drill 0.4) (layers "F.Cu" "B.Cu") (net 183))
+  (via (at 142.494 118.364) (size 0.8) (drill 0.4) (layers "F.Cu" "B.Cu") (net 183))
+  (segment (start 140.696 116.586) (end 142.474 118.364) (width 0.25) (layer "B.Cu") (net 183))
   (segment (start 179.07 116.84) (end 178.816 116.586) (width 0.25) (layer "B.Cu") (net 183))
+  (segment (start 142.474 118.364) (end 142.494 118.364) (width 0.25) (layer "B.Cu") (net 183))
   (segment (start 179.07 126.238) (end 179.07 116.84) (width 0.25) (layer "B.Cu") (net 183))
   (segment (start 190.5 116.585) (end 189.699001 117.385999) (width 0.25) (layer "F.Cu") (net 184))

Commit message: Use a discrete resistor for the PoR delay, rather than one from the 3K3 resistor pack.
Parts:
- added R104: 3K3, Resistor_THT:R_Axial_DIN0207_L6.3mm_D2.5mm_P7.62mm_Horizontal, F.Cu at (64.0, 129.8)
Connections:
- RN101 pad 2: Net-(D101-A) -> (no net)
Routing:
- net D2: track 157.8 -> 222.3 mm, vias 7 -> 8
- net D1: track 161.3 -> 223.5 mm, vias 6 -> 7
- net Net-(D101-A): track 0.00 -> 21.9 mm
- net -5V: track 207.0 -> 205.5 mm

Commit message: Use a 4-resistor pack, not 8.
Parts:
- RN101: footprint Resistor_THT:R_Array_SIP9 -> Resistor_THT:R_Array_SIP5
- moved RN101 2.54 mm to (102.9, 104.6)
Connections:
- RN101 pad 2: (no net) -> ~{WAIT}
- RN101 pad 3: ~{WAIT} -> ~{INT}
- RN101 pad 4: ~{INT} -> ~{NMI}
- RN101 pad 5: ~{NMI} -> Net-(RN101D-R4.2)
- U103 pad 6: Net-(RN101E-R5.2) -> Net-(RN101D-R4.2)
- U401 pad 19: Net-(RN101E-R5.2) -> Net-(RN101D-R4.2)
Routing:
- net Net-(RN101E-R5.2): track 80.5 -> 0.00 mm, vias 2 -> 0
- net Net-(RN101D-R4.2): track 0.00 -> 80.5 mm, vias 0 -> 2
- net VCC: track 43.7 -> 84.6 mm

Commit message: Data bus routed.
Routing:
- net D4: track 182.4 -> 407.8 mm, vias 8 -> 15
- net D3: track 186.4 -> 402.3 mm, vias 7 -> 11
- net D6: track 222.7 -> 404.4 mm, vias 10 -> 13
- net D5: track 223.0 -> 398.6 mm, vias 8 -> 10
- net D7: track 212.9 -> 385.4 mm, vias 3 -> 6
- net D0: track 155.2 -> 305.3 mm, vias 4 -> 8
- net D2: track 222.3 -> 352.1 mm, vias 8 -> 11
- net D1: track 223.5 -> 310.9 mm, vias 7 -> 9
- net ~{RFSH}: track 30.5 -> 31.7 mm
- net /Controller Interface/2V5: track 92.4 -> 93.6 mm
- net ~{M1}: track 37.7 -> 38.7 mm
- net /Controller Interface/C1_D7: track 67.0 -> 67.6 mm

Commit message: IODEC fully wired up.
Routing:
- net ~{VDPEN}: track 0.00 -> 117.8 mm, vias 0 -> 4
- net ~{VDPWSEL}: track 0.00 -> 109.2 mm, vias 0 -> 2
- net ~{VDPRSEL}: track 0.00 -> 97.7 mm, vias 0 -> 2
- net /Video/B3: track 29.1 -> 36.7 mm
- net /Video/B2: track 34.9 -> 36.9 mm
- net /Video/B1: track 14.2 -> 15.3 mm
- net /Video/CD1_L: track 27.5 -> 26.6 mm

Commit message: Cart address bus wired up.
Routing:
- net A10: track 47.8 -> 191.3 mm, vias 2 -> 7
- net A8: track 52.9 -> 188.5 mm, vias 1 -> 4
- net A14: track 20.6 -> 153.6 mm, vias 0 -> 4
- net A9: track 57.2 -> 185.6 mm, vias 3 -> 7
- net A12: track 30.4 -> 156.2 mm, vias 0 -> 4
- net A11: track 63.0 -> 187.8 mm, vias 2 -> 6
- net A4: track 35.7 -> 158.9 mm, vias 1 -> 5
- net A13: track 20.6 -> 139.3 mm, vias 0 -> 2
- net A3: track 34.8 -> 149.4 mm, vias 0 -> 2
- net A2: track 34.8 -> 138.0 mm, vias 0 -> 2
- net A1: track 96.4 -> 190.8 mm, vias 1 -> 3
- net A6: track 79.4 -> 173.9 mm, vias 2 -> 7
- net A5: track 77.4 -> 171.0 mm, vias 2 -> 5
- net A7: track 81.5 -> 173.6 mm, vias 2 -> 5
- net A0: track 122.4 -> 206.8 mm, vias 1 -> 2
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
Commit message: Cart slot all wired up.  Yeesh.
Routing:
- net ~{CRTASEL}: track 0.00 -> 204.1 mm, vias 0 -> 8
- net ~{CRT8SEL}: track 0.00 -> 186.0 mm, vias 0 -> 6
- net ~{RESET}: track 107.5 -> 287.6 mm, vias 3 -> 9
- net ~{CRTESEL}: track 0.00 -> 117.1 mm, vias 0 -> 3
- net ~{CRTCSEL}: track 0.00 -> 82.7 mm, vias 0 -> 2
- net D7: track 385.7 -> 387.2 mm
- net D5: track 398.6 -> 399.7 mm
- net D6: track 404.4 -> 403.3 mm
- net /Controller Interface/~{PAD_EN}: track 103.3 -> 104.3 mm
- net D4: track 407.8 -> 407.0 mm
- net A2: track 138.0 -> 138.7 mm
- net /Controller Interface/2V5: track 93.6 -> 94.2 mm
- net A14: track 153.6 -> 154.3 mm
- net /Controller Interface/C1_1: track 40.4 -> 40.9 mm
- net /Controller Interface/C1_4: track 33.8 -> 34.4 mm
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