File: design-files/CoPicoVision.kicad_pcb (KiCad board)
At the start: 4 copper layers, 165.9 x 110 mm, 110 parts, among them J101 USB_C_Receptacle_PowerOnly_6P, J102 Conn_02x15_Odd_Even, J301 DE15_Receptacle_HighDensity_M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, J401 Controller 1, J402 Controller 2, J501 AudioJack3, Q101 MMFTP3334K-AQ, Q401 2N3904, Q402 2N3904, SW101 SW_Push, SW102 SW_Push, U101 Z80CPU, U102 DS1813, U103 74ACT05, U104 ICL7660A, U105 MAX16054, U201 GAL22V10, U202 GAL22V10, U203 AT28C64, U204 AS6C62256, U205 74HCT08, U206 74HCT74, U301 Pico, U302 74LVC245, U303 74LVC245, U401 74LS541, U402 74LS541, U403 74HCT00, U501 SN76489AN, U502 TL071, X101 3.579545MHZ

Commit message: Add all of the SGM IODEC signals and re-pin the outputs to work better with the new board layout.
Connections:
- U201 pad 14: unconnected-(U201-IO1-Pad14) -> ~{SNWSEL}
- U201 pad 15: unconnected-(U201-IO2-Pad15) -> ~{AYSEL}
- U201 pad 16: unconnected-(U201-IO3-Pad16) -> ~{VDPEN}
- U201 pad 17: ~{CRSEL} -> ~{VDPWSEL}
- U201 pad 18: ~{C1WSEL} -> ~{VDPRSEL}
- U201 pad 19: ~{C2WSEL} -> ~{FF1WSEL}
- U201 pad 20: ~{VDPEN} -> ~{FF2WSEL}
- U201 pad 21: ~{VDPWSEL} -> ~{CRSEL}
- U201 pad 22: ~{VDPRSEL} -> ~{C1WSEL}
- U201 pad 23: ~{SNWSEL} -> ~{C2WSEL}

Commit message: Route most of the address / data lines.
Parts:
- moved C205 0.13 mm to (60.2, 55.2)
Connections:
- U201 pad 19: ~{FF1WSEL} -> ~{FF2WSEL}
- U201 pad 20: ~{FF2WSEL} -> ~{FF1WSEL}
Routing:
- net D0: track 87.8 -> 275.0 mm, vias 2 -> 8
- net D1: track 92.4 -> 275.6 mm, vias 2 -> 5
- net D2: track 123.7 -> 301.7 mm, vias 3 -> 9
- net A1: track 0.00 -> 177.4 mm, vias 0 -> 6
- net A4: track 0.00 -> 173.8 mm, vias 0 -> 9
- net D3: track 121.9 -> 295.3 mm, vias 3 -> 13
- net D7: track 121.2 -> 285.2 mm, vias 3 -> 12
- net A3: track 1.04 -> 162.9 mm, vias 1 -> 5
- net D5: track 132.1 -> 293.1 mm, vias 4 -> 10
- net D4: track 151.9 -> 309.6 mm, vias 6 -> 14
- net A2: track 0.00 -> 154.8 mm, vias 0 -> 7
- net Net-(D401-K): track 5.04 -> 159.4 mm, vias 0 -> 8
- net A0: track 40.6 -> 183.2 mm, vias 1 -> 5
- net D6: track 148.4 -> 290.3 mm, vias 4 -> 12
- net A14: track 1.79 -> 141.8 mm, vias 1 -> 4
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
Commit message: Put the AY-3-8910 on the schematic.  Need to make some more room on the board.
Parts:
- added C505: 0.1µF, Capacitor_SMD:C_0805_2012Metric_Pad1.18x1.45mm_HandSolder, F.Cu at (-8.84, 104.6)
- added C506: 0.1µF, Capacitor_SMD:C_0805_2012Metric_Pad1.18x1.45mm_HandSolder, F.Cu at (-8.84, 107.6)
- added R503: 1K, Resistor_SMD:R_0805_2012Metric_Pad1.20x1.40mm_HandSolder, F.Cu at (-8.87, 95.7)
- added R504: 1K, Resistor_SMD:R_0805_2012Metric_Pad1.20x1.40mm_HandSolder, F.Cu at (-8.87, 98.7)
- added R505: 1K, Resistor_SMD:R_0805_2012Metric_Pad1.20x1.40mm_HandSolder, F.Cu at (-8.87, 101.6)
- added U503: AY-3-8910, Package_DIP:DIP-40_W15.24mm, F.Cu at (-28.1, 86.1)
- added U504: 74HCT02, Package_SO:SOIC-14_3.9x8.7mm_P1.27mm, F.Cu at (-7.02, 89.1)

Commit message: Move the video module to the right, making room for the AY-3-8910.
Parts:
- moved C301 12.1 mm to (204.1, 54.0), turned to -90 degrees
- moved C302 11.8 mm to (204.1, 70.8), turned to -90 degrees
- moved U303 9.81 mm to (197.0, 75.4)
- moved D301 9.68 mm to (192.9, 40.3), turned to -90 degrees
- moved U302 9.17 mm to (197.1, 58.7)
- moved RN301 8.14 mm to (161.6, 57.7)
- moved RN302 8.14 mm to (164.9, 45.2)
- moved RN303 8.14 mm to (164.9, 66.5)
- moved RN304 8.14 mm to (161.6, 64.3)
- moved RN305 8.14 mm to (161.6, 54.3)
- moved RN306 8.14 mm to (161.6, 61.0)
- moved RN307 8.14 mm to (161.6, 67.6)
- moved U301 8.14 mm to (178.2, 64.2)
- moved J301 8.14 mm to (143.0, 50.4)
Routing:
- net A6: track 94.4 -> 67.2 mm, vias 9 -> 6
- net /Video/CD6_L: track 20.3 -> 3.24 mm
- net /Video/CD7_L: track 15.7 -> 0.20 mm, vias 1 -> 0
- net Net-(D301-K): track 4.73 -> 0.92 mm
- net ~{RESET}: vias 9 -> 8

Commit message: Put the AY-3-8910 on the board, clarify part numbers for the 74xx chips to ensure the correct SOIC footprints.
Parts:
- U103: value 74ACT05 -> MC74ACT05DR2G
- U205: value 74HCT08 -> MM74HCT08MX
- U206: value 74HCT74 -> MM74HCT74MX
- U302, U303: value 74LVC245 -> SN74LVC245ADWR
- U403: value 74HCT00 -> SN74HCT00DR
- U503: footprint Package_DIP:DIP-40_W15.24mm -> Package_DIP:DIP-40_W15.24mm_Socket
- U504: value 74HCT02 -> SN74HCT02D
- moved C506 138.2 mm to (118.9, 54.6)
- moved U504 131.8 mm to (121.4, 59.4), turned to 90 degrees
- moved U503 115.6 mm to (87.4, 81.0), turned to 90 degrees
- moved R505 108.7 mm to (92.5, 62.2), turned to -90 degrees
- moved R504 104.6 mm to (89.2, 62.2), turned to -90 degrees
- moved C505 100.8 mm to (84.6, 66.8), turned to -90 degrees
- moved R503 100.5 mm to (85.9, 62.2), turned to -90 degrees
- moved C502 3.09 mm to (118.6, 42.9)
- moved R501 2.50 mm to (103.1, 56.6), turned to 90 degrees
- moved U501 2.33 mm to (105.9, 42.4)
- moved C501 2.33 mm to (114.8, 39.6)
Connections:
- U503 pad 35: unconnected-(U503-DA2-Pad35) -> D2
Routing:
- net VCC: track 139.2 -> 114.8 mm
- net Net-(C503-Pad1): track 5.97 -> 0.00 mm
- net Net-(U501-AUDIO_OUT): track 3.82 -> 0.00 mm
- net ~{INT}: track 60.9 -> 61.6 mm
- net ~{NMI}: track 70.3 -> 71.0 mm
- net ~{RAMSEL}: track 63.8 -> 63.1 mm
Other:
- board text added: "Super"

Commit message: I think that's the whole right side of the board now routed.
Connections:
- U503 pad 31: D7 -> D6
Routing:
- net ~{RESET}: track 230.8 -> 459.9 mm, vias 8 -> 17
- net ~{VDPRSEL}: track 0.00 -> 175.1 mm, vias 0 -> 6
- net ~{VDPWSEL}: track 0.00 -> 174.5 mm, vias 0 -> 9
- net A7: track 65.1 -> 229.0 mm, vias 6 -> 12
- net ~{VDPEN}: track 0.00 -> 159.7 mm, vias 0 -> 9
- net A8: track 19.6 -> 165.2 mm, vias 1 -> 5
- net A9: track 18.6 -> 162.1 mm, vias 1 -> 5
- net A6: track 67.2 -> 205.8 mm, vias 6 -> 10
- net A11: track 15.7 -> 150.2 mm, vias 1 -> 5
- net D7: track 285.2 -> 411.6 mm, vias 12 -> 20
- net A12: track 97.3 -> 223.7 mm, vias 4 -> 6
- net A10: track 22.0 -> 142.2 mm, vias 1 -> 3
- net D6: track 290.3 -> 409.8 mm, vias 12 -> 20
- net A5: track 66.4 -> 185.1 mm, vias 6 -> 8
- net D5: track 293.1 -> 407.2 mm, vias 10 -> 17
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
Commit message: I think that's all the address lines now.
Routing:
- net A11: track 150.2 -> 215.9 mm, vias 5 -> 9
- net A8: track 165.2 -> 221.1 mm, vias 5 -> 9
- net A9: track 162.1 -> 213.1 mm, vias 5 -> 9
- net A10: track 142.2 -> 183.4 mm, vias 3 -> 8
- net A4: track 175.9 -> 178.1 mm
- net A5: track 185.1 -> 186.6 mm
- net A3: track 163.7 -> 164.9 mm
- net D7: track 411.6 -> 410.5 mm
- net D5: track 407.2 -> 406.2 mm
- net A2: track 155.4 -> 154.5 mm
- net ~{VDPWSEL}: track 174.5 -> 175.2 mm
- net A6: track 205.8 -> 205.2 mm
- net D6: track 409.8 -> 410.4 mm
- net ~{VDPRSEL}: track 175.1 -> 175.6 mm

Commit message: Fix a dumb mistake in the power supply (put the reservoir cap on VCC, not VBUS), and fix a bunch of unconnected items.
Parts:
- moved R103 0.11 mm to (73.4, 39.6), turned to 0 degrees
- moved Q101 0.08 mm to (73.3, 42.8), turned to -90 degrees
Connections:
- C105 pad 1: /VBUS -> VCC
Routing:
- net /Video/INT_L: track 0.00 -> 139.9 mm, vias 0 -> 6
- net ~{WR}: track 105.3 -> 174.8 mm, vias 5 -> 8
- net A1: track 172.2 -> 210.2 mm, vias 6 -> 9
- net VCC: track 120.3 -> 83.4 mm
- net ~{CRT8SEL}: track 218.7 -> 231.9 mm
- net GND: track 46.1 -> 58.1 mm, vias 5 -> 9
- net /VBUS: track 50.0 -> 39.7 mm, vias 0 -> 2
- net Net-(D301-K): track 0.92 -> 7.73 mm
- net Net-(Q101-G): track 14.1 -> 10.7 mm
- net Net-(RN303-R3.2): track 0.00 -> 2.54 mm
- net ~{RESET}: track 459.9 -> 460.9 mm
- net ~{WAIT}: track 134.0 -> 134.8 mm
- net ~{CRSEL}: track 163.7 -> 162.9 mm
- net ~{VDPEN}: track 159.5 -> 160.1 mm
