File: design-files/CoPicoVision_controllers.kicad_sch (KiCad schematic)
At the start: 41 parts, among them J401 Controller 1, J402 Controller 2, Q401 2N3904, Q402 2N3904, U103 74ACT05, U401 74LS541, U402 74LS541, U403 74HCT00

Commit message: BoM.
Parts:
- C101: Mouser (none) -> 81-RCER71H103K0A2H3B
- C101, C103, C104: Mouser (none) -> 81-RCER71E104K0A2H3B
- C104: Mouser (none) -> 81-RCER71H473K0A2H3B
- C104: Mouser (none) -> 81-RCE5C1H101J0A2H3B
- D401, D402: Mouser (none) -> 637-1N4001
- Q401, Q402: Mouser (none) -> 583-2N3904
- RN101: Mouser (none) -> 652-4605M-1LF-3.3K
- RN401, RN402: Mouser (none) -> 652-4608X-1LF-22K
- U103: Mouser (none) -> 595-CD74ACT05EE4
- U401, U402: Mouser (none) -> 595-SN74LS541NE4
- U403: Mouser (none) -> 595-SN74HCT00N
Changed lines of the file:
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@@
+      (effects (font (size 1.27 1.27)) hide)
+    )
+    (property "Mouser" "81-RCER71H103K0A2H3B" (at 160.274 105.41 0)
       (effects (font (size 1.27 1.27)) hide)
     )
@@
     )
     (property "Datasheet" "http://www.vishay.com/docs/31509/csc.pdf" (at 226.441 113.919 0)
+      (effects (font (size 1.27 1.27)) hide)
+    )
+    (property "Mouser" "652-4608X-1LF-22K" (at 226.441 113.919 0)
       (effects (font (size 1.27 1.27)) hide)
     )
@@
       (effects (font (size 1.27 1.27)) hide)
     )
+    (property "Mouser" "81-RCER71H473K0A2H3B" (at 92.71 144.272 90)
+      (effects (font (size 1.27 1.27)) hide)
+    )
     (pin "1")
     (pin "2")
@@
     (property "Datasheet" "https://www.onsemi.com/pub/Collateral/2N3903-D.PDF" (at 102.235 56.896 0)
       (effects (font (size 1.27 1.27)) (justify left) hide)
+    )
+    (property "Mouser" "583-2N3904" (at 102.235 56.896 0)
+      (effects (font (size 1.27 1.27)) hide)
     )
     (pin "1")
@@
     )
     (property "Datasheet" "http://www.ti.com/lit/gpn/sn74hct00" (at 82.55 154.305 0)
+      (effects (font (size 1.27 1.27)) hide)
+    )
+    (property "Mouser" "595-SN74HCT00N" (at 82.55 154.305 0)
       (effects (font (size 1.27 1.27)) hide)
     )
@@
       (effects (font (size 1.27 1.27)) hide)
     )
+    (property "Mouser" "81-RCER71E104K0A2H3B" (at 17.78 188.849 0)
+      (effects (font (size 1.27 1.27)) hide)
+    )
     (pin "1")
     (pin "2")
@@
     )
     (property "Datasheet" "http://www.vishay.com/docs/31509/csc.pdf" (at 226.441 38.1 0)
+      (effects (font (size 1.27 1.27)) hide)
+    )
+    (property "Mouser" "652-4608X-1LF-22K" (at 226.441 38.1 0)
       (effects (font (size 1.27 1.27)) hide)
     )
@@
     )
     (property "Datasheet" "http://www.ti.com/lit/gpn/sn74LS541" (at 252.603 137.922 0)
+      (effects (font (size 1.27 1.27)) hide)
+    )
+    (property "Mouser" "595-SN74LS541NE4" (at 252.603 137.922 0)
       (effects (font (size 1.27 1.27)) hide)
     )
@@
       (effects (font (size 1.27 1.27)) hide)
     )
+    (property "Mouser" "81-RCE5C1H101J0A2H3B" (at 94.615 56.896 90)
+      (effects (font (size 1.27 1.27)) hide)
+    )
     (pin "1")
     (pin "2")
@@
     )
     (property "Datasheet" "https://www.ti.com/lit/ds/symlink/cd74act05.pdf" (at 144.145 95.25 0)
+      (effects (font (size 1.27 1.27)) hide)
+    )
+    (property "Mouser" "595-CD74ACT05EE4" (at 144.145 95.25 0)
       (effects (font (size 1.27 1.27)) hide)
     )
@@
       (effects (font (size 1.27 1.27)) hide)
     )
+    (property "Mouser" "595-SN74HCT00N" (at 160.909 178.435 0)
+      (effects (font (size 1.27 1.27)) hide)
+    )
     (pin "1")
     (pin "2")
@@
       (effects (font (size 1.27 1.27)) hide)
     )
+    (property "Mouser" "81-RCER71H103K0A2H3B" (at 34.671 105.283 0)
+      (effects (font (size 1.27 1.27)) hide)
+    )
     (pin "1")
     (pin "2")
@@
     )
     (property "Datasheet" "http://www.vishay.com/docs/31509/csc.pdf" (at 239.903 78.613 0)
+      (effects (font (size 1.27 1.27)) hide)
+    )
+    (property "Mouser" "652-4605M-1LF-3.3K" (at 239.903 78.613 0)
       (effects (font (size 1.27 1.27)) hide)
     )
@@
       (effects (font (size 1.27 1.27)) hide)
     )
+    (property "Mouser" "81-RCER71E104K0A2H3B" (at 68.199 159.385 0)
+      (effects (font (size 1.27 1.27)) hide)
+    )
     (pin "1")
     (pin "2")
@@
       (effects (font (size 1.27 1.27)) hide)
     )
+    (property "Mouser" "81-RCER71E104K0A2H3B" (at 40.005 188.849 0)
+      (effects (font (size 1.27 1.27)) hide)
+    )
     (pin "1")
     (pin "2")
@@
     )
     (property "Datasheet" "http://www.ti.com/lit/gpn/sn74LS541" (at 252.603 62.103 0)
+      (effects (font (size 1.27 1.27)) hide)
+    )
+    (property "Mouser" "595-SN74LS541NE4" (at 252.603 62.103 0)
       (effects (font (size 1.27 1.27)) hide)
     )
@@
     )
     (property "Datasheet" "http://www.ti.com/lit/gpn/sn74hct00" (at 84.455 56.896 0)
+      (effects (font (size 1.27 1.27)) hide)
+    )
+    (property "Mouser" "595-SN74HCT00N" (at 84.455 56.896 0)
       (effects (font (size 1.27 1.27)) hide)
     )
@@
       (effects (font (size 1.27 1.27)) hide)
     )
+    (property "Mouser" "81-RCER71E104K0A2H3B" (at 28.829 188.849 0)
+      (effects (font (size 1.27 1.27)) hide)
+    )
     (pin "1")
     (pin "2")
@@
     )
     (property "Datasheet" "http://www.ti.com/lit/gpn/sn74hct00" (at 71.501 92.329 0)
+      (effects (font (size 1.27 1.27)) hide)
+    )
+    (property "Mouser" "595-SN74HCT00N" (at 71.501 92.329 0)
       (effects (font (size 1.27 1.27)) hide)
     )
@@
       (effects (font (size 1.27 1.27)) hide)
     )
+    (property "Mouser" "595-CD74ACT05EE4" (at 224.155 74.803 0)
+      (effects (font (size 1.27 1.27)) hide)
+    )
     (pin "1")
     (pin "2")
@@
       (effects (font (size 1.27 1.27)) hide)
     )
+    (property "Mouser" "81-RCER71H473K0A2H3B" (at 94.615 46.863 90)
+      (effects (font (size 1.27 1.27)) hide)
+    )
     (pin "1")
     (pin "2")
@@
       (effects (font (size 1.27 1.27)) hide)
     )
+    (property "Mouser" "81-RCER71H103K0A2H3B" (at 34.671 100.203 0)
+      (effects (font (size 1.27 1.27)) hide)
+    )
     (pin "1")
     (pin "2")
@@
       (effects (font (size 1.27 1.27)) hide)
     )
+    (property "Mouser" "637-1N4001" (at 160.274 99.06 90)
+      (effects (font (size 1.27 1.27)) hide)
+    )
     (pin "1")
     (pin "2")
@@
       (effects (font (size 1.27 1.27)) hide)
     )
+    (property "Mouser" "81-RCER71E104K0A2H3B" (at 70.104 61.976 0)
+      (effects (font (size 1.27 1.27)) hide)
+    )
     (pin "1")
     (pin "2")
@@
     (property "Datasheet" "https://www.onsemi.com/pub/Collateral/2N3903-D.PDF" (at 100.33 154.305 0)
       (effects (font (size 1.27 1.27)) (justify left) hide)
+    )
+    (property "Mouser" "583-2N3904" (at 100.33 154.305 0)
+      (effects (font (size 1.27 1.27)) hide)
     )
     (pin "1")
@@
     )
     (property "Datasheet" "http://www.ti.com/lit/gpn/sn74hct00" (at 71.501 113.284 0)
+      (effects (font (size 1.27 1.27)) hide)
+    )
+    (property "Mouser" "595-SN74HCT00N" (at 71.501 113.284 0)
       (effects (font (size 1.27 1.27)) hide)
     )
@@
       (effects (font (size 1.27 1.27)) hide)
     )
+    (property "Mouser" "637-1N4001" (at 160.274 91.44 90)
+      (effects (font (size 1.27 1.27)) hide)
+    )
     (pin "1")
     (pin "2")
@@
       (effects (font (size 1.27 1.27)) hide)
     )
+    (property "Mouser" "81-RCER71H103K0A2H3B" (at 160.274 85.09 0)
+      (effects (font (size 1.27 1.27)) hide)
+    )
     (pin "1")
     (pin "2")
@@
       (effects (font (size 1.27 1.27)) hide)
     )
+    (property "Mouser" "81-RCE5C1H101J0A2H3B" (at 92.71 154.305 90)
+      (effects (font (size 1.27 1.27)) hide)
+    )
