File: design-files/CoPicoVision_controllers.kicad_sch (KiCad schematic)
At the start: 41 parts, among them J401 Controller 1, J402 Controller 2, Q401 2N3904, Q402 2N3904, U103 74ACT05, U401 74LS541, U402 74LS541, U403 74HCT00

Commit message: Add title blocks.
Other:
- company: (none) -> (c) 2024 Jason R. Thorpe.  See LICENSE.
- title: (none) -> CoPicoVision
Changed lines of the file:
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@@
 (kicad_sch (version 20230121) (generator eeschema)
   (paper "A4")
+  (title_block
+    (title "CoPicoVision")
+    (date "2024-08-31")
+    (rev "0.1")
+    (company "(c) 2024 Jason R. Thorpe.  See LICENSE.")
+  )
   (junction (at 223.901 130.302) (diameter 0) (color 0 0 0 0)
   )

Commit message: Change R401 and R402 to 220R resistors.
Parts:
- R401, R402: value 210R -> 220R
Changed lines of the file:
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@@
       (effects (font (size 1.27 1.27)) (justify left))
     )
-    (property "Value" "210R" (at 147.32 182.88 0)
+    (property "Value" "220R" (at 147.32 182.88 0)
       (effects (font (size 1.27 1.27)) (justify left))
     )
@@
   )
   (symbol (lib_id "Device:R_Small") (at 144.78 175.895 0) (unit 1)
-    (in_bom yes) (on_board yes) (dnp no) (fields_autoplaced)
+    (in_bom yes) (on_board yes) (dnp no)
     (property "Reference" "R401" (at 147.32 175.26 0)
       (effects (font (size 1.27 1.27)) (justify left))
     )
-    (property "Value" "210R" (at 147.32 177.8 0)
-      (effects (font (size 1.27 1.27)) (justify left))
-    )
+    (property "Value" "220R" (at 147.32 177.8 0)
+      (effects (font (size 1.27 1.27)) (justify left))
+    )

Commit message: Fix the swapped controller problem that rev 0.1 boards have: the G2 input of the 74LS541 is active-low, so A1 low means Controller 1 is selected.
Connections:
- net A1: now also U401.19 (G2); no longer U402.19 (G2)
- net at U103.6: now also U402.19 (G2); no longer U401.19 (G2)
Other:
- moved on the sheet: RN101E, U103C
Changed lines of the file:
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@@
   (title_block
     (title "CoPicoVision")
-    (date "2024-08-31")
-    (rev "0.1")
+    (date "2024-10-12")
+    (rev "0.2")
     (company "(c) 2024 Jason R. Thorpe.  See LICENSE.")
   )
@@
   (junction (at 92.075 56.896) (diameter 0) (color 0 0 0 0)
   )
+  (junction (at 239.903 150.622) (diameter 0) (color 0 0 0 0)
+  )
   (junction (at 63.881 113.284) (diameter 0) (color 0 0 0 0)
   )
@@
     (stroke (width 0) (type default))
   )
-  (wire (pts (xy 231.775 74.803) (xy 239.903 74.803))
+  (wire (pts (xy 231.775 150.622) (xy 239.903 150.622))
     (stroke (width 0) (type default))
   )
@@
     )
   )
-  (global_label "A1" (shape input) (at 239.903 150.622 180) (fields_autoplaced)
+  (global_label "A1" (shape input) (at 239.903 74.803 180) (fields_autoplaced)
     (effects (font (size 1.27 1.27)) (justify right))
-    (property "Intersheetrefs" "${INTERSHEET_REFS}" (at 234.6991 150.622 0)
+    (property "Intersheetrefs" "${INTERSHEET_REFS}" (at 234.6991 74.803 0)
       (effects (font (size 1.27 1.27)) (justify right) hide)
     )
@@
     )
   )
-  (global_label "A1" (shape input) (at 216.535 74.803 180) (fields_autoplaced)
+  (global_label "A1" (shape input) (at 216.535 150.622 180) (fields_autoplaced)
     (effects (font (size 1.27 1.27)) (justify right))
-    (property "Intersheetrefs" "${INTERSHEET_REFS}" (at 211.3311 74.803 0)
+    (property "Intersheetrefs" "${INTERSHEET_REFS}" (at 211.3311 150.622 0)
       (effects (font (size 1.27 1.27)) (justify right) hide)
     )
@@
     )
   )
-  (symbol (lib_id "Device:R_Network04_Split") (at 239.903 78.613 180) (unit 5)
-    (in_bom yes) (on_board yes) (dnp no) (fields_autoplaced)
-    (property "Reference" "RN101" (at 237.744 79.248 0)
-      (effects (font (size 1.27 1.27)) (justify left))
-    )
-    (property "Value" "3K3" (at 237.744 76.708 0)
-      (effects (font (size 1.27 1.27)) (justify left))
-    )
-    (property "Footprint" "Resistor_THT:R_Array_SIP5" (at 241.935 78.613 90)
-      (effects (font (size 1.27 1.27)) hide)
-    )
-    (property "Datasheet" "http://www.vishay.com/docs/31509/csc.pdf" (at 239.903 78.613 0)
-      (effects (font (size 1.27 1.27)) hide)
-    )
-    (property "Mouser" "652-4605M-1LF-3.3K" (at 239.903 78.613 0)
+  (symbol (lib_id "Device:R_Network04_Split") (at 239.903 154.432 180) (unit 5)
+    (in_bom yes) (on_board yes) (dnp no) (fields_autoplaced)
+    (property "Reference" "RN101" (at 237.744 155.067 0)
+      (effects (font (size 1.27 1.27)) (justify left))
+    )
+    (property "Value" "3K3" (at 237.744 152.527 0)
+      (effects (font (size 1.27 1.27)) (justify left))
+    )
+    (property "Footprint" "Resistor_THT:R_Array_SIP5" (at 241.935 154.432 90)
+      (effects (font (size 1.27 1.27)) hide)
+    )
+    (property "Datasheet" "http://www.vishay.com/docs/31509/csc.pdf" (at 239.903 154.432 0)
+      (effects (font (size 1.27 1.27)) hide)
+    )
+    (property "Mouser" "652-4605M-1LF-3.3K" (at 239.903 154.432 0)
       (effects (font (size 1.27 1.27)) hide)
     )
@@
     )
   )
-  (symbol (lib_id "74xx:74LS05") (at 224.155 74.803 0) (unit 3)
+  (symbol (lib_id "74xx:74LS05") (at 224.155 150.622 0) (unit 3)
     (in_bom yes) (on_board yes) (dnp no)
-    (property "Reference" "U103" (at 219.71 69.977 0)
-      (effects (font (size 1.27 1.27)) (justify left))
-    )
-    (property "Value" "74ACT05" (at 219.964 79.883 0)
-      (effects (font (size 1.27 1.27)) (justify left))
-    )
-    (property "Footprint" "Package_DIP:DIP-14_W7.62mm_Socket" (at 224.155 74.803 0)
-      (effects (font (size 1.27 1.27)) hide)
-    )
-    (property "Datasheet" "https://www.ti.com/lit/ds/symlink/cd74act05.pdf" (at 224.155 74.803 0)
-      (effects (font (size 1.27 1.27)) hide)
-    )
-    (property "Mouser" "595-CD74ACT05EE4" (at 224.155 74.803 0)
+    (property "Reference" "U103" (at 219.71 145.796 0)
+      (effects (font (size 1.27 1.27)) (justify left))
+    )
+    (property "Value" "74ACT05" (at 219.964 155.702 0)
+      (effects (font (size 1.27 1.27)) (justify left))
+    )
+    (property "Footprint" "Package_DIP:DIP-14_W7.62mm_Socket" (at 224.155 150.622 0)
+      (effects (font (size 1.27 1.27)) hide)
+    )
+    (property "Datasheet" "https://www.ti.com/lit/ds/symlink/cd74act05.pdf" (at 224.155 150.622 0)
+      (effects (font (size 1.27 1.27)) hide)
+    )
+    (property "Mouser" "595-CD74ACT05EE4" (at 224.155 150.622 0)
       (effects (font (size 1.27 1.27)) hide)
     )
@@
     )
   )
-  (symbol (lib_id "power:VCC") (at 239.903 82.423 180) (unit 1)
-    (in_bom yes) (on_board yes) (dnp no) (fields_autoplaced)
-    (property "Reference" "#PWR0407" (at 239.903 78.613 0)
-      (effects (font (size 1.27 1.27)) hide)
-    )
-    (property "Value" "VCC" (at 239.903 86.487 0)
-      (effects (font (size 1.27 1.27)))
-    )
-    (property "Footprint" "" (at 239.903 82.423 0)
-      (effects (font (size 1.27 1.27)) hide)
-    )
-    (property "Datasheet" "" (at 239.903 82.423 0)
-      (effects (font (size 1.27 1.27)) hide)
-    )
+  (symbol (lib_id "power:VCC") (at 239.903 158.242 180) (unit 1)
+    (in_bom yes) (on_board yes) (dnp no) (fields_autoplaced)
+    (property "Reference" "#PWR0407" (at 239.903 154.432 0)
+      (effects (font (size 1.27 1.27)) hide)
+    )
+    (property "Value" "VCC" (at 239.903 162.306 0)
+      (effects (font (size 1.27 1.27)))
+    )
+    (property "Footprint" "" (at 239.903 158.242 0)
+      (effects (font (size 1.27 1.27)) hide)
+    )
+    (property "Datasheet" "" (at 239.903 158.242 0)
+      (effects (font (size 1.27 1.27)) hide)
+    )

Commit message: Add a 1.5K current limiting resistor between the SN76489AN audio output and the KSD1616A emitter-follower.
Changed lines of the file:
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@@
   (junction (at 92.075 56.896) (diameter 0) (color 0 0 0 0)
-  )
-  (junction (at 239.903 150.622) (diameter 0) (color 0 0 0 0)
   )
   (junction (at 63.881 113.284) (diameter 0) (color 0 0 0 0)

Commit message: All the bypass caps are now 0805s.
Parts:
- C101, C103, C104: footprint Capacitor_THT:C_Disc_D3.8mm_W2.6mm_P2.50mm -> Capacitor_SMD:C_0805_2012Metric_Pad1.18x1.45mm_HandSolder
Changed lines of the file:
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@@
       (effects (font (size 1.27 1.27)) (justify left))
     )
-    (property "Footprint" "Capacitor_THT:C_Disc_D3.8mm_W2.6mm_P2.50mm" (at 17.78 188.849 0)
+    (property "Footprint" "Capacitor_SMD:C_0805_2012Metric_Pad1.18x1.45mm_HandSolder" (at 17.78 188.849 0)
       (effects (font (size 1.27 1.27)) hide)
     )
@@
       (effects (font (size 1.27 1.27)) (justify left))
     )
-    (property "Footprint" "Capacitor_THT:C_Disc_D3.8mm_W2.6mm_P2.50mm" (at 40.005 188.849 0)
+    (property "Footprint" "Capacitor_SMD:C_0805_2012Metric_Pad1.18x1.45mm_HandSolder" (at 40.005 188.849 0)
       (effects (font (size 1.27 1.27)) hide)
     )
@@
       (effects (font (size 1.27 1.27)) (justify left))
     )
-    (property "Footprint" "Capacitor_THT:C_Disc_D3.8mm_W2.6mm_P2.50mm" (at 28.829 188.849 0)
-      (effects (font (size 1.27 1.27)) hide)
-    )
+    (property "Footprint" "Capacitor_SMD:C_0805_2012Metric_Pad1.18x1.45mm_HandSolder" (at 28.829 188.849 0)
+      (effects (font (size 1.27 1.27)) hide)
+    )

Commit message: Controller section is mostly SMT now.
Parts:
- C101, C104: footprint Capacitor_THT:C_Disc_D3.8mm_W2.6mm_P2.50mm -> Capacitor_SMD:C_0805_2012Metric_Pad1.18x1.45mm_HandSolder
- R401, R402, R403, R404, R405, R406, R407, R408, R409, R410, R411, R412, R413, R414, R415: footprint Resistor_THT:R_Axial_DIN0207_L6.3mm_D2.5mm_P7.62mm_Horizontal -> Resistor_SMD:R_0805_2012Metric_Pad1.20x1.40mm_HandSolder
- U103, U403: footprint Package_DIP:DIP-14_W7.62mm_Socket -> Package_SO:SOIC-14_3.9x8.7mm_P1.27mm

Commit message: Put the AY-3-8910 on the board, clarify part numbers for the 74xx chips to ensure the correct SOIC footprints.
Parts:
- U103: value 74ACT05 -> MC74ACT05DR2G
- U403: value 74HCT00 -> SN74HCT00DR
Changed lines of the file:
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@@
       (effects (font (size 1.27 1.27)))
     )
-    (property "Value" "74HCT00" (at 82.5417 148.717 0)
+    (property "Value" "SN74HCT00DR" (at 82.5417 148.717 0)
       (effects (font (size 1.27 1.27)))
     )
@@
       (effects (font (size 1.27 1.27)) (justify left))
     )
-    (property "Value" "74ACT05" (at 145.669 100.711 0)
+    (property "Value" "MC74ACT05DR2G" (at 145.669 100.711 0)
       (effects (font (size 1.27 1.27)) (justify left))
     )
@@
       (effects (font (size 1.27 1.27)) (justify left))
     )
-    (property "Value" "74HCT00" (at 167.64 180.34 0)
+    (property "Value" "SN74HCT00DR" (at 167.64 180.34 0)
       (effects (font (size 1.27 1.27)) (justify left))
     )
@@
       (effects (font (size 1.27 1.27)))
     )
-    (property "Value" "74HCT00" (at 84.4467 51.181 0)
+    (property "Value" "SN74HCT00DR" (at 84.4467 51.181 0)
       (effects (font (size 1.27 1.27)))
     )
@@
       (effects (font (size 1.27 1.27)))
     )
-    (property "Value" "74HCT00" (at 71.5093 87.122 0)
+    (property "Value" "SN74HCT00DR" (at 71.5093 87.122 0)
       (effects (font (size 1.27 1.27)))
     )
@@
       (effects (font (size 1.27 1.27)) (justify left))
     )
-    (property "Value" "74ACT05" (at 219.964 155.702 0)
+    (property "Value" "MC74ACT05DR2G" (at 212.598 155.575 0)
       (effects (font (size 1.27 1.27)) (justify left))
     )
@@
       (effects (font (size 1.27 1.27)))
     )
-    (property "Value" "74HCT00" (at 71.628 122.047 0)
-      (effects (font (size 1.27 1.27)))
-    )
+    (property "Value" "SN74HCT00DR" (at 71.628 122.047 0)
+      (effects (font (size 1.27 1.27)))
+    )
