File: design-files/CoPicoVision_controllers.kicad_sch (KiCad schematic)
At the start: 41 parts, among them J401 Controller 1, J402 Controller 2, Q401 2N3904, Q402 2N3904, U103 MC74ACT05D, U401 74LS541, U402 74LS541, U403 SN74HCT00D

Commit message: Change Q401 and Q402 to SOT-523 packages.
Parts:
- Q401, Q402: value 2N3904 -> MMBT3904T; footprint Package_TO_SOT_THT:TO-92_Inline -> Package_TO_SOT_SMD:SOT-523; symbol Transistor_BJT:2N3904 -> Device:Q_NPN_BEC; Mouser 583-2N3904 -> 621-MMBT3904T-F
Connections:
- net GND: now also Q401.2 (E), Q402.2 (E); no longer Q401.1 (E), Q402.1 (E)
- net at C104.2, R408.2: now also Q401.1 (B); no longer Q401.2 (B)
- net at C104.2, R411.2: now also Q402.1 (B); no longer Q402.2 (B)
Changed lines of the file:
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@@
     )
   )
-  (symbol (lib_id "Transistor_BJT:2N3904") (at 102.235 56.896 0) (unit 1)
+  (symbol (lib_id "Device:Q_NPN_BEC") (at 102.235 56.896 0) (unit 1)
     (in_bom yes) (on_board yes) (dnp no) (fields_autoplaced)
     (property "Reference" "Q401" (at 107.95 56.261 0)
       (effects (font (size 1.27 1.27)) (justify left))
     )
-    (property "Value" "2N3904" (at 107.95 58.801 0)
-      (effects (font (size 1.27 1.27)) (justify left))
-    )
-    (property "Footprint" "Package_TO_SOT_THT:TO-92_Inline" (at 107.315 58.801 0)
-      (effects (font (size 1.27 1.27) italic) (justify left) hide)
-    )
-    (property "Datasheet" "https://www.onsemi.com/pub/Collateral/2N3903-D.PDF" (at 102.235 56.896 0)
-      (effects (font (size 1.27 1.27)) (justify left) hide)
-    )
-    (property "Mouser" "583-2N3904" (at 102.235 56.896 0)
+    (property "Value" "MMBT3904T" (at 107.95 58.801 0)
+      (effects (font (size 1.27 1.27)) (justify left))
+    )
+    (property "Footprint" "Package_TO_SOT_SMD:SOT-523" (at 107.315 54.356 0)
+      (effects (font (size 1.27 1.27)) hide)
+    )
+    (property "Datasheet" "~" (at 102.235 56.896 0)
+      (effects (font (size 1.27 1.27)) hide)
+    )
+    (property "Mouser" "621-MMBT3904T-F" (at 102.235 56.896 0)
       (effects (font (size 1.27 1.27)) hide)
     )
@@
     )
   )
-  (symbol (lib_id "Transistor_BJT:2N3904") (at 100.33 154.305 0) (unit 1)
+  (symbol (lib_id "Device:Q_NPN_BEC") (at 100.33 154.305 0) (unit 1)
     (in_bom yes) (on_board yes) (dnp no) (fields_autoplaced)
     (property "Reference" "Q402" (at 106.045 153.67 0)
       (effects (font (size 1.27 1.27)) (justify left))
     )
-    (property "Value" "2N3904" (at 106.045 156.21 0)
-      (effects (font (size 1.27 1.27)) (justify left))
-    )
-    (property "Footprint" "Package_TO_SOT_THT:TO-92_Inline" (at 105.41 156.21 0)
-      (effects (font (size 1.27 1.27) italic) (justify left) hide)
-    )
-    (property "Datasheet" "https://www.onsemi.com/pub/Collateral/2N3903-D.PDF" (at 100.33 154.305 0)
-      (effects (font (size 1.27 1.27)) (justify left) hide)
-    )
-    (property "Mouser" "583-2N3904" (at 100.33 154.305 0)
-      (effects (font (size 1.27 1.27)) hide)
-    )
+    (property "Value" "MMBT3904T" (at 106.045 156.21 0)
+      (effects (font (size 1.27 1.27)) (justify left))
+    )
+    (property "Footprint" "Package_TO_SOT_SMD:SOT-523" (at 105.41 151.765 0)
+      (effects (font (size 1.27 1.27)) hide)
+    )
+    (property "Datasheet" "~" (at 100.33 154.305 0)
+      (effects (font (size 1.27 1.27)) hide)
+    )
+    (property "Mouser" "621-MMBT3904T-F" (at 100.33 154.305 0)
+      (effects (font (size 1.27 1.27)) hide)
+    )

Commit message: Update issue date.
Other:
- company: (c) 2024 Jason R. Thorpe.  See LICENSE. -> (c) 2024, 2025 Jason R. Thorpe.  See LICENSE.
Changed lines of the file:
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@@
   (title_block
     (title "CoPicoVision")
-    (date "2024-12-31")
+    (date "2025-01-23")
     (rev "3.0")
-    (company "(c) 2024 Jason R. Thorpe.  See LICENSE.")
+    (company "(c) 2024, 2025 Jason R. Thorpe.  See LICENSE.")
   )
   (junction (at 223.901 130.302) (diameter 0) (color 0 0 0 0)
