File: design-files/CoPicoVision_audio.kicad_sch (KiCad schematic)
At the start: 7 parts, among them J501 AudioJack3, Q501 KSD1616A, U501 SN76489AN

Commit message: BoM.
Parts:
- C102: value 10µF -> 22µF; Mouser (none) -> 647-RNS1C220MDS1
- C201: Mouser (none) -> 81-RCER71E104K0A2H3B
- C503: Mouser (none) -> 80-A750EQ477M1CAAE15
- Q501: Mouser (none) -> 512-KSD1616AGTA
Changed lines of the file:
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@@
+      (effects (font (size 1.27 1.27)) hide)
+    )
+    (property "Mouser" "80-A750EQ477M1CAAE15" (at 139.192 93.345 90)
       (effects (font (size 1.27 1.27)) hide)
     )
@@
       (effects (font (size 1.27 1.27)) (justify left))
     )
-    (property "Value" "10µF" (at 100.33 134.9629 0)
+    (property "Value" "22µF" (at 100.33 134.9629 0)
       (effects (font (size 1.27 1.27)) (justify left))
     )
@@
     )
     (property "Datasheet" "~" (at 97.028 133.604 0)
+      (effects (font (size 1.27 1.27)) hide)
+    )
+    (property "Mouser" "647-RNS1C220MDS1" (at 97.028 133.604 0)
       (effects (font (size 1.27 1.27)) hide)
     )
@@
     )
     (property "Datasheet" "https://www.mouser.com/datasheet/2/308/1/KSD1616A_D-2314918.pdf" (at 113.792 88.265 0)
+      (effects (font (size 1.27 1.27)) hide)
+    )
+    (property "Mouser" "512-KSD1616AGTA" (at 113.792 88.265 0)
       (effects (font (size 1.27 1.27)) hide)
     )
@@
       (effects (font (size 1.27 1.27)) hide)
     )
+    (property "Mouser" "81-RCER71E104K0A2H3B" (at 84.836 133.604 0)
+      (effects (font (size 1.27 1.27)) hide)
+    )

Commit message: Add title blocks.
Other:
- company: (none) -> (c) 2024 Jason R. Thorpe.  See LICENSE.
- title: (none) -> CoPicoVision
Changed lines of the file:
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@@
 (kicad_sch (version 20230121) (generator eeschema)
   (paper "A4")
+  (title_block
+    (title "CoPicoVision")
+    (date "2024-08-31")
+    (rev "0.1")
+    (company "(c) 2024 Jason R. Thorpe.  See LICENSE.")
+  )
   (junction (at 84.836 131.064) (diameter 0) (color 0 0 0 0)
   )
