File: design-files/CoPicoVision_audio.kicad_sch (KiCad schematic)
At the start: 7 parts, among them J501 AudioJack3, Q501 KSD1616A, U501 SN76489AN

Commit message: Use a vertical footprint for R501.
Parts:
- R501: footprint Resistor_THT:R_Axial_DIN0204_L3.6mm_D1.6mm_P5.08mm_Horizontal -> Resistor_THT:R_Axial_DIN0207_L6.3mm_D2.5mm_P2.54mm_Vertical
Changed lines of the file:
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@@
       (effects (font (size 1.27 1.27)) (justify left))
     )
-    (property "Footprint" "Resistor_THT:R_Axial_DIN0204_L3.6mm_D1.6mm_P5.08mm_Horizontal" (at 116.332 95.885 0)
+    (property "Footprint" "Resistor_THT:R_Axial_DIN0207_L6.3mm_D2.5mm_P2.54mm_Vertical" (at 116.332 95.885 0)
       (effects (font (size 1.27 1.27)) hide)
     )

Commit message: Add a 1.5K current limiting resistor between the SN76489AN audio output and the KSD1616A emitter-follower.
Parts:
- added R502: 1.5K, Resistor_THT:R_Axial_DIN0207_L6.3mm_D2.5mm_P2.54mm_Vertical, symbol Device:R_Small
Connections:
- net at Q501.3 (B): now also R502.2; no longer U501.7 (AUDIO_OUT)
- new net: R502.1, U501.7 (AUDIO_OUT)
Other:
- moved on the sheet: C503, J501, Q501, R501

Commit message: Add a 0.01uF cap to ground to the emitter-follower input to form a ~10KHz low-pass filter to try and tamp down the hissy noise.
Parts:
- added C101: 0.01µF, Capacitor_THT:C_Disc_D3.8mm_W2.6mm_P2.50mm, symbol Device:C_Small
Connections:
- net GND: now also C101.2
- net at Q501.3 (B): now also R502.1, C101.1; no longer R502.2
- net at U501.7 (AUDIO_OUT): now also R502.2; no longer R502.1
Other:
- note added: "~10KHz low-pass filter to reduce noise."
- moved on the sheet: R502
Changed lines of the file:
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@@
   (junction (at 163.322 93.345) (diameter 0) (color 0 0 0 0)
   )
+  (junction (at 114.173 88.265) (diameter 0) (color 0 0 0 0)
+  )
   (junction (at 84.836 136.144) (diameter 0) (color 0 0 0 0)
   )
   (junction (at 124.46 93.345) (diameter 0) (color 0 0 0 0)
   )
+  (junction (at 124.46 98.425) (diameter 0) (color 0 0 0 0)
+  )
   (wire (pts (xy 163.322 90.805) (xy 163.322 93.345))
     (stroke (width 0) (type default))
@@
     (stroke (width 0) (type default))
   )
+  (wire (pts (xy 114.173 98.425) (xy 124.46 98.425))
+    (stroke (width 0) (type default))
+  )
   (wire (pts (xy 84.836 131.064) (xy 97.028 131.064))
     (stroke (width 0) (type default))
@@
     (stroke (width 0) (type default))
   )
-  (wire (pts (xy 115.316 88.265) (xy 116.84 88.265))
+  (wire (pts (xy 114.173 88.265) (xy 116.84 88.265))
     (stroke (width 0) (type default))
   )
@@
     (stroke (width 0) (type default))
   )
-  (wire (pts (xy 103.759 88.265) (xy 110.236 88.265))
+  (wire (pts (xy 103.759 88.265) (xy 109.093 88.265))
+    (stroke (width 0) (type default))
+  )
+  (wire (pts (xy 114.173 88.265) (xy 114.173 92.964))
     (stroke (width 0) (type default))
   )
   (wire (pts (xy 84.836 136.144) (xy 97.028 136.144))
     (stroke (width 0) (type default))
+  )
+  (wire (pts (xy 114.173 98.044) (xy 114.173 98.425))
+    (stroke (width 0) (type default))
+  )
+  (text "~10KHz low-pass filter\nto reduce noise." (at 106.553 108.077 0)
+    (effects (font (size 1.27 1.27)) (justify left bottom))
   )
   (text "1/2 watt" (at 135.001 100.584 0)
@@
         (path "/d4d4c0fa-7a39-4b72-9fdb-c481b1e41ed4/6cf2d612-8129-4b9a-9cb3-eb8429f58846"
           (reference "#PWR0507") (unit 1)
+        )
+      )
+    )
+  )
+  (symbol (lib_id "Device:C_Small") (at 114.173 95.504 0) (unit 1)
+    (in_bom yes) (on_board yes) (dnp no)
+    (property "Reference" "C101" (at 116.459 94.869 0)
+      (effects (font (size 1.27 1.27)) (justify left))
+    )
+    (property "Value" "0.01µF" (at 116.459 97.409 0)
+      (effects (font (size 1.27 1.27)) (justify left))
+    )
+    (property "Footprint" "Capacitor_THT:C_Disc_D3.8mm_W2.6mm_P2.50mm" (at 114.173 95.504 0)
+      (effects (font (size 1.27 1.27)) hide)
+    )
+    (property "Datasheet" "~" (at 114.173 95.504 0)
+      (effects (font (size 1.27 1.27)) hide)
+    )
+    (property "Mouser" "81-RCER71H103K0A2H3B" (at 114.173 95.504 0)
+      (effects (font (size 1.27 1.27)) hide)
+    )
+    (pin "1")
+    (pin "2")
+    (instances
+      (project "CoPicoVision"
+        (path "/d4d4c0fa-7a39-4b72-9fdb-c481b1e41ed4"
+          (reference "C101") (unit 1)
+        )
+        (path "/d4d4c0fa-7a39-4b72-9fdb-c481b1e41ed4/e0ac0253-c368-4a00-80da-4eff7e9af602"
+          (reference "C413") (unit 1)
+        )
+        (path "/d4d4c0fa-7a39-4b72-9fdb-c481b1e41ed4/6cf2d612-8129-4b9a-9cb3-eb8429f58846"
+          (reference "C504") (unit 1)
         )
       )
@@
     )
   )
-  (symbol (lib_id "Device:R_Small") (at 112.776 88.265 90) (unit 1)
-    (in_bom yes) (on_board yes) (dnp no) (fields_autoplaced)
-    (property "Reference" "R502" (at 112.776 83.82 90)
-      (effects (font (size 1.27 1.27)))
-    )
-    (property "Value" "1.5K" (at 112.776 86.36 90)
-      (effects (font (size 1.27 1.27)))
-    )
-    (property "Footprint" "Resistor_THT:R_Axial_DIN0207_L6.3mm_D2.5mm_P2.54mm_Vertical" (at 112.776 88.265 0)
-      (effects (font (size 1.27 1.27)) hide)
-    )
-    (property "Datasheet" "~" (at 112.776 88.265 0)
-      (effects (font (size 1.27 1.27)) hide)
-    )
+  (symbol (lib_id "Device:R_Small") (at 111.633 88.265 270) (unit 1)
+    (in_bom yes) (on_board yes) (dnp no) (fields_autoplaced)
+    (property "Reference" "R502" (at 111.633 83.82 90)
+      (effects (font (size 1.27 1.27)))
+    )
+    (property "Value" "1.5K" (at 111.633 86.36 90)
+      (effects (font (size 1.27 1.27)))
+    )
+    (property "Footprint" "Resistor_THT:R_Axial_DIN0207_L6.3mm_D2.5mm_P2.54mm_Vertical" (at 111.633 88.265 0)
+      (effects (font (size 1.27 1.27)) hide)
+    )
+    (property "Datasheet" "~" (at 111.633 88.265 0)
+      (effects (font (size 1.27 1.27)) hide)
+    )

Commit message: Project update, and use a TL071 opamp for the audio output buffer.
Parts:
- removed C101: 0.01µF, Capacitor_THT:C_Disc_D3.8mm_W2.6mm_P2.50mm, symbol Device:C_Small
- removed Q501: KSD1616A, Package_TO_SOT_THT:TO-92L_Inline_Wide, symbol Device:Q_NPN_ECB
- removed R501: 100R, Resistor_THT:R_Axial_DIN0207_L6.3mm_D2.5mm_P2.54mm_Vertical, symbol Device:R_Small
- added C504: 2.2µF, Capacitor_THT:CP_Radial_D6.3mm_P2.50mm, symbol Device:C_Polarized_Small
- added R502: 10K, Resistor_SMD:R_0805_2012Metric_Pad1.20x1.40mm_HandSolder, symbol Device:R_Small
- added U502: TL071, Package_DIP:DIP-8_W7.62mm_Socket, symbol Amplifier_Operational:TL071
- C503: value 470µF -> 2.2µF
- R501: renamed from R502; value 1.5K -> 1K; footprint Resistor_THT:R_Axial_DIN0207_L6.3mm_D2.5mm_P2.54mm_Vertical -> Resistor_SMD:R_0805_2012Metric_Pad1.20x1.40mm_HandSolder
Connections:
- net GND: now also R502.2
- net VCC: now also U502.7 (V+)
- net at C503.1: now also R501.1
- net at J501.R, J501.T: now also C504.2; no longer C503.2
- new net: C503.2, R502.1, U502.3 (+)
- new net: C504.1, U502.2 (-), U502.6
- new net -5V: U502.4 (V-)
- no-connect marks 0 -> 2
Other:
- note removed: "1/2 watt"
- note removed: "~10KHz low-pass filter to reduce noise."
- moved on the sheet: C503, J501, R501

Commit message: All the bypass caps are now 0805s.
Parts:
- C201: footprint Capacitor_THT:C_Disc_D3.8mm_W2.6mm_P2.50mm -> Capacitor_SMD:C_0805_2012Metric_Pad1.18x1.45mm_HandSolder
Changed lines of the file:
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@@
       (effects (font (size 1.27 1.27)) (justify left))
     )
-    (property "Footprint" "Capacitor_THT:C_Disc_D3.8mm_W2.6mm_P2.50mm" (at 84.836 133.604 0)
+    (property "Footprint" "Capacitor_SMD:C_0805_2012Metric_Pad1.18x1.45mm_HandSolder" (at 84.836 133.604 0)
       (effects (font (size 1.27 1.27)) hide)
     )

Commit message: Put the AY-3-8910 on the schematic.  Need to make some more room on the board.
Parts:
- added C201 (x2): 0.1µF, Capacitor_SMD:C_0805_2012Metric_Pad1.18x1.45mm_HandSolder, symbol Device:C_Small
- added R503, R504, R505: 1K, Resistor_SMD:R_0805_2012Metric_Pad1.20x1.40mm_HandSolder, symbol Device:R_Small
- added U503: AY-3-8910, Package_DIP:DIP-40_W15.24mm, symbol jrt-ICs:AY-3-8910
- added U504: 74HCT02, Package_SO:SOIC-14_3.9x8.7mm_P1.27mm, symbol 74xx:74HCT02
Connections:
- net CPUCLK: now also U503.22 (CLOCK)
- net D0: now also U503.37 (DA0)
- net D1: now also U503.36 (DA1)
- net D3: now also U503.34 (DA3)
- net D4: now also U503.33 (DA4)
- net D5: now also U503.32 (DA5)
- net D7: now also U503.30 (DA7), U503.31 (DA6)
- net GND: now also C201.2, C201.2, U503.1 (GND), U504.11, U504.12, U504.7 (GND), U504.8, U504.9
- net VCC: now also C201.1, C201.1, U503.25 (A8), U503.28 (BC2), U503.40 (VCC), U504.14 (VCC)
- net at C503.1, R501.1: now also R503.1, R504.1, R505.1
- new net: U503.29 (BC1), U504.1
- new net: R505.2, U503.38 (OUT_C)
- new net: U503.27 (BDIR), U504.4
- new net: R503.2, U503.4 (OUT_A)
- new net: R504.2, U503.3 (OUT_B)
- new net A0: U504.2
- new net ~{AYSEL}: U503.24 (~{A9}), U504.3, U504.5
- new net ~{RESET}: U503.23 (~{RESET})
- new net ~{WR}: U504.6
- no-connect marks 2 -> 22
Other:
- moved on the sheet: C102, C201, C503, C504, J501, R501, R502, U501, U502

Commit message: Put the AY-3-8910 on the board, clarify part numbers for the 74xx chips to ensure the correct SOIC footprints.
Parts:
- U503: footprint Package_DIP:DIP-40_W15.24mm -> Package_DIP:DIP-40_W15.24mm_Socket
- U504: value 74HCT02 -> SN74HCT02D
Connections:
- net D2: now also U503.35 (DA2)
Changed lines of the file:
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@@
     )
   )
-  (global_label "D2" (shape bidirectional) (at 51.054 91.059 180) (fields_autoplaced)
+  (global_label "D2" (shape bidirectional) (at 51.181 91.059 180) (fields_autoplaced)
     (effects (font (size 1.27 1.27)) (justify right))
-    (property "Intersheetrefs" "${INTERSHEET_REFS}" (at 44.5574 91.059 0)
+    (property "Intersheetrefs" "${INTERSHEET_REFS}" (at 44.6844 91.059 0)
       (effects (font (size 1.27 1.27)) (justify right) hide)
     )
@@
       (effects (font (size 1.27 1.27)))
     )
-    (property "Value" "74HCT02" (at 28.956 100.711 0)
+    (property "Value" "SN74HCT02D" (at 28.956 100.711 0)
       (effects (font (size 1.27 1.27)))
     )
@@
       (effects (font (size 1.27 1.27)))
     )
-    (property "Value" "74HCT02" (at 87.63 184.15 0)
+    (property "Value" "SN74HCT02D" (at 87.63 184.15 0)
       (effects (font (size 1.27 1.27)))
     )
@@
       (effects (font (size 1.27 1.27)))
     )
-    (property "Value" "74HCT02" (at 28.956 113.411 0)
+    (property "Value" "SN74HCT02D" (at 28.956 113.411 0)
       (effects (font (size 1.27 1.27)))
     )
@@
       (effects (font (size 1.27 1.27)) (justify left))
     )
-    (property "Footprint" "Package_DIP:DIP-40_W15.24mm" (at 66.421 105.029 0)
+    (property "Footprint" "Package_DIP:DIP-40_W15.24mm_Socket" (at 66.421 105.029 0)
       (effects (font (size 1.27 1.27)) hide)
     )
@@
       (effects (font (size 1.27 1.27)) (justify left))
     )
-    (property "Value" "74HCT02" (at 119.126 180.594 0)
+    (property "Value" "SN74HCT02D" (at 119.126 180.594 0)
       (effects (font (size 1.27 1.27)) (justify left))
     )
@@
       (effects (font (size 1.27 1.27)))
     )
-    (property "Value" "74HCT02" (at 87.63 170.18 0)
-      (effects (font (size 1.27 1.27)))
-    )
+    (property "Value" "SN74HCT02D" (at 87.63 170.18 0)
+      (effects (font (size 1.27 1.27)))
+    )

Commit message: I think that's the whole right side of the board now routed.
Connections:
- net D6: now also U503.31 (DA6)
- net D7: no longer U503.31 (DA6)
Changed lines of the file:
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@@
     )
   )
-  (global_label "D7" (shape bidirectional) (at 51.181 101.219 180) (fields_autoplaced)
+  (global_label "D6" (shape bidirectional) (at 51.181 101.219 180) (fields_autoplaced)
     (effects (font (size 1.27 1.27)) (justify right))
     (property "Intersheetrefs" "${INTERSHEET_REFS}" (at 44.6844 101.219 0)
