File: design-files/CoPicoVision_audio.kicad_sch (KiCad schematic)
At the start: 16 parts, among them J501 AudioJack3, U501 SN76489AN, U502 TL071, U503 AY-3-8910, U504 SN74HCT02D

Commit message: Update Mouser part numbers / data sheet links.
Parts:
- U502: Mouser (none) -> 595-TL071CP
- U504: Mouser (none) -> 595-SN74HCT02DR
Changed lines of the file:
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@@
+      (effects (font (size 1.27 1.27)) hide)
+    )
+    (property "Mouser" "595-SN74HCT02DR" (at 28.956 105.41 0)
+      (effects (font (size 1.27 1.27)) hide)
+    )
+    (property "Field5" "" (at 28.956 105.41 0)
       (effects (font (size 1.27 1.27)) hide)
     )
@@
       (effects (font (size 1.27 1.27)) hide)
     )
+    (property "Mouser" "595-SN74HCT02DR" (at 87.63 189.484 0)
+      (effects (font (size 1.27 1.27)) hide)
+    )
+    (property "Field5" "" (at 87.63 189.484 0)
+      (effects (font (size 1.27 1.27)) hide)
+    )
     (pin "1")
     (pin "2")
@@
     )
     (property "Datasheet" "http://www.ti.com/lit/gpn/sn74hct02" (at 28.956 118.237 0)
+      (effects (font (size 1.27 1.27)) hide)
+    )
+    (property "Mouser" "595-SN74HCT02DR" (at 28.956 118.237 0)
+      (effects (font (size 1.27 1.27)) hide)
+    )
+    (property "Field5" "" (at 28.956 118.237 0)
       (effects (font (size 1.27 1.27)) hide)
     )
@@
       (effects (font (size 1.27 1.27)) hide)
     )
+    (property "Mouser" "595-SN74HCT02DR" (at 112.522 178.689 0)
+      (effects (font (size 1.27 1.27)) hide)
+    )
+    (property "Field5" "" (at 112.522 178.689 0)
+      (effects (font (size 1.27 1.27)) hide)
+    )
     (pin "1")
     (pin "2")
@@
       (effects (font (size 1.27 1.27)) hide)
     )
+    (property "Mouser" "595-TL071CP" (at 147.066 44.577 0)
+      (effects (font (size 1.27 1.27)) hide)
+    )
     (pin "1")
     (pin "2")
@@
       (effects (font (size 1.27 1.27)) hide)
     )
+    (property "Mouser" "595-SN74HCT02DR" (at 87.63 175.133 0)
+      (effects (font (size 1.27 1.27)) hide)
+    )
+    (property "Field5" "" (at 87.63 175.133 0)
+      (effects (font (size 1.27 1.27)) hide)
+    )

Commit message: Add / correct a bunch of Mouser part numbers for the BoM.
Parts:
- C201: Mouser 81-RCER71E104K0A2H3B -> 581-KAM21BR71H104JT
- C503, C504: Mouser 80-A750EQ477M1CAAE15 -> 667-ECA-2DM2R2I
- R501, R503, R504, R505: Mouser (none) -> 71-CRCW0805-1.0K-E3
- R502: Mouser (none) -> 71-CRCW0805-10K-E3
Changed lines of the file:
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@@
+      (effects (font (size 1.27 1.27)) hide)
+    )
+    (property "Mouser" "71-CRCW0805-1.0K-E3" (at 97.155 136.779 90)
       (effects (font (size 1.27 1.27)) hide)
     )
@@
       (effects (font (size 1.27 1.27)) hide)
     )
-    (property "Mouser" "80-A750EQ477M1CAAE15" (at 128.905 42.037 90)
+    (property "Mouser" "667-ECA-2DM2R2I" (at 128.905 42.037 90)
       (effects (font (size 1.27 1.27)) hide)
     )
@@
       (effects (font (size 1.27 1.27)) hide)
     )
+    (property "Mouser" "71-CRCW0805-1.0K-E3" (at 86.995 131.699 90)
+      (effects (font (size 1.27 1.27)) hide)
+    )
     (pin "1")
     (pin "2")
@@
       (effects (font (size 1.27 1.27)) hide)
     )
+    (property "Mouser" "71-CRCW0805-1.0K-E3" (at 92.075 134.239 90)
+      (effects (font (size 1.27 1.27)) hide)
+    )
     (pin "1")
     (pin "2")
@@
       (effects (font (size 1.27 1.27)) hide)
     )
-    (property "Mouser" "80-A750EQ477M1CAAE15" (at 158.242 44.577 90)
+    (property "Mouser" "667-ECA-2DM2R2I" (at 158.242 44.577 90)
       (effects (font (size 1.27 1.27)) hide)
     )
@@
       (effects (font (size 1.27 1.27)) hide)
     )
+    (property "Mouser" "71-CRCW0805-10K-E3" (at 132.588 44.577 0)
+      (effects (font (size 1.27 1.27)) hide)
+    )
     (pin "1")
     (pin "2")
@@
       (effects (font (size 1.27 1.27)) hide)
     )
+    (property "Mouser" "71-CRCW0805-1.0K-E3" (at 72.136 42.037 90)
+      (effects (font (size 1.27 1.27)) hide)
+    )
     (pin "1")
     (pin "2")
@@
       (effects (font (size 1.27 1.27)) hide)
     )
-    (property "Mouser" "81-RCER71E104K0A2H3B" (at 16.129 162.814 0)
+    (property "Mouser" "581-KAM21BR71H104JT" (at 16.129 162.814 0)
       (effects (font (size 1.27 1.27)) hide)
     )
@@
       (effects (font (size 1.27 1.27)) hide)
     )
-    (property "Mouser" "81-RCER71E104K0A2H3B" (at 51.816 162.814 0)
+    (property "Mouser" "581-KAM21BR71H104JT" (at 51.816 162.814 0)
       (effects (font (size 1.27 1.27)) hide)
     )
@@
       (effects (font (size 1.27 1.27)) hide)
     )
-    (property "Mouser" "81-RCER71E104K0A2H3B" (at 39.497 162.814 0)
-      (effects (font (size 1.27 1.27)) hide)
-    )
+    (property "Mouser" "581-KAM21BR71H104JT" (at 39.497 162.814 0)
+      (effects (font (size 1.27 1.27)) hide)
+    )
