File: design-files/CoPicoVision_memory.kicad_sch (KiCad schematic)
At the start: 9 parts, among them U103 74ACT05, U201 GAL22V10, U202 GAL22V10, U203 AT28C64, U204 AS6C6264

Commit message: All the bypass caps are now 0805s.
Parts:
- C201, C202, C203, C204: footprint Capacitor_THT:C_Disc_D3.8mm_W2.6mm_P2.50mm -> Capacitor_SMD:C_0805_2012Metric_Pad1.18x1.45mm_HandSolder
Changed lines of the file:
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@@
       (effects (font (size 1.27 1.27)) (justify left))
     )
-    (property "Footprint" "Capacitor_THT:C_Disc_D3.8mm_W2.6mm_P2.50mm" (at 110.871 158.496 0)
+    (property "Footprint" "Capacitor_SMD:C_0805_2012Metric_Pad1.18x1.45mm_HandSolder" (at 110.871 158.496 0)
       (effects (font (size 1.27 1.27)) hide)
     )
@@
       (effects (font (size 1.27 1.27)) (justify left))
     )
-    (property "Footprint" "Capacitor_THT:C_Disc_D3.8mm_W2.6mm_P2.50mm" (at 87.884 158.496 0)
+    (property "Footprint" "Capacitor_SMD:C_0805_2012Metric_Pad1.18x1.45mm_HandSolder" (at 87.884 158.496 0)
       (effects (font (size 1.27 1.27)) hide)
     )
@@
       (effects (font (size 1.27 1.27)) (justify left))
     )
-    (property "Footprint" "Capacitor_THT:C_Disc_D3.8mm_W2.6mm_P2.50mm" (at 76.454 158.496 0)
+    (property "Footprint" "Capacitor_SMD:C_0805_2012Metric_Pad1.18x1.45mm_HandSolder" (at 76.454 158.496 0)
       (effects (font (size 1.27 1.27)) hide)
     )
@@
       (effects (font (size 1.27 1.27)) (justify left))
     )
-    (property "Footprint" "Capacitor_THT:C_Disc_D3.8mm_W2.6mm_P2.50mm" (at 99.441 158.496 0)
+    (property "Footprint" "Capacitor_SMD:C_0805_2012Metric_Pad1.18x1.45mm_HandSolder" (at 99.441 158.496 0)
       (effects (font (size 1.27 1.27)) hide)
     )

Commit message: Controller section is mostly SMT now.
Parts:
- U103: footprint Package_DIP:DIP-14_W7.62mm_Socket -> Package_SO:SOIC-14_3.9x8.7mm_P1.27mm
Changed lines of the file:
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@@
       (effects (font (size 1.27 1.27)))
     )
-    (property "Footprint" "Package_DIP:DIP-14_W7.62mm_Socket" (at 143.129 106.299 0)
+    (property "Footprint" "Package_SO:SOIC-14_3.9x8.7mm_P1.27mm" (at 143.129 106.299 0)
       (effects (font (size 1.27 1.27)) hide)
     )

Commit message: Add the SGM memory logic chips, clean out board routing on the left half of the board.
Parts:
- added C205, C206: 0.1µF, Capacitor_SMD:C_0805_2012Metric_Pad1.18x1.45mm_HandSolder, symbol Device:C_Small
- added U205: 74HCT08, Package_SO:SOIC-14_3.9x8.7mm_P1.27mm, symbol 74xx:74LS08
- added U206: 74HCT74, Package_SO:SOIC-14_3.9x8.7mm_P1.27mm, symbol 74xx:74HC74
- U204: value AS6C6264 -> AS6C62256; footprint Package_DIP:DIP-28_W15.24mm_Socket -> Package_SO:SOIC-28W_7.5x17.9mm_P1.27mm; symbol jrt-ICs:AS6C6264 -> Memory_RAM:CY62256-70PC
Connections:
- net A10: now also U205.1
- net A11: now also U205.4
- net A12: now also U205.12
- net A13: now also U204.26 (A13)
- net A14: now also U204.1 (A14)
- net D0: now also U206.2 (D)
- net D1: now also U206.12 (D)
- net GND: now also C205.2, C206.2, U205.10, U205.7 (GND), U205.9, U206.7 (GND); no longer U204.2 (A12), U204.21 (A10), U204.23 (A11)
- net VCC: now also C205.1, C206.1, U205.14 (VCC), U206.13 (~{R}), U206.14 (VCC), U206.4 (~{S}); no longer U204.26 (CE2)
- new net: U204.21 (A10), U205.3
- new net: U204.2 (A12), U205.11
- new net: U204.23 (A11), U205.6
- new net ROMEN: U206.9 (Q)
- new net XRAMEN: U205.13, U205.2, U205.5, U206.5 (Q)
- new net ~{FF1WSEL}: U206.3 (C)
- new net ~{FF2WSEL}: U206.11 (C)
- new net ~{RESET}: U206.1 (~{R}), U206.10 (~{S})
- no-connect marks 18 -> 21

Commit message: Re-pin the inputs of the IODEC GAL, and make it take A0-A7 in prep for SGM additions.
Connections:
- net A0: now also U201.11 (I11)
- net A1: now also U201.10 (I10)
- net A2: now also U201.9 (I9)
- net A3: now also U201.8 (I8)
- net A4: now also U201.7 (I7)
- net A5: now also U201.6 (I6); no longer U201.3 (I3)
- net A6: now also U201.5 (I5); no longer U201.4 (I4)
- net A7: now also U201.4 (I4); no longer U201.5 (I5)
- no-connect marks 21 -> 16

Commit message: Rearrange the MEMDEC GAL to work better with the new board layout.
Connections:
- net A13: now also U202.9 (I9); no longer U202.5 (I5)
- net A14: now also U202.10 (I10); no longer U202.6 (I6)
- net A15: now also U202.11 (I11); no longer U202.7 (I7)
- net ~{CRT8SEL}: now also U202.17 (IO4); no longer U202.19 (IO6)
- net ~{CRTASEL}: now also U202.16 (IO3); no longer U202.18 (IO5)
- net ~{CRTCSEL}: now also U202.15 (IO2); no longer U202.17 (IO4)
- net ~{CRTESEL}: now also U202.14 (IO1); no longer U202.16 (IO3)
- net ~{M1}: now also U202.3 (I3); no longer U202.2 (I2)
- net ~{MREQ}: now also U202.5 (I5); no longer U202.3 (I3)
- net ~{RAMSEL}: now also U202.22 (IO9); no longer U202.20 (IO7)
- net ~{RFSH}: now also U202.2 (I2); no longer U202.4 (I4)
- net ~{WR}: now also U202.6 (I6)
- net at U103.1: now also U202.21 (IO8); no longer U202.15 (IO2)
- no-connect marks 16 -> 15
Changed lines of the file:
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@@
   (junction (at 99.441 155.956) (diameter 0) (color 0 0 0 0)
   )
-  (no_connect (at 95.885 124.079))
-  (no_connect (at 121.285 121.539))
-  (no_connect (at 121.285 103.759))
-  (no_connect (at 95.885 129.159))
   (no_connect (at 121.158 47.752))
   (no_connect (at 95.885 131.699))
   (no_connect (at 95.758 52.832))
-  (no_connect (at 95.885 126.619))
+  (no_connect (at 121.285 113.919))
   (no_connect (at 95.758 75.692))
   (no_connect (at 121.158 50.292))
   (no_connect (at 95.885 121.539))
   (no_connect (at 161.925 32.258))
-  (no_connect (at 121.285 124.079))
+  (no_connect (at 95.885 118.999))
+  (no_connect (at 121.285 118.999))
+  (no_connect (at 121.285 116.459))
   (no_connect (at 121.158 52.832))
   (no_connect (at 161.925 59.309))
+  (no_connect (at 95.885 111.379))
   (no_connect (at 173.863 161.671))
   (wire (pts (xy 154.305 42.164) (xy 154.305 37.338))
@@
     (stroke (width 0) (type default))
   )
+  (wire (pts (xy 135.509 106.299) (xy 135.509 121.539))
+    (stroke (width 0) (type default))
+  )
   (wire (pts (xy 121.412 166.497) (xy 121.412 163.957))
     (stroke (width 0) (type default))
@@
     (stroke (width 0) (type default))
   )
+  (wire (pts (xy 135.509 121.539) (xy 121.285 121.539))
+    (stroke (width 0) (type default))
+  )
   (wire (pts (xy 99.441 161.036) (xy 110.871 161.036))
     (stroke (width 0) (type default))
@@
   )
   (wire (pts (xy 99.441 155.956) (xy 110.871 155.956))
-    (stroke (width 0) (type default))
-  )
-  (wire (pts (xy 121.285 106.299) (xy 135.509 106.299))
     (stroke (width 0) (type default))
   )
@@
     )
   )
-  (global_label "~{RAMSEL}" (shape output) (at 121.285 118.999 0) (fields_autoplaced)
-    (effects (font (size 1.27 1.27)) (justify left))
-    (property "Intersheetrefs" "${INTERSHEET_REFS}" (at 131.3874 118.999 0)
+  (global_label "~{RAMSEL}" (shape output) (at 121.285 124.079 0) (fields_autoplaced)
+    (effects (font (size 1.27 1.27)) (justify left))
+    (property "Intersheetrefs" "${INTERSHEET_REFS}" (at 131.3874 124.079 0)
       (effects (font (size 1.27 1.27)) (justify left) hide)
     )
@@
     )
   )
-  (global_label "~{CRTASEL}" (shape output) (at 121.285 113.919 0) (fields_autoplaced)
-    (effects (font (size 1.27 1.27)) (justify left))
-    (property "Intersheetrefs" "${INTERSHEET_REFS}" (at 132.1736 113.919 0)
+  (global_label "~{CRTASEL}" (shape output) (at 121.285 108.839 0) (fields_autoplaced)
+    (effects (font (size 1.27 1.27)) (justify left))
+    (property "Intersheetrefs" "${INTERSHEET_REFS}" (at 132.1736 108.839 0)
       (effects (font (size 1.27 1.27)) (justify left) hide)
     )
@@
     )
   )
-  (global_label "A13" (shape input) (at 95.885 113.919 180) (fields_autoplaced)
-    (effects (font (size 1.27 1.27)) (justify right))
-    (property "Intersheetrefs" "${INTERSHEET_REFS}" (at 89.4716 113.919 0)
+  (global_label "A13" (shape input) (at 95.885 124.079 180) (fields_autoplaced)
+    (effects (font (size 1.27 1.27)) (justify right))
+    (property "Intersheetrefs" "${INTERSHEET_REFS}" (at 89.4716 124.079 0)
       (effects (font (size 1.27 1.27)) (justify right) hide)
     )
@@
     )
   )
-  (global_label "~{M1}" (shape input) (at 95.885 106.299 180) (fields_autoplaced)
-    (effects (font (size 1.27 1.27)) (justify right))
-    (property "Intersheetrefs" "${INTERSHEET_REFS}" (at 90.3183 106.299 0)
+  (global_label "~{M1}" (shape input) (at 95.885 108.839 180) (fields_autoplaced)
+    (effects (font (size 1.27 1.27)) (justify right))
+    (property "Intersheetrefs" "${INTERSHEET_REFS}" (at 90.3183 108.839 0)
       (effects (font (size 1.27 1.27)) (justify right) hide)
     )
@@
     )
   )
-  (global_label "A14" (shape input) (at 95.885 116.459 180) (fields_autoplaced)
-    (effects (font (size 1.27 1.27)) (justify right))
-    (property "Intersheetrefs" "${INTERSHEET_REFS}" (at 89.4716 116.459 0)
+  (global_label "A14" (shape input) (at 95.885 126.619 180) (fields_autoplaced)
+    (effects (font (size 1.27 1.27)) (justify right))
+    (property "Intersheetrefs" "${INTERSHEET_REFS}" (at 89.4716 126.619 0)
       (effects (font (size 1.27 1.27)) (justify right) hide)
     )
@@
     )
   )
+  (global_label "~{WR}" (shape input) (at 95.885 116.459 180) (fields_autoplaced)
+    (effects (font (size 1.27 1.27)) (justify right))
+    (property "Intersheetrefs" "${INTERSHEET_REFS}" (at 90.2578 116.459 0)
+      (effects (font (size 1.27 1.27)) (justify right) hide)
+    )
+  )
   (global_label "A7" (shape input) (at 95.758 55.372 180) (fields_autoplaced)
     (effects (font (size 1.27 1.27)) (justify right))
@@
     )
   )
-  (global_label "~{CRTESEL}" (shape output) (at 121.285 108.839 0) (fields_autoplaced)
-    (effects (font (size 1.27 1.27)) (justify left))
-    (property "Intersheetrefs" "${INTERSHEET_REFS}" (at 132.234 108.839 0)
+  (global_label "~{CRTESEL}" (shape output) (at 121.285 103.759 0) (fields_autoplaced)
+    (effects (font (size 1.27 1.27)) (justify left))
+    (property "Intersheetrefs" "${INTERSHEET_REFS}" (at 132.234 103.759 0)
       (effects (font (size 1.27 1.27)) (justify left) hide)
     )
@@
     )
   )
-  (global_label "~{CRTCSEL}" (shape output) (at 121.285 111.379 0) (fields_autoplaced)
-    (effects (font (size 1.27 1.27)) (justify left))
-    (property "Intersheetrefs" "${INTERSHEET_REFS}" (at 132.355 111.379 0)
-      (effects (font (size 1.27 1.27)) (justify left) hide)
-    )
-  )
-  (global_label "~{RFSH}" (shape input) (at 95.885 111.379 180) (fields_autoplaced)
-    (effects (font (size 1.27 1.27)) (justify right))
-    (property "Intersheetrefs" "${INTERSHEET_REFS}" (at 88.0806 111.379 0)
-      (effects (font (size 1.27 1.27)) (justify right) hide)
-    )
-  )
-  (global_label "A15" (shape input) (at 95.885 118.999 180) (fields_autoplaced)
-    (effects (font (size 1.27 1.27)) (justify right))
-    (property "Intersheetrefs" "${INTERSHEET_REFS}" (at 89.4716 118.999 0)
+  (global_label "~{CRTCSEL}" (shape output) (at 121.285 106.299 0) (fields_autoplaced)
+    (effects (font (size 1.27 1.27)) (justify left))
+    (property "Intersheetrefs" "${INTERSHEET_REFS}" (at 132.355 106.299 0)
+      (effects (font (size 1.27 1.27)) (justify left) hide)
+    )
+  )
+  (global_label "~{RFSH}" (shape input) (at 95.885 106.299 180) (fields_autoplaced)
+    (effects (font (size 1.27 1.27)) (justify right))
+    (property "Intersheetrefs" "${INTERSHEET_REFS}" (at 88.0806 106.299 0)
+      (effects (font (size 1.27 1.27)) (justify right) hide)
+    )
+  )
+  (global_label "A15" (shape input) (at 95.885 129.159 180) (fields_autoplaced)
+    (effects (font (size 1.27 1.27)) (justify right))
+    (property "Intersheetrefs" "${INTERSHEET_REFS}" (at 89.4716 129.159 0)
       (effects (font (size 1.27 1.27)) (justify right) hide)
     )
@@
     )
   )
-  (global_label "~{MREQ}" (shape input) (at 95.885 108.839 180) (fields_autoplaced)
-    (effects (font (size 1.27 1.27)) (justify right))
-    (property "Intersheetrefs" "${INTERSHEET_REFS}" (at 87.7783 108.839 0)
-      (effects (font (size 1.27 1.27)) (justify right) hide)
-    )
-  )
-  (global_label "~{CRT8SEL}" (shape output) (at 121.285 116.459 0) (fields_autoplaced)
-    (effects (font (size 1.27 1.27)) (justify left))
-    (property "Intersheetrefs" "${INTERSHEET_REFS}" (at 132.2945 116.459 0)
-      (effects (font (size 1.27 1.27)) (justify left) hide)
-    )
+  (global_label "~{MREQ}" (shape input) (at 95.885 113.919 180) (fields_autoplaced)
+    (effects (font (size 1.27 1.27)) (justify right))
+    (property "Intersheetrefs" "${INTERSHEET_REFS}" (at 87.7783 113.919 0)
+      (effects (font (size 1.27 1.27)) (justify right) hide)
+    )
+  )
+  (global_label "~{CRT8SEL}" (shape output) (at 121.285 111.379 0) (fields_autoplaced)
+    (effects (font (size 1.27 1.27)) (justify left))
+    (property "Intersheetrefs" "${INTERSHEET_REFS}" (at 132.2945 111.379 0)
+      (effects (font (size 1.27 1.27)) (justify left) hide)
+    )

Commit message: Add the XRAMEN and ROMEN signals to the MEMDEC GAL.
Connections:
- net ROMEN: now also U202.8 (I8)
- net XRAMEN: now also U202.7 (I7)
- no-connect marks 15 -> 13
Changed lines of the file:
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@@
   (no_connect (at 95.758 75.692))
   (no_connect (at 121.158 50.292))
-  (no_connect (at 95.885 121.539))
   (no_connect (at 161.925 32.258))
-  (no_connect (at 95.885 118.999))
   (no_connect (at 121.285 118.999))
   (no_connect (at 121.285 116.459))
@@
     )
   )
+  (global_label "XRAMEN" (shape input) (at 95.885 118.999 180) (fields_autoplaced)
+    (effects (font (size 1.27 1.27)) (justify right))
+    (property "Intersheetrefs" "${INTERSHEET_REFS}" (at 85.4802 118.999 0)
+      (effects (font (size 1.27 1.27)) (justify right) hide)
+    )
+  )
   (global_label "D6" (shape bidirectional) (at 213.995 116.84 0) (fields_autoplaced)
     (effects (font (size 1.27 1.27)) (justify left))
@@
       (effects (font (size 1.27 1.27)) (justify right) hide)
     )
+  )
+  (global_label "ROMEN" (shape input) (at 95.885 121.539 180) (fields_autoplaced)
+    (effects (font (size 1.27 1.27)) (justify right))
+    (property "Intersheetrefs" "${INTERSHEET_REFS}" (at 86.4478 121.539 0)
+      (effects (font (size 1.27 1.27)) (justify right) hide)
+    )

Commit message: Add all of the SGM IODEC signals and re-pin the outputs to work better with the new board layout.
Connections:
- net ~{C1WSEL}: now also U201.22 (IO9); no longer U201.18 (IO5)
- net ~{C2WSEL}: now also U201.23 (IO10); no longer U201.19 (IO6)
- net ~{CRSEL}: now also U201.21 (IO8); no longer U201.17 (IO4)
- net ~{FF1WSEL}: now also U201.19 (IO6)
- net ~{FF2WSEL}: now also U201.20 (IO7)
- net ~{SNWSEL}: now also U201.14 (IO1); no longer U201.23 (IO10)
- net ~{VDPEN}: now also U201.16 (IO3); no longer U201.20 (IO7)
- net ~{VDPRSEL}: now also U201.18 (IO5); no longer U201.22 (IO9)
- net ~{VDPWSEL}: now also U201.17 (IO4); no longer U201.21 (IO8)
- net ~{AYSEL}: now reaches U201.15 (IO2)
- no-connect marks 13 -> 10
Changed lines of the file:
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@@
   (junction (at 99.441 155.956) (diameter 0) (color 0 0 0 0)
   )
-  (no_connect (at 121.158 47.752))
   (no_connect (at 95.885 131.699))
   (no_connect (at 95.758 52.832))
   (no_connect (at 121.285 113.919))
   (no_connect (at 95.758 75.692))
-  (no_connect (at 121.158 50.292))
   (no_connect (at 161.925 32.258))
   (no_connect (at 121.285 118.999))
   (no_connect (at 121.285 116.459))
-  (no_connect (at 121.158 52.832))
   (no_connect (at 161.925 59.309))
   (no_connect (at 95.885 111.379))
@@
     )
   )
-  (global_label "~{VDPWSEL}" (shape output) (at 121.158 65.532 0) (fields_autoplaced)
-    (effects (font (size 1.27 1.27)) (justify left))
-    (property "Intersheetrefs" "${INTERSHEET_REFS}" (at 132.5304 65.532 0)
+  (global_label "~{VDPWSEL}" (shape output) (at 121.158 55.372 0) (fields_autoplaced)
+    (effects (font (size 1.27 1.27)) (justify left))
+    (property "Intersheetrefs" "${INTERSHEET_REFS}" (at 132.5304 55.372 0)
       (effects (font (size 1.27 1.27)) (justify left) hide)
     )
@@
     )
   )
-  (global_label "~{C1WSEL}" (shape output) (at 121.158 57.912 0) (fields_autoplaced)
-    (effects (font (size 1.27 1.27)) (justify left))
-    (property "Intersheetrefs" "${INTERSHEET_REFS}" (at 131.3813 57.912 0)
+  (global_label "~{C1WSEL}" (shape output) (at 121.158 68.072 0) (fields_autoplaced)
+    (effects (font (size 1.27 1.27)) (justify left))
+    (property "Intersheetrefs" "${INTERSHEET_REFS}" (at 131.3813 68.072 0)
       (effects (font (size 1.27 1.27)) (justify left) hide)
     )
@@
     )
   )
-  (global_label "~{CRSEL}" (shape output) (at 121.158 55.372 0) (fields_autoplaced)
-    (effects (font (size 1.27 1.27)) (justify left))
-    (property "Intersheetrefs" "${INTERSHEET_REFS}" (at 129.9904 55.372 0)
+  (global_label "~{CRSEL}" (shape output) (at 121.158 65.532 0) (fields_autoplaced)
+    (effects (font (size 1.27 1.27)) (justify left))
+    (property "Intersheetrefs" "${INTERSHEET_REFS}" (at 129.9904 65.532 0)
       (effects (font (size 1.27 1.27)) (justify left) hide)
     )
@@
     )
   )
-  (global_label "~{VDPEN}" (shape output) (at 121.158 62.992 0) (fields_autoplaced)
-    (effects (font (size 1.27 1.27)) (justify left))
-    (property "Intersheetrefs" "${INTERSHEET_REFS}" (at 130.1719 62.992 0)
+  (global_label "~{VDPEN}" (shape output) (at 121.158 52.832 0) (fields_autoplaced)
+    (effects (font (size 1.27 1.27)) (justify left))
+    (property "Intersheetrefs" "${INTERSHEET_REFS}" (at 130.1719 52.832 0)
       (effects (font (size 1.27 1.27)) (justify left) hide)
     )
@@
     )
   )
+  (global_label "~{FF2WSEL}" (shape output) (at 121.158 62.992 0) (fields_autoplaced)
+    (effects (font (size 1.27 1.27)) (justify left))
+    (property "Intersheetrefs" "${INTERSHEET_REFS}" (at 132.2885 62.992 0)
+      (effects (font (size 1.27 1.27)) (justify left) hide)
+    )
+  )
   (global_label "A2" (shape input) (at 95.758 68.072 180) (fields_autoplaced)
     (effects (font (size 1.27 1.27)) (justify right))
@@
     )
   )
+  (global_label "~{FF1WSEL}" (shape output) (at 121.158 60.452 0) (fields_autoplaced)
+    (effects (font (size 1.27 1.27)) (justify left))
+    (property "Intersheetrefs" "${INTERSHEET_REFS}" (at 132.2885 60.452 0)
+      (effects (font (size 1.27 1.27)) (justify left) hide)
+    )
+  )
   (global_label "D6" (shape bidirectional) (at 213.995 116.84 0) (fields_autoplaced)
     (effects (font (size 1.27 1.27)) (justify left))
@@
     )
   )
-  (global_label "~{SNWSEL}" (shape output) (at 121.158 70.612 0) (fields_autoplaced)
-    (effects (font (size 1.27 1.27)) (justify left))
-    (property "Intersheetrefs" "${INTERSHEET_REFS}" (at 131.4418 70.612 0)
+  (global_label "~{SNWSEL}" (shape output) (at 121.158 47.752 0) (fields_autoplaced)
+    (effects (font (size 1.27 1.27)) (justify left))
+    (property "Intersheetrefs" "${INTERSHEET_REFS}" (at 131.4418 47.752 0)
       (effects (font (size 1.27 1.27)) (justify left) hide)
     )
@@
     )
   )
-  (global_label "~{C2WSEL}" (shape output) (at 121.158 60.452 0) (fields_autoplaced)
-    (effects (font (size 1.27 1.27)) (justify left))
-    (property "Intersheetrefs" "${INTERSHEET_REFS}" (at 131.3813 60.452 0)
+  (global_label "~{C2WSEL}" (shape output) (at 121.158 70.612 0) (fields_autoplaced)
+    (effects (font (size 1.27 1.27)) (justify left))
+    (property "Intersheetrefs" "${INTERSHEET_REFS}" (at 131.3813 70.612 0)
       (effects (font (size 1.27 1.27)) (justify left) hide)
     )
@@
     )
   )
-  (global_label "~{VDPRSEL}" (shape output) (at 121.158 68.072 0) (fields_autoplaced)
-    (effects (font (size 1.27 1.27)) (justify left))
-    (property "Intersheetrefs" "${INTERSHEET_REFS}" (at 132.349 68.072 0)
+  (global_label "~{VDPRSEL}" (shape output) (at 121.158 57.912 0) (fields_autoplaced)
+    (effects (font (size 1.27 1.27)) (justify left))
+    (property "Intersheetrefs" "${INTERSHEET_REFS}" (at 132.349 57.912 0)
       (effects (font (size 1.27 1.27)) (justify left) hide)
     )
@@
       (effects (font (size 1.27 1.27)) (justify left) hide)
     )
+  )
+  (global_label "~{AYSEL}" (shape output) (at 121.158 50.292 0) (fields_autoplaced)
+    (effects (font (size 1.27 1.27)) (justify left))
+    (property "Intersheetrefs" "${INTERSHEET_REFS}" (at 129.6276 50.292 0)
+      (effects (font (size 1.27 1.27)) (justify left) hide)
+    )

Commit message: Route most of the address / data lines.
Connections:
- net ~{FF1WSEL}: now also U201.20 (IO7); no longer U201.19 (IO6)
- net ~{FF2WSEL}: now also U201.19 (IO6); no longer U201.20 (IO7)
Changed lines of the file:
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@@
     )
   )
-  (global_label "~{FF2WSEL}" (shape output) (at 121.158 62.992 0) (fields_autoplaced)
+  (global_label "~{FF2WSEL}" (shape output) (at 121.158 60.452 0) (fields_autoplaced)
     (effects (font (size 1.27 1.27)) (justify left))
-    (property "Intersheetrefs" "${INTERSHEET_REFS}" (at 132.2885 62.992 0)
+    (property "Intersheetrefs" "${INTERSHEET_REFS}" (at 132.2885 60.452 0)
       (effects (font (size 1.27 1.27)) (justify left) hide)
     )
@@
     )
   )
-  (global_label "~{FF1WSEL}" (shape output) (at 121.158 60.452 0) (fields_autoplaced)
+  (global_label "~{FF1WSEL}" (shape output) (at 121.158 62.992 0) (fields_autoplaced)
     (effects (font (size 1.27 1.27)) (justify left))
-    (property "Intersheetrefs" "${INTERSHEET_REFS}" (at 132.2885 60.452 0)
+    (property "Intersheetrefs" "${INTERSHEET_REFS}" (at 132.2885 62.992 0)
       (effects (font (size 1.27 1.27)) (justify left) hide)
     )
