File: design-files/CoPicoVision_memory.kicad_sch (KiCad schematic)
At the start: 13 parts, among them U103 74ACT05, U201 GAL22V10, U202 GAL22V10, U203 AT28C64, U204 AS6C62256, U205 74HCT08, U206 74HCT74

Commit message: Put the AY-3-8910 on the board, clarify part numbers for the 74xx chips to ensure the correct SOIC footprints.
Parts:
- U103: value 74ACT05 -> MC74ACT05DR2G
- U205: value 74HCT08 -> MM74HCT08MX
- U206: value 74HCT74 -> MM74HCT74MX
Other:
- moved on the sheet: U206C
Changed lines of the file:
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@@
     (stroke (width 0) (type default))
   )
-  (wire (pts (xy 121.412 186.817) (xy 121.412 189.357))
+  (wire (pts (xy 117.475 186.817) (xy 117.475 189.357))
     (stroke (width 0) (type default))
   )
@@
     (stroke (width 0) (type default))
   )
-  (wire (pts (xy 121.412 166.497) (xy 121.412 163.957))
+  (wire (pts (xy 117.475 166.497) (xy 117.475 163.957))
     (stroke (width 0) (type default))
   )
@@
     (stroke (width 0) (type default))
   )
-  (wire (pts (xy 121.412 163.957) (xy 146.177 163.957))
+  (wire (pts (xy 117.475 163.957) (xy 146.177 163.957))
     (stroke (width 0) (type default))
   )
@@
     (stroke (width 0) (type default))
   )
-  (wire (pts (xy 121.412 189.357) (xy 146.177 189.357))
+  (wire (pts (xy 117.475 189.357) (xy 146.177 189.357))
     (stroke (width 0) (type default))
   )
@@
       (effects (font (size 1.27 1.27)) (justify left))
     )
-    (property "Value" "74HCT74" (at 156.2609 22.86 0)
+    (property "Value" "MM74HCT74MX" (at 156.2609 22.86 0)
       (effects (font (size 1.27 1.27)) (justify left))
     )
@@
       (effects (font (size 1.27 1.27)))
     )
-    (property "Value" "74HCT08" (at 166.2347 116.84 0)
+    (property "Value" "MM74HCT08MX" (at 166.2347 116.84 0)
       (effects (font (size 1.27 1.27)))
     )
@@
       (effects (font (size 1.27 1.27)) (justify left))
     )
-    (property "Value" "74HCT74" (at 156.2609 49.911 0)
+    (property "Value" "MM74HCT74MX" (at 156.2609 49.911 0)
       (effects (font (size 1.27 1.27)) (justify left))
     )
@@
     )
   )
-  (symbol (lib_id "74xx:74HC74") (at 121.412 176.657 0) (unit 3)
+  (symbol (lib_id "74xx:74HC74") (at 117.475 176.657 0) (unit 3)
     (in_bom yes) (on_board yes) (dnp no)
-    (property "Reference" "U206" (at 107.823 175.387 0)
-      (effects (font (size 1.27 1.27)) (justify left))
-    )
-    (property "Value" "74HCT74" (at 107.823 177.927 0)
-      (effects (font (size 1.27 1.27)) (justify left))
-    )
-    (property "Footprint" "Package_SO:SOIC-14_3.9x8.7mm_P1.27mm" (at 121.412 176.657 0)
-      (effects (font (size 1.27 1.27)) hide)
-    )
-    (property "Datasheet" "74xx/74hc_hct74.pdf" (at 121.412 176.657 0)
+    (property "Reference" "U206" (at 103.886 175.387 0)
+      (effects (font (size 1.27 1.27)) (justify left))
+    )
+    (property "Value" "MM74HCT74MX" (at 97.79 177.927 0)
+      (effects (font (size 1.27 1.27)) (justify left))
+    )
+    (property "Footprint" "Package_SO:SOIC-14_3.9x8.7mm_P1.27mm" (at 117.475 176.657 0)
+      (effects (font (size 1.27 1.27)) hide)
+    )
+    (property "Datasheet" "74xx/74hc_hct74.pdf" (at 117.475 176.657 0)
       (effects (font (size 1.27 1.27)) hide)
     )
@@
       (effects (font (size 1.27 1.27)))
     )
-    (property "Value" "74HCT08" (at 166.2347 142.494 0)
+    (property "Value" "MM74HCT08MX" (at 166.2347 142.494 0)
       (effects (font (size 1.27 1.27)))
     )
@@
       (effects (font (size 1.27 1.27)))
     )
-    (property "Value" "74ACT05" (at 143.129 101.6 0)
+    (property "Value" "MC74ACT05DR2G" (at 143.129 101.6 0)
       (effects (font (size 1.27 1.27)))
     )
@@
       (effects (font (size 1.27 1.27)) (justify left))
     )
-    (property "Value" "74HCT08" (at 132.08 176.911 0)
+    (property "Value" "MM74HCT08MX" (at 126.873 176.403 0)
       (effects (font (size 1.27 1.27)) (justify left))
     )
@@
       (effects (font (size 1.27 1.27)))
     )
-    (property "Value" "74HCT08" (at 166.2347 155.956 0)
+    (property "Value" "MM74HCT08MX" (at 166.2347 155.956 0)
       (effects (font (size 1.27 1.27)))
     )
@@
       (effects (font (size 1.27 1.27)))
     )
-    (property "Value" "74HCT08" (at 166.2347 129.54 0)
-      (effects (font (size 1.27 1.27)))
-    )
+    (property "Value" "MM74HCT08MX" (at 166.2347 129.54 0)
+      (effects (font (size 1.27 1.27)))
+    )

Commit message: Give a slightly more generous footprint to the RAM chip.
Parts:
- U204: value AS6C62256 -> AS6C62256-55SCN; Mouser 913-AS6C6264-55PCN -> 913-AS6C62256-55SCN
Changed lines of the file:
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@@
       (effects (font (size 1.27 1.27)) (justify left))
     )
-    (property "Value" "AS6C62256" (at 204.724 97.028 0)
+    (property "Value" "AS6C62256-55SCN" (at 204.724 97.028 0)
       (effects (font (size 1.27 1.27)) (justify left))
     )
@@
       (effects (font (size 1.27 1.27)) hide)
     )
-    (property "Datasheet" "https://ecee.colorado.edu/~mcclurel/Cypress_SRAM_CY62256.pdf" (at 201.295 121.92 0)
+    (property "Datasheet" "https://www.mouser.com/datasheet/2/12/AS6C62256_23_March_2016_rev1_2-1288423.pdf" (at 201.295 121.92 0)
       (effects (font (size 1.27 1.27)) hide)
     )
-    (property "Mouser" "913-AS6C6264-55PCN" (at 201.295 119.38 0)
+    (property "Mouser" "913-AS6C62256-55SCN" (at 201.295 119.38 0)
       (effects (font (size 1.27 1.27)) hide)
     )

Commit message: Update dates / version numbers in drawings.
Parts:
- U204: footprint Package_SO:SOIC-28W_7.5x17.9mm_P1.27mm -> Package_SO:SOIC-28W_7.5x18.7mm_P1.27mm
Changed lines of the file:
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@@
   (title_block
     (title "CoPicoVision")
-    (date "2024-10-12")
-    (rev "0.2")
+    (date "2024-12-21")
+    (rev "2.0")
     (company "(c) 2024 Jason R. Thorpe.  See LICENSE.")
   )
@@
       (effects (font (size 1.27 1.27)) (justify left))
     )
-    (property "Footprint" "Package_SO:SOIC-28W_7.5x17.9mm_P1.27mm" (at 201.295 121.92 0)
-      (effects (font (size 1.27 1.27)) hide)
-    )
+    (property "Footprint" "Package_SO:SOIC-28W_7.5x18.7mm_P1.27mm" (at 201.295 121.92 0)
+      (effects (font (size 1.27 1.27)) hide)
+    )

Commit message: Update Mouser part numbers / data sheet links.
Parts:
- U103: value MC74ACT05DR2G -> MC74ACT05D; Mouser 595-CD74ACT05EE4 -> 863-MC74ACT05DR2G
- U205: value MM74HCT08MX -> MM74HCT08M; Mouser (none) -> 512-MM74HCT08MX
- U206: value MM74HCT74MX -> MM74HCT74M; Mouser (none) -> 512-MM74HCT74MX
Changed lines of the file:
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@@
       (effects (font (size 1.27 1.27)) (justify left))
     )
-    (property "Value" "MM74HCT74MX" (at 156.2609 22.86 0)
+    (property "Value" "MM74HCT74M" (at 156.2609 22.86 0)
       (effects (font (size 1.27 1.27)) (justify left))
     )
@@
       (effects (font (size 1.27 1.27)) hide)
     )
-    (property "Datasheet" "74xx/74hc_hct74.pdf" (at 154.305 29.718 0)
+    (property "Datasheet" "https://www.mouser.com/datasheet/2/308/1/MM74HCT74_D-2315726.pdf" (at 154.305 29.718 0)
+      (effects (font (size 1.27 1.27)) hide)
+    )
+    (property "Mouser" "512-MM74HCT74MX" (at 154.305 29.718 0)
       (effects (font (size 1.27 1.27)) hide)
     )
@@
       (effects (font (size 1.27 1.27)))
     )
-    (property "Value" "MM74HCT08MX" (at 166.2347 116.84 0)
+    (property "Value" "MM74HCT08M" (at 166.2347 116.84 0)
       (effects (font (size 1.27 1.27)))
     )
@@
       (effects (font (size 1.27 1.27)) hide)
     )
-    (property "Datasheet" "http://www.ti.com/lit/gpn/sn74LS08" (at 166.243 121.92 0)
+    (property "Datasheet" "https://www.mouser.com/datasheet/2/308/1/MM74HCT08_D-2315856.pdf" (at 166.243 121.92 0)
+      (effects (font (size 1.27 1.27)) hide)
+    )
+    (property "Mouser" "512-MM74HCT08MX" (at 166.243 121.92 0)
       (effects (font (size 1.27 1.27)) hide)
     )
@@
       (effects (font (size 1.27 1.27)) (justify left))
     )
-    (property "Value" "MM74HCT74MX" (at 156.2609 49.911 0)
+    (property "Value" "MM74HCT74M" (at 156.2609 49.911 0)
       (effects (font (size 1.27 1.27)) (justify left))
     )
@@
       (effects (font (size 1.27 1.27)) hide)
     )
-    (property "Datasheet" "74xx/74hc_hct74.pdf" (at 154.305 56.769 0)
+    (property "Datasheet" "https://www.mouser.com/datasheet/2/308/1/MM74HCT74_D-2315726.pdf" (at 154.305 56.769 0)
+      (effects (font (size 1.27 1.27)) hide)
+    )
+    (property "Mouser" "512-MM74HCT74MX" (at 154.305 56.769 0)
       (effects (font (size 1.27 1.27)) hide)
     )
@@
       (effects (font (size 1.27 1.27)) (justify left))
     )
-    (property "Value" "MM74HCT74MX" (at 97.79 177.927 0)
+    (property "Value" "MM74HCT74M" (at 97.79 177.927 0)
       (effects (font (size 1.27 1.27)) (justify left))
     )
@@
       (effects (font (size 1.27 1.27)) hide)
     )
-    (property "Datasheet" "74xx/74hc_hct74.pdf" (at 117.475 176.657 0)
+    (property "Datasheet" "https://www.mouser.com/datasheet/2/308/1/MM74HCT74_D-2315726.pdf" (at 117.475 176.657 0)
+      (effects (font (size 1.27 1.27)) hide)
+    )
+    (property "Mouser" "512-MM74HCT74MX" (at 117.475 176.657 0)
       (effects (font (size 1.27 1.27)) hide)
     )
@@
       (effects (font (size 1.27 1.27)))
     )
-    (property "Value" "MM74HCT08MX" (at 166.2347 142.494 0)
+    (property "Value" "MM74HCT08M" (at 166.2347 142.494 0)
       (effects (font (size 1.27 1.27)))
     )
@@
       (effects (font (size 1.27 1.27)) hide)
     )
-    (property "Datasheet" "http://www.ti.com/lit/gpn/sn74LS08" (at 166.243 147.955 0)
+    (property "Datasheet" "https://www.mouser.com/datasheet/2/308/1/MM74HCT08_D-2315856.pdf" (at 166.243 147.955 0)
+      (effects (font (size 1.27 1.27)) hide)
+    )
+    (property "Mouser" "512-MM74HCT08MX" (at 166.243 147.955 0)
       (effects (font (size 1.27 1.27)) hide)
     )
@@
       (effects (font (size 1.27 1.27)))
     )
-    (property "Value" "MC74ACT05DR2G" (at 143.129 101.6 0)
+    (property "Value" "MC74ACT05D" (at 143.129 101.6 0)
       (effects (font (size 1.27 1.27)))
     )
@@
       (effects (font (size 1.27 1.27)) hide)
     )
-    (property "Datasheet" "https://www.ti.com/lit/ds/symlink/cd74act05.pdf" (at 143.129 106.299 0)
-      (effects (font (size 1.27 1.27)) hide)
-    )
-    (property "Mouser" "595-CD74ACT05EE4" (at 143.129 106.299 0)
+    (property "Datasheet" "https://www.mouser.com/datasheet/2/308/1/MC74AC05_D-2315319.pdf" (at 143.129 106.299 0)
+      (effects (font (size 1.27 1.27)) hide)
+    )
+    (property "Mouser" "863-MC74ACT05DR2G" (at 143.129 106.299 0)
       (effects (font (size 1.27 1.27)) hide)
     )
@@
       (effects (font (size 1.27 1.27)) (justify left))
     )
-    (property "Value" "MM74HCT08MX" (at 126.873 176.403 0)
+    (property "Value" "MM74HCT08M" (at 126.873 176.403 0)
       (effects (font (size 1.27 1.27)) (justify left))
     )
@@
       (effects (font (size 1.27 1.27)) hide)
     )
-    (property "Datasheet" "http://www.ti.com/lit/gpn/sn74LS08" (at 146.177 176.657 0)
+    (property "Datasheet" "https://www.mouser.com/datasheet/2/308/1/MM74HCT08_D-2315856.pdf" (at 146.177 176.657 0)
+      (effects (font (size 1.27 1.27)) hide)
+    )
+    (property "Mouser" "512-MM74HCT08MX" (at 146.177 176.657 0)
       (effects (font (size 1.27 1.27)) hide)
     )
@@
       (effects (font (size 1.27 1.27)))
     )
-    (property "Value" "MM74HCT08MX" (at 166.2347 155.956 0)
+    (property "Value" "MM74HCT08M" (at 166.2347 155.956 0)
       (effects (font (size 1.27 1.27)))
     )
@@
       (effects (font (size 1.27 1.27)) hide)
     )
-    (property "Datasheet" "http://www.ti.com/lit/gpn/sn74LS08" (at 166.243 161.671 0)
+    (property "Datasheet" "https://www.mouser.com/datasheet/2/308/1/MM74HCT08_D-2315856.pdf" (at 166.243 161.671 0)
+      (effects (font (size 1.27 1.27)) hide)
+    )
+    (property "Mouser" "512-MM74HCT08MX" (at 166.243 161.671 0)
       (effects (font (size 1.27 1.27)) hide)
     )
@@
       (effects (font (size 1.27 1.27)))
     )
-    (property "Value" "MM74HCT08MX" (at 166.2347 129.54 0)
+    (property "Value" "MM74HCT08M" (at 166.2347 129.54 0)
       (effects (font (size 1.27 1.27)))
     )
@@
       (effects (font (size 1.27 1.27)) hide)
     )
-    (property "Datasheet" "http://www.ti.com/lit/gpn/sn74LS08" (at 166.243 134.874 0)
-      (effects (font (size 1.27 1.27)) hide)
-    )
+    (property "Datasheet" "https://www.mouser.com/datasheet/2/308/1/MM74HCT08_D-2315856.pdf" (at 166.243 134.874 0)
+      (effects (font (size 1.27 1.27)) hide)
+    )
+    (property "Mouser" "512-MM74HCT08MX" (at 166.243 134.874 0)
+      (effects (font (size 1.27 1.27)) hide)
+    )

Commit message: Add / correct a bunch of Mouser part numbers for the BoM.
Parts:
- C201, C202, C203, C204, C205, C206: Mouser 81-RCER71E104K0A2H3B -> 581-KAM21BR71H104JT
Changed lines of the file:
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@@
       (effects (font (size 1.27 1.27)) hide)
     )
-    (property "Mouser" "81-RCER71E104K0A2H3B" (at 110.871 158.496 0)
+    (property "Mouser" "581-KAM21BR71H104JT" (at 110.871 158.496 0)
       (effects (font (size 1.27 1.27)) hide)
     )
@@
       (effects (font (size 1.27 1.27)) hide)
     )
-    (property "Mouser" "81-RCER71E104K0A2H3B" (at 87.884 158.496 0)
+    (property "Mouser" "581-KAM21BR71H104JT" (at 87.884 158.496 0)
       (effects (font (size 1.27 1.27)) hide)
     )
@@
       (effects (font (size 1.27 1.27)) hide)
     )
-    (property "Mouser" "81-RCER71E104K0A2H3B" (at 76.454 158.496 0)
+    (property "Mouser" "581-KAM21BR71H104JT" (at 76.454 158.496 0)
       (effects (font (size 1.27 1.27)) hide)
     )
@@
       (effects (font (size 1.27 1.27)) hide)
     )
-    (property "Mouser" "81-RCER71E104K0A2H3B" (at 99.441 158.496 0)
+    (property "Mouser" "581-KAM21BR71H104JT" (at 99.441 158.496 0)
       (effects (font (size 1.27 1.27)) hide)
     )
@@
       (effects (font (size 1.27 1.27)) hide)
     )
-    (property "Mouser" "81-RCER71E104K0A2H3B" (at 133.985 158.496 0)
+    (property "Mouser" "581-KAM21BR71H104JT" (at 133.985 158.496 0)
       (effects (font (size 1.27 1.27)) hide)
     )
@@
       (effects (font (size 1.27 1.27)) hide)
     )
-    (property "Mouser" "81-RCER71E104K0A2H3B" (at 122.428 158.496 0)
-      (effects (font (size 1.27 1.27)) hide)
-    )
+    (property "Mouser" "581-KAM21BR71H104JT" (at 122.428 158.496 0)
+      (effects (font (size 1.27 1.27)) hide)
+    )
