File: design-files/CoPicoVision_video.kicad_sch (KiCad schematic)
At the start: 15 parts, among them J301 DE15_Receptacle_HighDensity_M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, U103 74ACT05, U301 Pico, U302 74LVC245, U303 74LVC245

Commit message: BoM.
Parts:
- C201, C202: Mouser (none) -> 81-RCER71E104K0A2H3B
- D301: Mouser (none) -> 511-1N5817
- U103: Mouser (none) -> 595-CD74ACT05EE4
- U302, U303: Mouser (none) -> 595-SN74LVC245ANE4
Changed lines of the file:
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@@
+      (effects (font (size 1.27 1.27)) hide)
+    )
+    (property "Mouser" "595-CD74ACT05EE4" (at 133.223 25.781 0)
       (effects (font (size 1.27 1.27)) hide)
     )
@@
     )
     (property "Datasheet" "http://www.ti.com/lit/gpn/sn74HC245" (at 132.588 59.182 0)
+      (effects (font (size 1.27 1.27)) hide)
+    )
+    (property "Mouser" "595-SN74LVC245ANE4" (at 132.588 59.182 0)
       (effects (font (size 1.27 1.27)) hide)
     )
@@
       (effects (font (size 1.27 1.27)) hide)
     )
+    (property "Mouser" "81-RCER71E104K0A2H3B" (at 175.133 108.712 0)
+      (effects (font (size 1.27 1.27)) hide)
+    )
     (pin "1")
     (pin "2")
@@
     )
     (property "Datasheet" "http://www.ti.com/lit/gpn/sn74HC245" (at 186.309 61.341 0)
+      (effects (font (size 1.27 1.27)) hide)
+    )
+    (property "Mouser" "595-SN74LVC245ANE4" (at 186.309 61.341 0)
       (effects (font (size 1.27 1.27)) hide)
     )
@@
       (effects (font (size 1.27 1.27)) hide)
     )
+    (property "Mouser" "81-RCER71E104K0A2H3B" (at 186.563 108.712 0)
+      (effects (font (size 1.27 1.27)) hide)
+    )
     (pin "1")
     (pin "2")
@@
       (effects (font (size 1.27 1.27)) hide)
     )
+    (property "Mouser" "511-1N5817" (at 105.537 30.861 0)
+      (effects (font (size 1.27 1.27)) hide)
+    )

Commit message: Add title blocks.
Other:
- company: (none) -> (c) 2024 Jason R. Thorpe.  See LICENSE.
- title: (none) -> CoPicoVision
Changed lines of the file:
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@@
 (kicad_sch (version 20230121) (generator eeschema)
   (paper "A4")
+  (title_block
+    (title "CoPicoVision")
+    (date "2024-08-31")
+    (rev "0.1")
+    (company "(c) 2024 Jason R. Thorpe.  See LICENSE.")
+  )
   (junction (at 145.288 61.722) (diameter 0) (color 0 0 0 0)
   )
