File: design-files/CoPicoVision_video.kicad_sch (KiCad schematic)
At the start: 15 parts, among them J301 DE15_Receptacle_HighDensity_M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, U103 74ACT05, U301 Pico, U302 74LVC245, U303 74LVC245

Commit message: All the bypass caps are now 0805s.
Parts:
- C201, C202: footprint Capacitor_THT:C_Disc_D3.8mm_W2.6mm_P2.50mm -> Capacitor_SMD:C_0805_2012Metric_Pad1.18x1.45mm_HandSolder
Changed lines of the file:
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@@
       (effects (font (size 1.27 1.27)) (justify left))
     )
-    (property "Footprint" "Capacitor_THT:C_Disc_D3.8mm_W2.6mm_P2.50mm" (at 175.133 108.712 0)
+    (property "Footprint" "Capacitor_SMD:C_0805_2012Metric_Pad1.18x1.45mm_HandSolder" (at 175.133 108.712 0)
       (effects (font (size 1.27 1.27)) hide)
     )
@@
       (effects (font (size 1.27 1.27)) (justify left))
     )
-    (property "Footprint" "Capacitor_THT:C_Disc_D3.8mm_W2.6mm_P2.50mm" (at 186.563 108.712 0)
-      (effects (font (size 1.27 1.27)) hide)
-    )
+    (property "Footprint" "Capacitor_SMD:C_0805_2012Metric_Pad1.18x1.45mm_HandSolder" (at 186.563 108.712 0)
+      (effects (font (size 1.27 1.27)) hide)
+    )

Commit message: Controller section is mostly SMT now.
Parts:
- U103: footprint Package_DIP:DIP-14_W7.62mm_Socket -> Package_SO:SOIC-14_3.9x8.7mm_P1.27mm
Changed lines of the file:
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@@
       (effects (font (size 1.27 1.27)))
     )
-    (property "Footprint" "Package_DIP:DIP-14_W7.62mm_Socket" (at 133.223 25.781 0)
+    (property "Footprint" "Package_SO:SOIC-14_3.9x8.7mm_P1.27mm" (at 133.223 25.781 0)
       (effects (font (size 1.27 1.27)) hide)
     )

Commit message: Make the 74LVC245s SMT components.
Parts:
- U302, U303: footprint Package_DIP:DIP-20_W7.62mm_Socket -> Package_SO:SOIC-20W_7.5x12.8mm_P1.27mm
Changed lines of the file:
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@@
       (effects (font (size 1.27 1.27)) (justify left))
     )
-    (property "Footprint" "Package_DIP:DIP-20_W7.62mm_Socket" (at 132.588 59.182 0)
+    (property "Footprint" "Package_SO:SOIC-20W_7.5x12.8mm_P1.27mm" (at 132.588 59.182 0)
       (effects (font (size 1.27 1.27)) hide)
     )
@@
       (effects (font (size 1.27 1.27)) (justify left))
     )
-    (property "Footprint" "Package_DIP:DIP-20_W7.62mm_Socket" (at 186.309 61.341 0)
-      (effects (font (size 1.27 1.27)) hide)
-    )
+    (property "Footprint" "Package_SO:SOIC-20W_7.5x12.8mm_P1.27mm" (at 186.309 61.341 0)
+      (effects (font (size 1.27 1.27)) hide)
+    )

Commit message: Put the AY-3-8910 on the board, clarify part numbers for the 74xx chips to ensure the correct SOIC footprints.
Parts:
- U103: value 74ACT05 -> MC74ACT05DR2G
- U302, U303: value 74LVC245 -> SN74LVC245ADWR
Changed lines of the file:
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@@
       (effects (font (size 1.27 1.27)))
     )
-    (property "Value" "74ACT05" (at 133.223 21.082 0)
+    (property "Value" "MC74ACT05DR2G" (at 133.223 21.082 0)
       (effects (font (size 1.27 1.27)))
     )
@@
       (effects (font (size 1.27 1.27)) (justify left))
     )
-    (property "Value" "74LVC245" (at 134.5439 43.053 0)
+    (property "Value" "SN74LVC245ADWR" (at 134.5439 43.053 0)
       (effects (font (size 1.27 1.27)) (justify left))
     )
@@
       (effects (font (size 1.27 1.27)) (justify left))
     )
-    (property "Value" "74LVC245" (at 188.2649 45.212 0)
-      (effects (font (size 1.27 1.27)) (justify left))
-    )
+    (property "Value" "SN74LVC245ADWR" (at 188.2649 45.212 0)
+      (effects (font (size 1.27 1.27)) (justify left))
+    )

Commit message: Update Mouser part numbers / data sheet links.
Parts:
- U103: value MC74ACT05DR2G -> MC74ACT05D; Mouser 595-CD74ACT05EE4 -> 863-MC74ACT05DR2G
- U302, U303: value SN74LVC245ADWR -> SN74LVC245ADW; Mouser 595-SN74LVC245ANE4 -> 595-SN74LVC245ADWR
Changed lines of the file:
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@@
       (effects (font (size 1.27 1.27)))
     )
-    (property "Value" "MC74ACT05DR2G" (at 133.223 21.082 0)
+    (property "Value" "MC74ACT05D" (at 133.223 21.082 0)
       (effects (font (size 1.27 1.27)))
     )
@@
       (effects (font (size 1.27 1.27)) hide)
     )
-    (property "Datasheet" "https://www.ti.com/lit/ds/symlink/cd74act05.pdf" (at 133.223 25.781 0)
-      (effects (font (size 1.27 1.27)) hide)
-    )
-    (property "Mouser" "595-CD74ACT05EE4" (at 133.223 25.781 0)
+    (property "Datasheet" "https://www.mouser.com/datasheet/2/308/1/MC74AC05_D-2315319.pdf" (at 133.223 25.781 0)
+      (effects (font (size 1.27 1.27)) hide)
+    )
+    (property "Mouser" "863-MC74ACT05DR2G" (at 133.223 25.781 0)
       (effects (font (size 1.27 1.27)) hide)
     )
@@
       (effects (font (size 1.27 1.27)) (justify left))
     )
-    (property "Value" "SN74LVC245ADWR" (at 134.5439 43.053 0)
+    (property "Value" "SN74LVC245ADW" (at 134.5439 43.053 0)
       (effects (font (size 1.27 1.27)) (justify left))
     )
@@
       (effects (font (size 1.27 1.27)) hide)
     )
-    (property "Datasheet" "http://www.ti.com/lit/gpn/sn74HC245" (at 132.588 59.182 0)
-      (effects (font (size 1.27 1.27)) hide)
-    )
-    (property "Mouser" "595-SN74LVC245ANE4" (at 132.588 59.182 0)
+    (property "Datasheet" "https://www.ti.com/lit/ds/symlink/sn74lvc245a.pdf" (at 132.588 59.182 0)
+      (effects (font (size 1.27 1.27)) hide)
+    )
+    (property "Mouser" "595-SN74LVC245ADWR" (at 132.588 59.182 0)
       (effects (font (size 1.27 1.27)) hide)
     )
@@
       (effects (font (size 1.27 1.27)) (justify left))
     )
-    (property "Value" "SN74LVC245ADWR" (at 188.2649 45.212 0)
+    (property "Value" "SN74LVC245ADW" (at 188.2649 45.212 0)
       (effects (font (size 1.27 1.27)) (justify left))
     )
@@
       (effects (font (size 1.27 1.27)) hide)
     )
-    (property "Datasheet" "http://www.ti.com/lit/gpn/sn74HC245" (at 186.309 61.341 0)
-      (effects (font (size 1.27 1.27)) hide)
-    )
-    (property "Mouser" "595-SN74LVC245ANE4" (at 186.309 61.341 0)
-      (effects (font (size 1.27 1.27)) hide)
-    )
+    (property "Datasheet" "https://www.ti.com/lit/ds/symlink/sn74lvc245a.pdf" (at 186.309 61.341 0)
+      (effects (font (size 1.27 1.27)) hide)
+    )
+    (property "Mouser" "595-SN74LVC245ADWR" (at 186.309 61.341 0)
+      (effects (font (size 1.27 1.27)) hide)
+    )

Commit message: Add / correct a bunch of Mouser part numbers for the BoM.
Parts:
- C201, C202: Mouser 81-RCER71E104K0A2H3B -> 581-KAM21BR71H104JT
Changed lines of the file:
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@@
       (effects (font (size 1.27 1.27)) hide)
     )
-    (property "Mouser" "81-RCER71E104K0A2H3B" (at 175.133 108.712 0)
+    (property "Mouser" "581-KAM21BR71H104JT" (at 175.133 108.712 0)
       (effects (font (size 1.27 1.27)) hide)
     )
@@
       (effects (font (size 1.27 1.27)) hide)
     )
-    (property "Mouser" "81-RCER71E104K0A2H3B" (at 186.563 108.712 0)
-      (effects (font (size 1.27 1.27)) hide)
-    )
+    (property "Mouser" "581-KAM21BR71H104JT" (at 186.563 108.712 0)
+      (effects (font (size 1.27 1.27)) hide)
+    )
