File: design-files/CoPicoVision_video.kicad_sch (KiCad schematic)
At the start: 15 parts, among them J301 DE15_Receptacle_HighDensity_M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, U103 MC74ACT05D, U301 Pico, U302 SN74LVC245ADW, U303 SN74LVC245ADW

Commit message: Change the VGA resistor ladder DAC to surface mount packages.
Parts:
- removed RN301, RN302, RN303, RN304, RN305, RN306, RN307: 1K, Resistor_THT:R_Array_SIP8, symbol Device:R_Pack04_SIP
- added R501 (x3): 1K, Resistor_SMD:R_0805_2012Metric_Pad1.20x1.40mm_HandSolder, symbol Device:R_Small
- added RN301, RN302, RN303: 1K, Package_SO:SOIC-16_3.9x9.9mm_P1.27mm, symbol Device:R_Pack08
Connections:
- net B0: now also RN303.16 (R1.2)
- net B1: now also RN303.12 (R5.2)
- net B2: now also R501.1
- net B3: now also RN303.10 (R7.2), RN303.9 (R8.2)
- net G0: now also RN302.16 (R1.2)
- net G1: now also RN302.12 (R5.2)
- net G2: now also R501.1
- net G3: now also RN302.10 (R7.2), RN302.9 (R8.2)
- net R0: now also RN301.16 (R1.2)
- net R1: now also RN301.12 (R5.2)
- net R2: now also R501.1
- net R3: now also RN301.10 (R7.2), RN301.9 (R8.2)
- net VGA_B: now also R501.2, RN303.11 (R6.2), RN303.13 (R4.2), RN303.7 (R7.1), RN303.8 (R8.1)
- net VGA_G: now also R501.2, RN302.11 (R6.2), RN302.13 (R4.2), RN302.7 (R7.1), RN302.8 (R8.1)
- net VGA_R: now also R501.2, RN301.11 (R6.2), RN301.13 (R4.2), RN301.7 (R7.1), RN301.8 (R8.1)
- new net: RN303.1 (R1.1), RN303.2 (R2.1)
- new net: RN303.14 (R3.2), RN303.15 (R2.2)
- new net: RN303.3 (R3.1), RN303.4 (R4.1)
- new net: RN303.5 (R5.1), RN303.6 (R6.1)
- new net: RN301.1 (R1.1), RN301.2 (R2.1)
- new net: RN301.14 (R3.2), RN301.15 (R2.2)
- new net: RN301.3 (R3.1), RN301.4 (R4.1)
- new net: RN301.5 (R5.1), RN301.6 (R6.1)
- new net: RN302.1 (R1.1), RN302.2 (R2.1)
- new net: RN302.14 (R3.2), RN302.15 (R2.2)
- new net: RN302.3 (R3.1), RN302.4 (R4.1)
- new net: RN302.5 (R5.1), RN302.6 (R6.1)
- no-connect marks 16 -> 14

Commit message: Update issue date.
Other:
- company: (c) 2024 Jason R. Thorpe.  See LICENSE. -> (c) 2024, 2025 Jason R. Thorpe.  See LICENSE.
Changed lines of the file:
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@@
   (title_block
     (title "CoPicoVision")
-    (date "2024-12-31")
+    (date "2025-01-23")
     (rev "3.0")
-    (company "(c) 2024 Jason R. Thorpe.  See LICENSE.")
+    (company "(c) 2024, 2025 Jason R. Thorpe.  See LICENSE.")
   )
   (junction (at 145.288 61.722) (diameter 0) (color 0 0 0 0)
